File: msl_electronic_boards/powerSwitch/pcb/Project-PowerSwitch001.brd (EAGLE design)
At the start: 80 x 100 mm, 129 parts, among them IC10 BTS6133, IC11 BTS6133, IC12 BTS6133, IC15 BTS6133, IC3 LM2574M-5.0, IC4 BTS555E3146, IC7 MAX202, Q1 16Mhz, T1 BC847, T2 BC849, T5 BC849, T6 BC849, T7 BC849

Commit message: Projekt PowerSwitch
Parts:
- moved U$1 35.3 mm to (15.0, 3.05)
Changed lines of the file:
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@@
 <attribute name="OC_NEWARK" value="unknown" x="5.08" y="52.07" size="1.778" layer="27" rot="R90" display="off"/>
 </element>
-<element name="U$1" library="Microchip-MCP2551-I_SN" package="SOIC127P600X175-8N" value="MCP2551-I/SN" x="-19.05" y="-6.35">
-<attribute name="PACKAGE" value="SOIC-8" x="-19.05" y="-6.35" size="1.778" layer="27" display="off"/>
-<attribute name="OC_NEWARK" value="69K7604" x="-19.05" y="-6.35" size="1.778" layer="27" display="off"/>
-<attribute name="MPN" value="MCP2551-I/SN" x="-19.05" y="-6.35" size="1.778" layer="27" display="off"/>
-<attribute name="SUPPLIER" value="Microchip" x="-19.05" y="-6.35" size="1.778" layer="27" display="off"/>
-<attribute name="OC_FARNELL" value="9758569" x="-19.05" y="-6.35" size="1.778" layer="27" display="off"/>
+<element name="U$1" library="Microchip-MCP2551-I_SN" package="SOIC127P600X175-8N" value="MCP2551-I/SN" x="14.986" y="3.048">
+<attribute name="PACKAGE" value="SOIC-8" x="14.986" y="3.048" size="1.778" layer="27" display="off"/>
+<attribute name="OC_NEWARK" value="69K7604" x="14.986" y="3.048" size="1.778" layer="27" display="off"/>
+<attribute name="MPN" value="MCP2551-I/SN" x="14.986" y="3.048" size="1.778" layer="27" display="off"/>
+<attribute name="SUPPLIER" value="Microchip" x="14.986" y="3.048" size="1.778" layer="27" display="off"/>
+<attribute name="OC_FARNELL" value="9758569" x="14.986" y="3.048" size="1.778" layer="27" display="off"/>
 </element>
 <element name="R31" library="rcl" package="R0805" value="1k" x="-24.13" y="-15.24"/>
@@
 <wire x1="57.32" y1="38.1" x2="57.32" y2="58.42" width="0" layer="19" extent="16-16"/>
 <wire x1="57.6375" y1="27.94" x2="57.32" y2="38.1" width="0" layer="19" extent="16-16"/>
-<wire x1="-21.7678" y1="-6.985" x2="6.35" y2="18.542" width="0" layer="19" extent="1-1"/>
-<wire x1="-36.0426" y1="-12.3" x2="-21.7678" y2="-6.985" width="0" layer="19" extent="1-1"/>
+<wire x1="12.2682" y1="2.413" x2="6.35" y2="18.542" width="0" layer="19" extent="1-1"/>
+<wire x1="-36.0426" y1="-12.3" x2="12.2682" y2="2.413" width="0" layer="19" extent="1-1"/>
 <wire x1="-36.83" y1="-25.4" x2="-36.0426" y2="-12.3" width="0" layer="19" extent="1-1"/>
 <wire x1="-36.83" y1="-27.94" x2="-36.83" y2="-25.4" width="0" layer="19" extent="1-1"/>
@@
 <wire x1="21.59" y1="92.71" x2="21.59" y2="95.25" width="0" layer="19" extent="1-1"/>
 <wire x1="5" y1="5" x2="4.23" y2="22.86" width="0" layer="19" extent="16-16"/>
-<wire x1="-21.7678" y1="-5.715" x2="5" y2="5" width="0" layer="19" extent="1-1"/>
-<wire x1="-27.4574" y1="-13.1" x2="-21.7678" y2="-5.715" width="0" layer="19" extent="1-1"/>
+<wire x1="12.2682" y1="3.683" x2="5" y2="5" width="0" layer="19" extent="1-1"/>
+<wire x1="-27.4574" y1="-13.1" x2="12.2682" y2="3.683" width="0" layer="19" extent="1-1"/>
 <wire x1="-25.08" y1="-15.24" x2="-27.4574" y2="-13.1" width="0" layer="19" extent="1-1"/>
 <wire x1="-36.0426" y1="-13.1" x2="-27.4574" y2="-13.1" width="0" layer="19" extent="1-1"/>
@@
 <contactref element="U$1" pad="1"/>
 <contactref element="U$2" pad="6"/>
-<wire x1="-21.7678" y1="-4.445" x2="-36.0426" y2="-13.9" width="0" layer="19" extent="1-1"/>
+<wire x1="12.2682" y1="4.953" x2="-36.0426" y2="-13.9" width="0" layer="19" extent="1-1"/>
 </signal>
 <signal name="RXCAN">
 <contactref element="U$1" pad="4"/>
 <contactref element="U$2" pad="7"/>
-<wire x1="-21.7678" y1="-8.255" x2="-36.0426" y2="-14.7" width="0" layer="19" extent="1-1"/>
+<wire x1="12.2682" y1="1.143" x2="-36.0426" y2="-14.7" width="0" layer="19" extent="1-1"/>
 </signal>
 <signal name="CANH">
@@
 <wire x1="16.1925" y1="16.71" x2="28.8925" y2="16.71" width="0" layer="19" extent="1-1"/>
 <wire x1="3.81" y1="12.38" x2="16.1925" y2="16.71" width="0" layer="19" extent="16-16"/>
-<wire x1="-16.3322" y1="-5.715" x2="3.81" y2="12.38" width="0" layer="19" extent="1-16"/>
+<wire x1="17.7038" y1="3.683" x2="3.81" y2="12.38" width="0" layer="19" extent="1-16"/>
 </signal>
 <signal name="CANL">
@@
 <wire x1="14.2875" y1="19.25" x2="26.9875" y2="19.25" width="0" layer="19" extent="1-1"/>
 <wire x1="6.35" y1="12.7" x2="14.2875" y2="19.25" width="0" layer="19" extent="1-1"/>
-<wire x1="-16.3322" y1="-6.985" x2="6.35" y2="12.7" width="0" layer="19" extent="1-1"/>
+<wire x1="17.7038" y1="2.413" x2="6.35" y2="12.7" width="0" layer="19" extent="1-1"/>
 </signal>
 <signal name="N$15">
@@
 <contactref element="R31" pad="2"/>
 <contactref element="U$1" pad="8"/>
-<wire x1="-16.3322" y1="-4.445" x2="-23.18" y2="-15.24" width="0" layer="19" extent="1-1"/>
+<wire x1="17.7038" y1="4.953" x2="-23.18" y2="-15.24" width="0" layer="19" extent="1-1"/>
 </signal>
 <signal name="N$13">

Commit message: Projekt PowerSwitch
Parts:
- moved SV4 174.7 mm to (94.2, 82.8)
- moved JP9 117.2 mm to (32.0, 26.2)
- moved TDB-05 106.7 mm to (114.3, 86.4)
- moved T1 105.7 mm to (111.4, 81.9)
- moved R5 105.7 mm to (114.6, 82.3)
- moved JP7 95.7 mm to (7.62, 64.0), turned to 90 degrees
- moved JP6 88.2 mm to (2.54, 64.3), turned to 90 degrees
- moved SV2 71.3 mm to (94.5, 71.9)
- moved D1 63.7 mm to (104.5, 46.5)
- moved U$2 63.6 mm to (17.5, 27.4), flipped to the bottom
- moved R31 53.2 mm to (24.9, 5.33)
- moved IC15 51.5 mm to (98.8, 58.4)
- moved SV1 43.3 mm to (18.5, 93.2), turned to 0 degrees
- moved C21 42.6 mm to (12.1, 88.3), turned to 180 degrees
- moved C19 40.2 mm to (8.89, 88.3), turned to 0 degrees
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Routing:
- net GND: track 0.00 -> 20.7 mm
- net N$40: track 0.00 -> 16.4 mm, vias 0 -> 1
- net N$41: track 0.00 -> 9.40 mm
- net N$37: track 0.00 -> 5.14 mm
- net N$35: track 0.00 -> 2.43 mm
- net N$38: track 0.00 -> 2.17 mm
- net N$36: track 0.00 -> 2.11 mm
- net N$18: track 0.00 -> 2.11 mm
- net N$15: track 0.00 -> 2.11 mm
- net +5V: track 0.00 -> 2.11 mm

Commit message: PowerSwitch PCB
Parts:
- moved TDB-05 95.1 mm to (19.3, 81.8), turned to 180 degrees
- moved R5 94.5 mm to (23.6, 56.6)
- moved SV2 93.4 mm to (11.9, 28.2), turned to 180 degrees
- moved SV4 91.3 mm to (6.60, 57.1), turned to 90 degrees
- moved T1 84.9 mm to (27.1, 71.8), turned to 90 degrees
- moved IC15 62.3 mm to (38.4, 73.4), turned to 270 degrees
- moved D1 59.5 mm to (54.7, 79.0), turned to 90 degrees
- moved IC10 56.2 mm to (38.1, 81.5), turned to 270 degrees
- moved R22 44.5 mm to (31.2, 67.1), turned to 90 degrees
- moved R21 38.6 mm to (38.1, 56.9)
- moved Q1 26.0 mm to (4.83, 39.2)
- moved C5 23.9 mm to (8.00, 45.0), turned to 270 degrees
- moved C11 23.5 mm to (3.81, 38.6), turned to 180 degrees
- moved C10 23.4 mm to (3.81, 39.8), turned to 180 degrees
- moved R44 21.7 mm to (47.0, 70.9)
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Routing:
- net N$40: track 16.4 -> 16.9 mm
Other:
- board size 80 x 100 mm -> 79.7 x 100.3 mm

Commit message: PCB
Parts:
- moved SV1 22.7 mm to (16.8, 71.1)
- moved R50 20.6 mm to (38.4, 87.6), flipped to the top, turned to 0 degrees
- moved R21 20.6 mm to (38.1, 77.5), flipped to the top, turned to 0 degrees
- moved R13 17.3 mm to (38.4, 85.1), flipped to the top, turned to 0 degrees
- moved C4 14.8 mm to (26.9, 79.5)
- moved R22 14.7 mm to (38.1, 80.0), flipped to the top, turned to 0 degrees
- moved TDB-05 10.8 mm to (15.7, 91.9)
- moved R18 8.39 mm to (54.1, 95.2), turned to 270 degrees
- moved IC15 5.43 mm to (39.4, 78.7)
- moved IC3 5.39 mm to (29.0, 94.7)
- moved L3 5.11 mm to (26.4, 86.6)
- moved IC10 4.99 mm to (39.4, 86.4)
- moved LED5 4.58 mm to (49.0, 90.4)
- moved F2-0.5A 4.44 mm to (49.0, 95.8)
- moved C3 4.10 mm to (44.2, 95.8)
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Routing:
- net GND: track 20.7 -> 0.00 mm
- net N$40: track 16.9 -> 0.00 mm, vias 1 -> 0
- net N$41: track 9.69 -> 0.00 mm
- net N$37: track 5.14 -> 0.00 mm
- net N$35: track 2.43 -> 0.00 mm
- net N$38: track 2.17 -> 0.00 mm
- net N$36: track 2.11 -> 0.00 mm
- net N$18: track 2.11 -> 0.00 mm
- net N$15: track 2.11 -> 0.00 mm
- net +5V: track 2.11 -> 0.00 mm
