File: msl_electronic_boards/powerSwitch/pcb/Project-PowerSwitch001.sch (EAGLE design)
At the start: 129 parts, among them IC10 BTS6133, IC11 BTS6133, IC12 BTS6133, IC15 BTS6133, IC3 LM2574M-5.0, IC4 BTS555E3146, IC7 MAX202, Q1 16Mhz, T1 BC847, T2 BC849, T5 BC849, T6 BC849, T7 BC849

Commit message: Projekt PowerSwitch
Other:
- moved on the sheet: JP9
Changed lines of the file:
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@@
 <instance part="GND14" gate="1" x="223.52" y="104.14"/>
 <instance part="GND20" gate="1" x="243.84" y="104.14"/>
-<instance part="JP9" gate="A" x="187.96" y="114.3" rot="R270"/>
+<instance part="JP9" gate="A" x="190.5" y="114.3" rot="R270"/>
 </instances>
 <busses>
@@
 </segment>
 <segment>
-<wire x1="185.42" y1="114.3" x2="182.88" y2="114.3" width="0.1524" layer="91"/>
+<wire x1="187.96" y1="114.3" x2="182.88" y2="114.3" width="0.1524" layer="91"/>
 <label x="182.88" y="114.3" size="1.27" layer="95" rot="R180" xref="yes"/>
 <pinref part="JP9" gate="A" pin="1"/>
@@
 </segment>
 <segment>
-<wire x1="185.42" y1="111.76" x2="182.88" y2="111.76" width="0.1524" layer="91"/>
+<wire x1="187.96" y1="111.76" x2="182.88" y2="111.76" width="0.1524" layer="91"/>
 <label x="182.88" y="111.76" size="1.27" layer="95" rot="R180" xref="yes"/>
 <pinref part="JP9" gate="A" pin="2"/>

Commit message: PCB
Changed lines of the file:
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@@
 <net name="RXCAN" class="0">
 <segment>
-<wire x1="96.52" y1="124.46" x2="101.6" y2="124.46" width="0.1524" layer="91"/>
-<label x="101.6" y="124.46" size="1.27" layer="95" xref="yes"/>
+<wire x1="96.52" y1="124.46" x2="99.06" y2="124.46" width="0.1524" layer="91"/>
+<label x="99.06" y="124.46" size="1.27" layer="95" xref="yes"/>
 <pinref part="U$2" gate="G$1" pin="(RXCAN)PC3"/>
 </segment>
@@
 <net name="TXCAN" class="0">
 <segment>
-<wire x1="96.52" y1="121.92" x2="101.6" y2="121.92" width="0.1524" layer="91"/>
-<label x="101.6" y="121.92" size="1.27" layer="95" xref="yes"/>
+<wire x1="96.52" y1="121.92" x2="99.06" y2="121.92" width="0.1524" layer="91"/>
+<label x="99.06" y="121.92" size="1.27" layer="95" xref="yes"/>
 <pinref part="U$2" gate="G$1" pin="(TXCAN)PC2"/>
 </segment>
@@
 </segment>
 <segment>
-<label x="101.6" y="134.62" size="1.27" layer="95" xref="yes"/>
-<wire x1="96.52" y1="134.62" x2="101.6" y2="134.62" width="0.1524" layer="91"/>
+<label x="106.68" y="134.62" size="1.27" layer="95" xref="yes"/>
+<wire x1="96.52" y1="134.62" x2="106.68" y2="134.62" width="0.1524" layer="91"/>
 <pinref part="U$2" gate="G$1" pin="PC7"/>
 </segment>
@@
 <net name="SW_1" class="0">
 <segment>
-<label x="101.6" y="119.38" size="1.27" layer="95" xref="yes"/>
-<wire x1="96.52" y1="119.38" x2="101.6" y2="119.38" width="0.1524" layer="91"/>
+<label x="106.68" y="119.38" size="1.27" layer="95" xref="yes"/>
+<wire x1="96.52" y1="119.38" x2="106.68" y2="119.38" width="0.1524" layer="91"/>
 <pinref part="U$2" gate="G$1" pin="PC1"/>
 </segment>
