File: msl_electronic_boards/powerSwitch/pcb/powerSwitch002.brd (EAGLE design)
At the start: 80 x 100 mm, 129 parts, among them IC10 BTS6133, IC11 BTS6133, IC12 BTS6133, IC15 BTS6133, IC3 LM2574M-5.0, IC4 BTS555E3146, IC7 MAX202, Q1 16Mhz, T1 BC847, T2 BC849, T5 BC849, T6 BC849, T7 BC849

Commit message: PCB PowerSwitch
Parts:
- moved ISP 143.5 mm to (14.7, 90.9), turned to 90 degrees
- moved JP7 135.7 mm to (4.06, 85.9), turned to 270 degrees
- moved RS232 129.9 mm to (24.4, 90.9), turned to 90 degrees
- moved JP6 129.7 mm to (7.62, 85.9), turned to 270 degrees
- moved C25 113.0 mm to (32.6, 95.8), turned to 270 degrees
- moved IC7 106.5 mm to (37.7, 91.9), turned to 270 degrees
- moved R7 106.4 mm to (10.7, 24.9), turned to 270 degrees
- moved R31 106.1 mm to (1.27, 55.1), turned to 270 degrees
- moved R4 105.7 mm to (13.2, 24.9), turned to 270 degrees
- moved C20 105.4 mm to (37.7, 98.0), turned to 0 degrees
- moved R12 105.1 mm to (15.7, 24.9), turned to 270 degrees
- moved C21 100.2 mm to (42.8, 88.8), turned to 270 degrees
- moved C19 99.4 mm to (42.8, 91.9), turned to 90 degrees
- moved R25 99.2 mm to (46.7, 4.57)
- moved R26 99.2 mm to (46.7, 2.03), turned to 0 degrees
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Routing:
- net +5V: track 0.00 -> 113.4 mm, vias 0 -> 3
- net ADC5: track 0.00 -> 89.9 mm, vias 0 -> 4
- net ICLED_ROT: track 0.00 -> 87.3 mm, vias 0 -> 3
- net ICLED_KICK: track 0.00 -> 82.4 mm, vias 0 -> 2
- net ICLED_GRUEN: track 0.00 -> 68.5 mm, vias 0 -> 3
- net ICLED_AKT: track 0.00 -> 66.6 mm, vias 0 -> 3
- net ADC6: track 0.00 -> 66.2 mm
- net N$12: track 0.00 -> 61.6 mm, vias 0 -> 1
- net ADC10: track 0.00 -> 58.9 mm
- net N$23: track 0.00 -> 53.9 mm, vias 0 -> 1
- net N$19: track 0.00 -> 53.4 mm
- net ADC7: track 0.00 -> 37.2 mm, vias 0 -> 2
- net 12VIN: track 0.00 -> 37.0 mm, vias 0 -> 1
- net RXD: track 0.00 -> 33.5 mm, vias 0 -> 1
- net TXD: track 0.00 -> 33.4 mm, vias 0 -> 1
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- added copper zone on layer 16, net 12V
- added copper zone on layer 16, net 12VOUT
- added copper zone on layer 16, net AKTUATOR
- added copper zone on layer 16, net EXT
- added copper zone on layer 1, net GND
- added copper zone on layer 16, net GND
- added copper zone on layer 16, net KICKER
Other:
- board size 80 x 100 mm -> 80.5 x 100.3 mm

Commit message: PCB PowerSwitch
Parts:
- added C1: 100n, rcl:C0603
- moved R11 8.89 mm to (26.4, 71.1), flipped to the top, turned to 0 degrees
- moved R3 8.89 mm to (26.4, 68.6), flipped to the top, turned to 180 degrees
- moved SJ2 8.46 mm to (16.0, 61.7), turned to 180 degrees
- moved R1 7.04 mm to (16.0, 64.0), turned to 0 degrees
- moved R5 6.67 mm to (30.5, 61.0), turned to 90 degrees
- moved C13 6.43 mm to (16.0, 66.3), turned to 180 degrees
- moved R6 6.15 mm to (24.6, 55.4), turned to 180 degrees
- moved C12 3.30 mm to (9.40, 67.1)
- moved C5 3.30 mm to (9.40, 69.1)
- moved RJ_1 2.54 mm to (10.7, 43.2)
- moved R16 2.41 mm to (11.9, 35.3)
- moved JP1 2.09 mm to (24.6, 52.1), turned to 90 degrees
- moved C11 1.93 mm to (3.05, 68.8), turned to 90 degrees
- moved T5 1.44 mm to (11.7, 30.7), turned to 180 degrees
- moved JP6 1.30 mm to (7.87, 87.1)
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Connections:
- net +5V: now also C1.2
- net GND: now also C1.1
Routing:
- net +5V: track 113.4 -> 231.2 mm, vias 3 -> 7
- net N$25: track 14.7 -> 110.2 mm, vias 0 -> 4
- net SW_KICK: track 24.5 -> 101.0 mm, vias 0 -> 5
- net SW_1: track 3.36 -> 72.9 mm, vias 0 -> 4
- net 12VOUT: track 24.5 -> 88.6 mm, vias 1 -> 6
- net SW_MOT: track 6.22 -> 68.7 mm, vias 0 -> 1
- net SW_AKT: track 20.7 -> 70.2 mm, vias 1 -> 2
- net AKTUATOR: track 1.04 -> 46.4 mm, vias 0 -> 1
- net 24VIN: track 31.2 -> 69.8 mm, vias 2 -> 5
- net ADC3: track 7.05 -> 44.6 mm, vias 1 -> 2
- net ICLED_AKT: track 66.6 -> 97.9 mm, vias 3 -> 5
- net ICLED_GRUEN: track 68.5 -> 93.8 mm, vias 3 -> 5
- net 12VIN: track 37.0 -> 61.8 mm, vias 1 -> 2
- net EXTIN: track 15.3 -> 39.1 mm, vias 1 -> 2
- net ADC2: track 0.00 -> 21.8 mm, vias 0 -> 2
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