File: msl_electronic_boards/powerSwitch/pcb/powerSwitch002.sch (EAGLE design)
At the start: 129 parts, among them IC10 BTS6133, IC11 BTS6133, IC12 BTS6133, IC15 BTS6133, IC3 LM2574M-5.0, IC4 BTS555E3146, IC7 MAX202, Q1 16Mhz, T1 BC847, T2 BC849, T5 BC849, T6 BC849, T7 BC849

Commit message: PCB PowerSwitch
Parts:
- added C1: 100n, rcl:C-EUC0603
Connections:
- net +5V: now also C1.2
- net GND: now also C1.1
Changed lines of the file:
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@@
 <part name="GND20" library="supply1" deviceset="GND" device=""/>
 <part name="JP9" library="jumper" deviceset="JP1E" device=""/>
+<part name="C1" library="rcl" deviceset="C-EU" device="C0603" value="100n"/>
+<part name="P+11" library="supply1" deviceset="+5V" device=""/>
+<part name="GND21" library="supply1" deviceset="GND" device=""/>
 </parts>
 <sheets>
@@
 <instance part="U$1" gate="A" x="53.34" y="162.56"/>
 <instance part="R31" gate="G$1" x="22.86" y="157.48"/>
+<instance part="C1" gate="G$1" x="215.9" y="96.52" rot="MR180"/>
+<instance part="P+11" gate="1" x="215.9" y="104.14" smashed="yes">
+<attribute name="VALUE" x="218.44" y="106.68" size="1.778" layer="96" rot="R180"/>
+</instance>
+<instance part="GND21" gate="1" x="215.9" y="91.44"/>
 </instances>
 <busses>
@@
 <pinref part="P+1" gate="1" pin="+5V"/>
 <pinref part="T2" gate="G$1" pin="C"/>
+</segment>
+<segment>
+<pinref part="C1" gate="G$1" pin="2"/>
+<pinref part="P+11" gate="1" pin="+5V"/>
 </segment>
 </net>
@@
 <pinref part="KICK" gate="G$1" pin="C"/>
 </segment>
-</net>
+<segment>
+<pinref part="C1" gate="G$1" pin="1"/>
+<pinref part="GND21" gate="1" pin="GND"/>
+</segment>
+</net>
