File: msl_electronic_boards/powerSwitch/pcb/Project-PowerSwitch-005.sch (EAGLE design)
At the start: 127 parts, among them IC10 BTS6133, IC11 BTS6133, IC12 BTS6133, IC15 BTS6133, IC4 BTS555E3146, P1 39-30-06_S, P4 39-30-06_S, P6 39-30-04_S, P8 39-30-04_S, Q1 16Mhz, T1 BC847, T2 BC849, T3 BC849, T4 BC859, T5 BC849, T6 BC849, T7 BC849, U1 LM2675M

Commit message: powerswitch
Parts:
- removed 12IN+, 12IN-, 12OUT+, 12OUT-, 24IN+, 24IN-, ACTU+, ACTU-, EXT+, EXT-, KICK+, KICK-, MOT1+, MOT1-, MOT2+, MOT2-: WIREPADSMD5-5, mywirepad:WIREPADSMD5-5
- IC4: value BTS555E3146 -> BTS555; device micro-siemens:BTS555E3146 -> micro-siemens:BTS555
Connections:
- net 12VIN: no longer 12IN+.P
- net 12VOUT: no longer 12OUT+.P
- net 24VIN: no longer 24IN+.P
- net ADC2/I-AKT: now also U$2.PB5; no longer U$2.PD5
- net ADC5/I-KICK: now also U$2.PB6; no longer U$2.PB2
- net ADC6/I-MOT: now also U$2.PD5; no longer U$2.PB5
- net ADC7/I-EXT: now also U$2.PB2; no longer U$2.PB6
- net AKTUATOR: no longer ACTU+.P
- net EXTIN: no longer EXT+.P
- net GND: no longer 12IN-.P, 12OUT-.P, 24IN-.P, ACTU-.P, EXT-.P, KICK-.P, MOT1-.P, MOT2-.P
- net KICKER: no longer KICK+.P
- net MOTION: no longer MOT1+.P, MOT2+.P
Other:
- note removed: "Aktuator"
- note removed: "Bat_12V"
- note removed: "Bat_24V"
- note removed: "Motor_1"
- note removed: "Motor_2"
- note removed: "PC"
