File: msl_electronic_boards/powerSwitch/pcb/Project-PowerSwitch-005.brd (EAGLE design)
At the start: 65.3 x 99.7 mm, 130 parts, among them IC10 BTS6133, IC11 BTS6133, IC12 BTS6133, IC15 BTS6133, IC3 LM2574M-5.0, IC4 BTS555E3146, IC7 MAX202, Q1 16Mhz, T1 BC847, T2 BC849, T5 BC849, T6 BC849, T7 BC849

Commit message: rekick board  and  powerswitch board changes
Parts:
- removed C12, C13, C18, C19, C20, C21, C25: 100n, rcl:C0603K
- removed F2-0.5A: SMD-MICRO-FUSE, f-lf-omniblok-s:SMD-6,1X2,6
- removed IC3: LM2574M-5.0, linear:SO14W
- removed IC7: MAX202, maxim:SO16
- removed JP1: JP_CAN, jumper:JP1
- removed JP6, JP7: (no value), jumper:JP2
- removed JP9: (no value), jumper:JP1
- removed L1: 10µH, myrcl:R0805
- removed L3: WE-TPC 2811 10uH, rcl:POWER-CHOKE_WE-TPC
- removed R22, R47, R48, R49, R50: 10k, rcl:R0805
- removed R24: 150, rcl:R0805
- removed R42, R43, R44: 20k 0.1%, rcl:R0805
- removed RS232: (no value), con-ml:ML6
- added C2: 47µ/35V, rcl:PANASONIC_D
- added D10, D11, D8, D9: DB2430700L, DB2430700L:TMINIP2-F2-B
- added D2: ES1A, diode:SMA-DO214AC
- added F1: FUSETE5, fuse:TE5
- added L2: 100µ, Inductor-Fastron:PISM
- added LED_BLAU: (no value), led:CHIPLED_0805
- added OK1: ACPL-227-500E, optocoupler:SOIC08
- added P1, P4: 39-30-06?_S, con-molex-mini-fit:39-30-?06?
- added P6, P8: 39-30-04?_S, con-molex-mini-fit:39-30-?04?
- added R_NULL_1, R_NULL_2, R_NULL_3, R_NULL_4: 0, rcl:R0402
- added SJ1, SJ3: (no value), jumper:SJ
- added T3: BC849, transistor:SOT23
- added T4: BC859, transistor:SOT23-BEC
- added U1: LM2675M, LM2675:SOIC127P620X175-8N
- C10, C11, C14, C16, C5: device rcl:C0603K -> rcl:C0603
- C3: value VF 22/35 P-C -> 47µ/35V; device rcl:PANASONIC_C -> rcl:PANASONIC_D
- C4: value VF 220/16 K-D8 -> 10n/35V; device rcl:PANASONIC_D -> rcl:C0603
- D1: value SFS1602G -> ES1A; device ownParts:D2PAK -> diode:SMA-DO214AC
- D3: value MBRS140 -> ES1A; device diode:SMB -> diode:SMA-DO214AC
- H5, H6, H7, H8: value MOUNT-PAD-ROUND2.8 -> MOUNT-PAD-ROUND3.0; device holes:2,8-PAD -> holes:3,0-PAD
- ISP: device con-ml:ML6 -> con-ml:ML10
- JP2, JP3, JP4, JP5: device jumper:JP2 -> jumper:SJ_2
- Q1: device crystal:HC49U-V@1 -> crystal:HC49UP
- R1: value 10k -> 50k
- R12: value 150 -> 1k
- R15, R16, R17, R23: value 10k -> 100k
- R36, R38, R40: value 30k 0.1% -> 100k 0.1%
- R37, R39, R41: value 300k 0.1% -> 560k 0.1%
- R7: value 150 -> 50k
- moved IC4 95.1 mm to (8.64, 91.9), flipped to the bottom, turned to 270 degrees
- moved 12V 86.9 mm to (41.8, 3.68), turned to 180 degrees
- moved VR9 83.2 mm to (26.3, 93.3), flipped to the top, turned to 180 degrees
- moved 12IN+ 81.8 mm to (135.4, 62.7)
- moved 12IN- 81.8 mm to (143.0, 67.8)
- moved 12OUT+ 81.8 mm to (135.4, 72.9)
- moved 12OUT- 81.8 mm to (143.0, 78.0)
- moved 24IN+ 81.8 mm to (135.4, 42.4)
- moved 24IN- 81.8 mm to (143.0, 47.5)
- moved ACTU+ 81.8 mm to (135.4, 52.6)
- moved ACTU- 81.8 mm to (143.0, 57.7)
- moved EXT+ 81.8 mm to (135.4, 83.1)
- moved EXT- 81.8 mm to (143.0, 88.1)
- moved KICK+ 81.8 mm to (135.4, 32.3)
- moved KICK- 81.8 mm to (143.0, 37.3)
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Connections:
- net ADC3 renamed ADC3/I-12V
- net ADC5 renamed ADC5/I-KICK
- net ADC6 renamed ADC6/I-MOT
- net ADC7 renamed ADC7/I-EXT
- net ADC8 renamed ADC8/12VIN
- net ADC9 renamed ADC9/EXT
- net CS renamed N$3
- removed net ADC10: IC11.IS, R19.2, U$2.22
- removed net ADC2: R11.1, R9.2, U$2.13
- removed net MISO: ISP.1, U$2.1
- removed net MOSI: ISP.4, JP7.1
- removed net N$3 (its old number): IC15.IN, R22.2
- removed net N$35: C18.1, IC7.3
- removed net N$38: C21.1, IC7.6
- removed net N$39: R49.1, VR7.1
- removed net N$41: IC7.7, RS232.1
- removed net N$43: IC12.IN, R47.2
- removed net N$46: IC4.2, R48.2
- removed net N$47: R38.1, R42.2
- removed net N$48: R40.1, R43.2
- removed net N$49: R36.1, R44.2
- removed net N$51: R47.1, VR8.1
- removed net N$52: R48.1, VR9.1
- removed net N$53: IC11.IN, R49.2
- removed net N$54: R50.1, VR6.1
- removed net N$64: D3.C, IC3.12, L3.1
- removed net RESET: ISP.5
- removed net RXD: IC7.12, JP6.3
- removed net SCK: ISP.3, JP6.1
- removed net TXD: IC7.10, JP7.3
- new net ADC10/24VIN: R11.1, R9.2, U$2.22
- new net ADC2/I-AKT: IC11.IS, R19.2, U$2.13
- new net LED_3: SV4.3
- new net LED_BLAU: SV2.9, T4.C
- new net N$26: OK1.1, OK1.4
- new net N$27: C4.2, D2.K, L2.2, U1.8
- new net N$29: C4.1, U1.1
- new net N$30: OK1.7, VR6.1
- new net N$31: IC15.IN, OK1.6
- new net N$32: IC10.IN, OK1.8
- new net SW_1/SCK_A: ISP.7, U$2.12
- new net SW_2/MOSI_A: ISP.1, U$2.2
- new net SW_3: SV4.4
- new net SW_3/MISO_A: ISP.9, U$2.1
- new net SW_BLAU: SV2.10, U$2.3
- net +5V: now also C16.1, C3.+, L2.1, R25.1, R26.1, R27.1, R29.1, R4.1, T4.E, U$2.19, U1.4; no longer C12.2, C25.1, C4.+, IC3.3, IC7.16, L1.2, L3.2, R1.2, SV2.10, SV2.9, SV4.10, SV4.9, T2.3, T5.3, T6.3, T7.3
- net 12V: now also D8.A, D9.A; no longer D1.P$1
- net 12VIN: now also D3.A, P1.6
- net 12VOUT: now also D10.C, D11.C, D8.C, D9.C, F1.1, P1.5, R_NULL_3.1; no longer D1.P$3, F2-0.5A.1
- net 24VIN: now also P4.4, P4.5, P4.6
- net AKTUATOR: now also P6.3, R_NULL_2.1
- net CANH: now also RJ_1.P$2, RJ_2.P$2; no longer RJ_1.P$3, RJ_2.P$3
- net CANL: now also RJ_1.P$3, RJ_2.P$3, SJ1.1; no longer JP1.2, RJ_1.P$2, RJ_2.P$2
- net EXT: now also D10.A, D11.A; no longer D1.P$2
- net EXTIN: now also D1.A, P1.4, R1.1
- net GND: now also C2.-, D2.A, H5.B3,0, H6.B3,0, H7.B3,0, H8.B3,0, ISP.10, ISP.4, ISP.8, OK1.5, P1.1, P1.2, P1.3, P4.1, P4.2, P4.3, P6.1, P6.2, P8.1, P8.2, R36.1, R38.1, R40.1, RJ_1.P$1, RJ_2.P$1, T2.2, T3.2, T5.2, T6.2, T7.2, U1.6, VR6.3; no longer C12.1, C13.1, C20.2, C21.2, C25.2, C4.-, D3.A, GELB.C, GRÜN.C, H5.B2,8, H6.B2,8, H7.B2,8, H8.B2,8, IC3.4, IC3.5, IC3.6, IC7.11, IC7.15, IC7.8, KICK.C, R42.1, R43.1, R44.1, RJ_1.P$4, RJ_2.P$4, ROT.C, RS232.5
- net ICLED_AKT: now also GELB.C, T6.3; no longer R25.1, R4.1, T6.2
- net ICLED_GRUEN: now also GRÜN.C, T7.3; no longer R12.1, R27.1, T7.2
- net ICLED_KICK: now also KICK.C, T2.3; no longer R24.1, R29.1, T2.2
- net ICLED_ROT: now also ROT.C, T5.3; no longer R26.1, R7.1, T5.2
- net KICKER: now also P6.4, R_NULL_1.1
- net LED_1: now also SV4.7; no longer SV4.5
- net LED_2: now also SV4.5; no longer SV4.3
- net LED_GELB: now also R_NULL_2.2; no longer R4.2
- net LED_GRUEN: now also R_NULL_4.2; no longer R12.2
- net LED_KICK: now also R_NULL_1.2, SV4.9; no longer R24.2, SV4.7
- net LED_ROT: now also R_NULL_3.2; no longer R7.2
- net MOTION: now also P8.3, P8.4, R_NULL_4.1
- net N$14: now also R1.2, T3.1; no longer C16.1, L1.1, U$2.19
- net N$15: now also LED_BLAU.A, R4.2; no longer C18.2, IC7.1
- net N$16: now also LED_BLAU.C, R7.1, T3.3; no longer JP6.2, U$2.12
- net N$17: now also R7.2, T4.B; no longer JP7.2, U$2.2
- net N$18: now also JP5.2, OK1.2; no longer C19.2, IC7.4
- net N$2: now also RJ_1.P$4, RJ_2.P$4; no longer RJ_1.P$1, RJ_2.P$1
- net N$22: now also C2.+, F1.2, U1.7; no longer C3.+, F2-0.5A.2, IC3.10
- net N$25: now also D1.K, D3.K, R12.1; no longer JP5.2, R22.1, VR6.3
- net N$28: now also OK1.3, R12.2; no longer IC10.IN, R50.2
- net N$36: now also IC12.IN, VR8.1; no longer C19.1, IC7.5
- net N$37: now also IC4.2, VR9.1; no longer C20.1, IC7.2
- net N$40: now also IC11.IN, VR7.1; no longer IC7.13, RS232.3
- net N$7: now also SJ1.2; no longer JP1.1
- net RST: now also ISP.5; no longer C13.2, R1.1
- net SW_1: now also SV4.8; no longer SV4.6, U$2.3
- net SW_2: now also SV4.6; no longer SV4.4
- net SW_AKT: now also SJ3.1; no longer JP9.2
- net SW_KICK: now also SJ3.2, SV4.10; no longer JP9.1, SV4.8
Routing:
- net +5V: track 231.1 -> 8.48 mm, vias 7 -> 1
- net SW_KICK: track 99.5 -> 0.00 mm, vias 5 -> 0
- net ICLED_ROT: track 106.0 -> 7.76 mm, vias 3 -> 1
- net N$25: track 110.2 -> 14.5 mm, vias 4 -> 1
- net ICLED_AKT: track 97.7 -> 2.93 mm, vias 5 -> 1
- net ADC5/I-KICK: track 94.0 -> 0.00 mm, vias 4 -> 0
- net ICLED_GRUEN: track 94.0 -> 2.93 mm, vias 5 -> 1
- net SW_12V: track 90.3 -> 0.00 mm, vias 4 -> 0
- net ICLED_KICK: track 88.1 -> 7.76 mm, vias 3 -> 1
- net SW_1: track 72.9 -> 0.00 mm, vias 4 -> 0
- net 12VOUT: track 88.6 -> 16.1 mm, vias 6 -> 0
- net SW_AKT: track 70.8 -> 0.00 mm, vias 2 -> 0
- net 24VIN: track 68.3 -> 0.00 mm, vias 5 -> 0
- net SW_MOT: track 68.1 -> 0.00 mm, vias 1 -> 0
- net ADC6/I-MOT: track 66.0 -> 0.00 mm
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- removed copper zone on layer 16, net 12V
- removed copper zone on layer 16, net 12VOUT
- removed copper zone on layer 16, net 24VIN
- removed copper zone on layer 16, net AKTUATOR
- removed copper zone on layer 16, net EXT
- removed copper zone on layer 1, net GND
- removed copper zone on layer 16, net GND
- removed copper zone on layer 16, net KICKER
- removed copper zone on layer 16, net MOTION

Commit message: powerswitch 005
Parts:
- moved R5 86.7 mm to (104.6, 66.4)
- moved C1 85.4 mm to (101.9, 76.2)
- moved ISP 85.4 mm to (89.8, 76.2)
- moved T1 85.4 mm to (105.7, 71.8)
- moved TDB-05 85.4 mm to (101.9, 76.2)
- moved R41 76.3 mm to (101.2, 79.8)
- moved R40 75.4 mm to (98.0, 79.6)
- moved VR7 46.7 mm to (84.3, 56.4), turned to 180 degrees
- moved R37 44.9 mm to (81.3, 56.4), turned to 270 degrees
- moved R36 43.9 mm to (79.0, 56.4), turned to 90 degrees
- moved IC4 36.5 mm to (35.1, 66.8), flipped to the top, turned to 180 degrees
- moved R2 29.4 mm to (2.29, 79.8), turned to 180 degrees
- moved R3 29.4 mm to (2.29, 79.8), turned to 0 degrees
- moved R10 28.2 mm to (2.29, 77.5), turned to 0 degrees
- moved R8 28.2 mm to (2.29, 77.5), turned to 180 degrees
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Routing:
- net 24VIN: track 0.00 -> 59.9 mm, vias 0 -> 1
- net MOTION: track 0.00 -> 41.2 mm

Commit message: powerswitch
Parts:
- removed 12IN+, 12IN-, 12OUT+, 12OUT-, 24IN+, 24IN-, ACTU+, ACTU-, EXT+, EXT-, KICK+, KICK-, MOT1+, MOT1-, MOT2+, MOT2-: WIREPADSMD5-5, mywirepad:5-5
- IC4: value BTS555E3146 -> BTS555; device micro-siemens:TO220-52 -> micro-siemens:TO220-51
- moved C1 98.0 mm to (6.48, 53.5), turned to 270 degrees
- moved T1 97.4 mm to (9.91, 53.7), flipped to the bottom
- moved TDB-05 97.3 mm to (7.24, 53.5), turned to 270 degrees
- moved R5 94.2 mm to (10.8, 58.7), flipped to the bottom, turned to 270 degrees
- moved ISP 73.8 mm to (18.4, 95.0), turned to 180 degrees
- moved R_NULL_1 67.3 mm to (75.3, 39.8)
- moved R41 61.2 mm to (41.3, 92.3), turned to 0 degrees
- moved R40 58.7 mm to (41.3, 94.6), turned to 180 degrees
- moved SJ3 50.0 mm to (10.4, 35.8), turned to 90 degrees
- moved VR7 48.1 mm to (36.6, 50.3), flipped to the bottom, turned to 270 degrees
- moved R_NULL_4 42.1 mm to (75.3, 38.0)
- moved R_NULL_2 41.9 mm to (75.6, 35.7)
- moved R_NULL_3 41.2 mm to (75.4, 33.1)
- moved R37 38.6 mm to (43.4, 48.8), flipped to the bottom, turned to 180 degrees
- moved SV2 37.7 mm to (5.08, 31.5)
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Connections:
- net 12VIN: no longer 12IN+.P$1
- net 12VOUT: no longer 12OUT+.P$1
- net 24VIN: no longer 24IN+.P$1
- net ADC2/I-AKT: now also U$2.26; no longer U$2.13
- net ADC5/I-KICK: now also U$2.27; no longer U$2.16
- net ADC6/I-MOT: now also U$2.13; no longer U$2.26
- net ADC7/I-EXT: now also U$2.16; no longer U$2.27
- net AKTUATOR: no longer ACTU+.P$1
- net EXTIN: no longer EXT+.P$1
- net GND: no longer 12IN-.P$1, 12OUT-.P$1, 24IN-.P$1, ACTU-.P$1, EXT-.P$1, KICK-.P$1, MOT1-.P$1, MOT2-.P$1
- net KICKER: no longer KICK+.P$1
- net MOTION: no longer MOT1+.P$1, MOT2+.P$1
Routing:
- net SW_AKT: track 0.00 -> 80.4 mm, vias 0 -> 2
- net RXCAN: track 0.00 -> 79.0 mm, vias 0 -> 1
- net TXCAN: track 0.00 -> 77.3 mm, vias 0 -> 1
- net AKTUATOR: track 0.00 -> 61.6 mm, vias 0 -> 1
- net KICKER: track 0.00 -> 58.7 mm, vias 0 -> 1
- net SW_MOT: track 0.00 -> 55.3 mm, vias 0 -> 1
- net SW_BLAU: track 0.00 -> 53.5 mm, vias 0 -> 1
- net SW_12V: track 0.00 -> 44.9 mm, vias 0 -> 1
- net SW_1/SCK_A: track 0.00 -> 37.4 mm, vias 0 -> 1
- net CANH: track 0.00 -> 32.2 mm, vias 0 -> 1
- net 24VIN: track 59.9 -> 89.2 mm, vias 1 -> 0
- net RST: track 0.00 -> 27.6 mm, vias 0 -> 1
- net N$32: track 26.7 -> 0.00 mm, vias 1 -> 0
- net CANL: track 0.00 -> 25.5 mm
- net N$40: track 0.00 -> 25.0 mm
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- added copper zone on layer 1, net GND
- added copper zone on layer 16, net GND
- added copper zone on layer 16, net N$34
Other:
- board size 65.3 x 99.7 mm -> 53.3 x 99.7 mm
- board text added: "Carpe Noctem 2016"
- board text added: "PowerSwitch-005"
- board text removed: "Carpe Noctem 2015"
- board text removed: "PowerSwitch-002"

Commit message: PowerSwitch CN 2016 v1.0 finished
Parts:
- moved R_NULL_3 68.4 mm to (7.62, 24.4), turned to 90 degrees
- moved R_NULL_2 67.0 mm to (9.14, 26.9), turned to 90 degrees
- moved R_NULL_4 65.5 mm to (10.3, 29.8), turned to 90 degrees
- moved R_NULL_1 62.7 mm to (14.6, 23.9), turned to 90 degrees
- moved R9 8.98 mm to (12.6, 61.0), turned to 90 degrees
- moved R7 7.44 mm to (22.0, 5.84), turned to 90 degrees
- moved SJ2 7.01 mm to (25.3, 13.8), turned to 180 degrees
- moved R11 6.97 mm to (14.9, 61.0), flipped to the bottom, turned to 270 degrees
- moved R41 4.10 mm to (37.5, 93.9), turned to 270 degrees
- moved R6 2.56 mm to (17.9, 17.1), turned to 270 degrees
- moved R5 2.34 mm to (10.3, 61.0)
- moved 12V 2.29 mm to (50.8, 28.8)
- moved 5V 2.29 mm to (50.8, 26.5)
- moved R18 2.29 mm to (46.0, 26.5)
- moved R28 2.29 mm to (46.0, 28.8)
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Routing:
- net +5V: track 24.8 -> 187.1 mm, vias 3 -> 6
- net MOTION: track 28.8 -> 150.8 mm, vias 0 -> 2
- net ICLED_GRUEN: track 2.93 -> 100.0 mm, vias 1 -> 3
- net ICLED_KICK: track 7.76 -> 100.2 mm, vias 1 -> 4
- net ICLED_AKT: track 2.93 -> 94.1 mm, vias 1 -> 5
- net ICLED_ROT: track 7.76 -> 93.3 mm, vias 1 -> 4
- net N$23: track 0.00 -> 72.3 mm, vias 0 -> 2
- net ADC3/I-12V: track 13.6 -> 71.1 mm, vias 0 -> 3
- net LED_BLAU: track 0.00 -> 48.7 mm, vias 0 -> 1
- net EXTIN: track 14.7 -> 59.0 mm
- net 12VOUT: track 29.4 -> 69.7 mm, vias 0 -> 4
- net 12VIN: track 15.2 -> 50.9 mm
- net ADC7/I-EXT: track 4.02 -> 35.8 mm, vias 0 -> 1
- net SW_KICK: track 5.33 -> 35.9 mm
- net AKTUATOR: track 61.6 -> 89.7 mm, vias 1 -> 3
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- removed copper zone on layer 16, net N$34
Other:
- board text added: "PowerSwitch CN 2016"
- board text added: "v1.0"
- board text removed: "Carpe Noctem 2016"
- board text removed: "PowerSwitch-005"
