File: msl_electronic_boards/rekick2015/pcb/rekick2015-001.sch (EAGLE design)
At the start: 35 parts, among them Q1 16MHz, U1 TXB0108PWR, U2 LM2675M-3.3, U3 HIP4082IBZ

Commit message: rekick2015 schematic
Parts:
- added D101: 270V, diode:ZENER-DIODESOD57-10
- added D102, D103: 3.9V, diode:DIODE-SOD323-W
- added IC1: LM393D, linear:LM393D
- added R101: 1M, rcl:R-EU_0207/15
- added R102: 470k, rcl:R-EU_0207/15
- added R103: 10k, rcl:R-EU_R0805
- added R104: 20k, rcl:R-EU_R0805
- added R105: 1k, rcl:R-EU_R0805
- added R106: 1, rcl:R-EU_R0805
Connections:
- new net CAP_330V: R101.2, R102.2
- new net CAP_GND: R103.1, R104.1
- new net N$13: IC1A.-IN, IC1A.OUT, R105.1
- new net N$14: IC1B.-IN, IC1B.OUT, R106.1
- new net N$15: IC1A.+IN, R101.1, R103.2
- new net N$21: D101.A, IC1B.+IN, R104.2
- new net N$22: D101.C, R102.1
- new net ZU-ADC-FEIN: D103.C, R106.2
- new net ZU-ADC-GROB: D102.C, R105.2
- net GND: now also D102.A, D103.A
Changed lines of the file:
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@@
 <part name="SHUNT" library="rcl" deviceset="R-EU_" device="0204/2V" value="200µ"/>
 <part name="SUPPLY3" library="supply2" deviceset="GND1" device=""/>
+<part name="FRAME5" library="frames" deviceset="A4L-LOC" device=""/>
+<part name="IC1" library="linear" deviceset="LM393" device="D"/>
+<part name="R101" library="rcl" deviceset="R-EU_" device="0207/15" value="1M">
+<attribute name="FARNELL" value="2396016"/>
+</part>
+<part name="R102" library="rcl" deviceset="R-EU_" device="0207/15" value="470k">
+<attribute name="FARNELL" value=""/>
+</part>
+<part name="D101" library="diode" deviceset="ZENER-DIODE" device="SOD57-10" value="270V">
+<attribute name="FARNELL" value="9398597"/>
+</part>
+<part name="R104" library="rcl" deviceset="R-EU_" device="R0805" value="20k"/>
+<part name="R103" library="rcl" deviceset="R-EU_" device="R0805" value="10k"/>
+<part name="R105" library="rcl" deviceset="R-EU_" device="R0805" value="1k"/>
+<part name="R106" library="rcl" deviceset="R-EU_" device="R0805" value="1"/>
+<part name="D102" library="diode" deviceset="DIODE-" device="SOD323-W" value="3.9V">
+<attribute name="FARNELL" value="2069513"/>
+</part>
+<part name="D103" library="diode" deviceset="DIODE-" device="SOD323-W" value="3.9V">
+<attribute name="FARNELL" value="2069513"/>
+</part>
+<part name="GND8" library="supply1" deviceset="GND" device=""/>
+<part name="GND9" library="supply1" deviceset="GND" device=""/>
 </parts>
 <sheets>
@@
 </nets>
 </sheet>
+<sheet>
+<description>Überwachung/Monitoring</description>
+<plain>
+</plain>
+<instances>
+<instance part="FRAME5" gate="G$1" x="0" y="0"/>
+<instance part="IC1" gate="A" x="88.9" y="144.78"/>
+<instance part="IC1" gate="B" x="88.9" y="127"/>
+<instance part="R101" gate="G$1" x="66.04" y="154.94" rot="R90">
+<attribute name="FARNELL" x="66.04" y="154.94" size="1.778" layer="96" rot="R90" align="top-left" display="name"/>
+</instance>
+<instance part="R102" gate="G$1" x="43.18" y="154.94" rot="R90">
+<attribute name="FARNELL" x="43.18" y="154.94" size="1.778" layer="96" rot="R90" align="top-left" display="name"/>
+</instance>
+<instance part="D101" gate="G$1" x="43.18" y="139.7" rot="R90">
+<attribute name="FARNELL" x="43.18" y="139.7" size="1.778" layer="96" rot="R90" align="top-left" display="name"/>
+</instance>
+<instance part="R104" gate="G$1" x="43.18" y="121.92" rot="R90"/>
+<instance part="R103" gate="G$1" x="66.04" y="121.92" rot="R90"/>
+<instance part="R105" gate="G$1" x="111.76" y="144.78"/>
+<instance part="R106" gate="G$1" x="111.76" y="127"/>
+<instance part="D102" gate="G$1" x="119.38" y="139.7" rot="R90">
+<attribute name="FARNELL" x="119.38" y="139.7" size="1.778" layer="96" rot="R90" align="top-left" display="name"/>
+</instance>
+<instance part="D103" gate="G$1" x="119.38" y="121.92" rot="R90">
+<attribute name="FARNELL" x="119.38" y="121.92" size="1.778" layer="96" rot="R90" align="top-left" display="name"/>
+</instance>
+<instance part="GND8" gate="1" x="119.38" y="132.08"/>
+<instance part="GND9" gate="1" x="119.38" y="114.3"/>
+</instances>
+<busses>
+</busses>
+<nets>
+<net name="CAP_330V" class="0">
+<segment>
+<wire x1="25.4" y1="165.1" x2="43.18" y2="165.1" width="0.1524" layer="91"/>
+<label x="25.4" y="165.1" size="1.778" layer="95" rot="R180" xref="yes"/>
+<pinref part="R102" gate="G$1" pin="2"/>
+<wire x1="43.18" y1="165.1" x2="66.04" y2="165.1" width="0.1524" layer="91"/>
+<wire x1="43.18" y1="160.02" x2="43.18" y2="165.1" width="0.1524" layer="91"/>
+<junction x="43.18" y="165.1"/>
+<pinref part="R101" gate="G$1" pin="2"/>
+<wire x1="66.04" y1="165.1" x2="66.04" y2="160.02" width="0.1524" layer="91"/>
+</segment>
+</net>
+<net name="CAP_GND" class="0">
+<segment>
+<wire x1="27.94" y1="111.76" x2="43.18" y2="111.76" width="0.1524" layer="91"/>
+<label x="27.94" y="111.76" size="1.778" layer="95" rot="R180" xref="yes"/>
+<pinref part="R104" gate="G$1" pin="1"/>
+<wire x1="43.18" y1="111.76" x2="66.04" y2="111.76" width="0.1524" layer="91"/>
+<wire x1="43.18" y1="116.84" x2="43.18" y2="111.76" width="0.1524" layer="91"/>
+<junction x="43.18" y="111.76"/>
+<pinref part="R103" gate="G$1" pin="1"/>
+<wire x1="66.04" y1="116.84" x2="66.04" y2="111.76" width="0.1524" layer="91"/>
+</segment>
+</net>
+<net name="N$13" class="0">
+<segment>
+<pinref part="IC1" gate="A" pin="OUT"/>
+<wire x1="96.52" y1="144.78" x2="101.6" y2="144.78" width="0.1524" layer="91"/>
+<wire x1="101.6" y1="144.78" x2="101.6" y2="137.16" width="0.1524" layer="91"/>
+<wire x1="101.6" y1="137.16" x2="78.74" y2="137.16" width="0.1524" layer="91"/>
+<wire x1="78.74" y1="137.16" x2="78.74" y2="142.24" width="0.1524" layer="91"/>
+<pinref part="IC1" gate="A" pin="-IN"/>
+<wire x1="78.74" y1="142.24" x2="81.28" y2="142.24" width="0.1524" layer="91"/>
+<wire x1="101.6" y1="144.78" x2="106.68" y2="144.78" width="0.1524" layer="91"/>
+<junction x="101.6" y="144.78"/>
+<pinref part="R105" gate="G$1" pin="1"/>
+</segment>
+</net>
+<net name="N$14" class="0">
+<segment>
+<pinref part="IC1" gate="B" pin="OUT"/>
+<wire x1="96.52" y1="127" x2="101.6" y2="127" width="0.1524" layer="91"/>
+<wire x1="101.6" y1="127" x2="101.6" y2="116.84" width="0.1524" layer="91"/>
+<wire x1="101.6" y1="116.84" x2="78.74" y2="116.84" width="0.1524" layer="91"/>
+<wire x1="78.74" y1="116.84" x2="78.74" y2="124.46" width="0.1524" layer="91"/>
+<pinref part="IC1" gate="B" pin="-IN"/>
+<wire x1="78.74" y1="124.46" x2="81.28" y2="124.46" width="0.1524" layer="91"/>
+<wire x1="101.6" y1="127" x2="106.68" y2="127" width="0.1524" layer="91"/>
+<junction x="101.6" y="127"/>
+<pinref part="R106" gate="G$1" pin="1"/>
+</segment>
+</net>
+<net name="N$15" class="0">
+<segment>
+<pinref part="IC1" gate="A" pin="+IN"/>
+<wire x1="81.28" y1="147.32" x2="66.04" y2="147.32" width="0.1524" layer="91"/>
+<pinref part="R101" gate="G$1" pin="1"/>
+<wire x1="66.04" y1="149.86" x2="66.04" y2="147.32" width="0.1524" layer="91"/>
+<pinref part="R103" gate="G$1" pin="2"/>
+<wire x1="66.04" y1="147.32" x2="66.04" y2="127" width="0.1524" layer="91"/>
+<junction x="66.04" y="147.32"/>
+</segment>
+</net>
+<net name="N$21" class="0">
+<segment>
+<pinref part="IC1" gate="B" pin="+IN"/>
+<wire x1="81.28" y1="129.54" x2="43.18" y2="129.54" width="0.1524" layer="91"/>
+<pinref part="D101" gate="G$1" pin="A"/>
+<wire x1="43.18" y1="137.16" x2="43.18" y2="129.54" width="0.1524" layer="91"/>
+<pinref part="R104" gate="G$1" pin="2"/>
+<wire x1="43.18" y1="129.54" x2="43.18" y2="127" width="0.1524" layer="91"/>
+<junction x="43.18" y="129.54"/>
+</segment>
+</net>
+<net name="N$22" class="0">
+<segment>
+<pinref part="R102" gate="G$1" pin="1"/>
+<pinref part="D101" gate="G$1" pin="C"/>
+<wire x1="43.18" y1="149.86" x2="43.18" y2="142.24" width="0.1524" layer="91"/>
+</segment>
+</net>
+<net name="ZU-ADC-GROB" class="0">
+<segment>
+<pinref part="R105" gate="G$1" pin="2"/>
+<wire x1="116.84" y1="144.78" x2="119.38" y2="144.78" width="0.1524" layer="91"/>
+<pinref part="D102" gate="G$1" pin="C"/>
+<wire x1="119.38" y1="144.78" x2="124.46" y2="144.78" width="0.1524" layer="91"/>
+<wire x1="119.38" y1="142.24" x2="119.38" y2="144.78" width="0.1524" layer="91"/>
+<junction x="119.38" y="144.78"/>
+<label x="124.46" y="144.78" size="1.778" layer="95" xref="yes"/>
+</segment>
+</net>
+<net name="ZU-ADC-FEIN" class="0">
+<segment>
+<pinref part="R106" gate="G$1" pin="2"/>
+<wire x1="116.84" y1="127" x2="119.38" y2="127" width="0.1524" layer="91"/>
+<pinref part="D103" gate="G$1" pin="C"/>
+<wire x1="119.38" y1="127" x2="124.46" y2="127" width="0.1524" layer="91"/>
+<wire x1="119.38" y1="124.46" x2="119.38" y2="127" width="0.1524" layer="91"/>
+<junction x="119.38" y="127"/>
+<label x="124.46" y="127" size="1.778" layer="95" xref="yes"/>
+</segment>
+</net>
+<net name="GND" class="0">
+<segment>
+<pinref part="D102" gate="G$1" pin="A"/>
+<wire x1="119.38" y1="137.16" x2="119.38" y2="134.62" width="0.1524" layer="91"/>
+<pinref part="GND8" gate="1" pin="GND"/>
+</segment>
+<segment>
+<pinref part="D103" gate="G$1" pin="A"/>
+<wire x1="119.38" y1="119.38" x2="119.38" y2="116.84" width="0.1524" layer="91"/>
+<pinref part="GND9" gate="1" pin="GND"/>
+</segment>
+</net>
+</nets>
+</sheet>
+<sheet>
+<plain>
+</plain>
+<instances>
+</instances>
+<busses>
+</busses>
+<nets>
+</nets>
+</sheet>

Commit message: Rekick 2015
Parts:
- added C14, C15, C16: 100p, rcl:C-EUC0603
- added D5: 270V, diode:ZENER-DIODESOD57-10
- added IC3: LM393D, linear:LM393D
- added Q2: SiHB24N65E, transistor-power:IRG4BC15UD-S
- added R2, R3: 47, resistor-power:RHS50
- added R4, R8: 10k, rcl:R-EU_R0805
- added R5: 470k, rcl:R-EU_0207/15
- added R6: 20k, rcl:R-EU_R0805
- added R7: 7,5k, rcl:R-EU_R0805
- added R9: 11k, rcl:R-EU_R0805
- added U4: LM2675M-12, LM2675M-12:LM2675M-12
Connections:
- new net N$23: R2.2, R3.1
- new net N$24: Q2.C, R3.2
- new net N$25: R8.2, R9.1
- new net N$27: IC3B.-IN, R4.2, R7.1
- new net N$29: C16.1, D5.A, IC3A.+IN, IC3B.+IN, R6.2
- new net N$30: D5.C, R5.1
- new net NOTAUS: Q2.G
- new net ZU-NOTAUS: IC3B.OUT
- new net ZU-TREIBER-AUS: IC3A.OUT
- net +5V: now also R7.2, R9.2
- net CAP_330V: now also R2.1, R5.2
- net CAP_GND: now also C14.2, C15.2, C16.2, Q2.E, R6.1
- net GND: now also R4.1, R8.1
- net N$15: now also C15.1
- net N$21: now also C14.1

Commit message: new rekick
Parts:
- removed D101, D5: 270V, diode:ZENER-DIODESOD57-10
- removed D102, D103: 3.9V, diode:DIODE-SOD323-W
- removed IC3: LM393D, linear:LM393D
- removed R102: 470k, rcl:R-EU_0207/15
- removed R104: 20k, rcl:R-EU_R0805
- removed R106: 1, rcl:R-EU_R0805
- removed SHUNT: 200µ, rcl:R-EU_0204/2V
- removed U$5, U$6: (no value), PSMN0R9:PSMN0R9
- added C17, C20: 47µF/35V, rcl:CPOL-EUD
- added C18, C21: 47µF/16V, rcl:CPOL-EUD
- added C19, C22: 10nF/50V, rcl:C-EUC0603
- added C23, C24: 100p, rcl:C-EUC0603
- added C25: 2200µ, rcl:CPOL-EUE10-20
- added CF, CSS, C_DELAY, C_ISEN_A, C_ISEN_B: (no value), rcl:C-EUC0603
- added C_BOOT: 100n, rcl:C-EUC0603
- added D10, D11, D8, D9: STTH1R06A, diode:GF1
- added D6, D7: ES1A, diode:GF1
- added IC2: 4043D, 40xx:4043D
- added L3: 20µ, rcl:L-EUTJ9-U2
- added L4: 820n, rcl:L-EUTJ9-U2
- added L5: 100µH, Inductor-Fastron:L-EUPISM
- added L6: 150µH, Inductor-Fastron:L-EUPISM
- added L7: (no value), EagleLibrary_Wuerth_Elektronik_eiSos_rev15h:WE-LLCR_760895641
- added OK1, OK2: ILD213, optocoupler:ILD213
- added Q3, Q4: (no value), transistor-power:PMOSFET_NTO220BV
- added R10, R11: 1k, rcl:R-EU_R0805
- added RF_MAX, RF_MIN, R_DELAY, R_ISEN_A, R_ISEN_B, R_SS, R_SS2: (no value), rcl:R-EU_R0805
- added R_LINE: 10k, rcl:R-EU_R0805
- C1: value 100µF/35V -> 47µF/35V; device rcl:CPOL-EUUD-6,3X7,7 -> rcl:CPOL-EUD
- C10, C9: value 560µ -> 2200µ
- C11: value 220n -> 100n
- C12: value 220n -> (none)
- C13: value 100n -> 2.2µ; device rcl:C-EUC0603 -> rcl:C-EUC1206
- C2: value 68µF/16V -> 47µF/16V; device rcl:CPOL-EUUD-6,3X7,7 -> rcl:CPOL-EUD
- D1: value MBRS130LT3 -> GF1; device diode:MBRS130LT3 -> diode:GF1
- D2: value MBRS130LT3 -> ES1A; device diode:MBRS130LT3 -> diode:GF1
- D3, D4: value MBRS360 -> MBR0520LT; device diode:MBRS130LT3 -> diode:MBR0520LT
- IC1: value LM393D -> LM1458D; device linear:LM393D -> linear:LM1458D
- L1: value 47µH -> 68µH; device rcl:L-EUPIS2816 -> Inductor-Fastron:L-EUPISM
- L2: device myrcl:L-EU-0805L0805 -> rcl:L-EUL2012C
- Q1: device crystal:CRYSTALHC49U-V -> crystal:CRYSTALHC49UP
- R103: value 10k -> 12k
- R105: value 1k -> 10
- R5: value 470k -> 1M; FARNELL (none) -> 2396016
- R6: value 20k -> 12k
- R7: value 7,5k -> 20k
- R8: value 10k -> 1k
- R9: value 11k -> 10k
- U$3: value (none) -> L6599; device PSMN0R9:PSMN0R9 -> l6599:L6599
- U$4: value (none) -> TMH-D; device PSMN0R9:PSMN0R9 -> traco-tm:TMH-D
- U2: value LM2675M-3.3 -> LM2675
- U3: value HIP4082IBZ -> LM2675; device Intersil-HIP4082IBZ:HIP4082IBZ -> LM2675M-3.3:LM2675M-3.3
- U4: value LM2675M-12 -> LM2675; device LM2675M-12:LM2675M-12 -> LM2675M-3.3:LM2675M-3.3
Connections:
- removed net !V_PWM: U3.ALI
- removed net CAP_GND: C14.2, C15.2, C16.2, Q2.E, R103.1, R104.1, R6.1
- removed net V_DELAY: U3.DEL
- removed net V_DISABLE: U3.DIS
- removed net V_PWM: U3.BLI
- removed net ZU-ADC-FEIN: D103.C, R106.2
- removed net ZU-ADC-GROB: D102.C, R105.2
- removed net ZU-NOTAUS: IC3B.OUT
- removed net ZU-TREIBER-AUS: IC3A.OUT
- new net 1.25V-BIS-6V: R_LINE.2, U$3.LINE
- new net CAP_+12V: IC1P.V+, OK1A.COL, R7.2, U$4.+U_OUT
- new net CAP_-12V: IC1P.V-, U$4.-U_OUT
- new net CAP_0V: C14.2, C15.2, C16.2, C25.-, D10.A, D11.A, OK1B.C, OK2A.C, Q2.E, R103.1, R11.1, R4.1, R6.1, U$4.0V
- new net MCU_UIN: IC2A.R0
- new net N$26: C22.2, D7.C, L6.2, U4.VSW
- new net N$28: C_ISEN_B.1, D3.C, R_ISEN_B.2, U$3.ISEN
- new net N$31: D3.A, D4.C, R_ISEN_A.1
- new net N$32: C_ISEN_A.1, R_ISEN_A.2
- new net N$33: C22.1, U4.CB
- new net N$34: D10.C, D8.A, L7.8
- new net N$35: OK2A.A, R9.2
- new net N$36: D11.C, D9.A, L7.1
- new net N$39: IC2A.S1
- new net N$40: IC2A.R1
- new net SEK-FEEDBACK: C12.1, RF_MAX.1, U$3.STBY
- new net TASTER: IC2A.S3
- new net TRAFO1: C_BOOT.2, L3.1, L7.3, Q3.S, Q4.D, U$3.OUT
- new net TRAFO2: L3.2, L4.1, L7.2
- new net U_IN: IC2A.S0
- new net VON_NOTAUS: Q2.G
- new net ZU-ADC_OPV: C23.1, OK1B.EMIT, R8.2
- new net ZU-NOTAUS-FF: C24.1, OK2A.EMIT, R10.2
- new net ZU_CR_LR-KNOTEN: C13.1, C_ISEN_A.2, L4.2
- new net ÜBERSPANNUNG: IC2A.S2
- net +12V: now also C11.1, C21.+, L6.1, OK1B.COL, U$3.VCC, U4.FB; no longer C13.1, D3.A, D4.A, U3.AHI, U3.BHI, U3.VDD
- net +24V: now also C1.+, C17.+, C20.+, D1.C, F1.1, U$4.U_IN, U2.VIN, U3.VIN, U4.VIN; no longer F1.2
- net +3V3: now also C2.+, L1.1, U2.FB
- net +5V: now also C18.+, IC2P.VDD, L5.1, OK2A.COL, R_LINE.1, U3.FB; no longer C2.+, L1.1, R7.2, R9.2, U2.FB
- net BOOSTER_24V: now also Q3.D; no longer U$3.D, U$5.D
- net CAP_330V: now also C25.+, D8.C, D9.C; no longer R102.2
- net GND: now also C11.2, C12.2, C17.-, C18.-, C20.-, C21.-, C23.2, C24.2, CF.2, CSS.2, C_DELAY.2, C_ISEN_B.2, D4.A, D6.A, D7.A, IC2A.R2, IC2A.R3, IC2P.VSS, R10.1, RF_MIN.1, R_DELAY.1, R_ISEN_B.1, U$3.GND, U$4.GND, U2.GND, U3.GND, U4.GND; no longer D102.A, D103.A, R4.1
- net GND1: now also Q4.S; no longer SHUNT.1, U3.VSS
- net N$1: now also C19.2, D6.C, L5.2, U3.VSW; no longer C3.2, U2.CB
- net N$11: now also CF.1, U$3.CF; no longer C11.1, D3.C, U3.BHB
- net N$12: now also C3.1, U2.CB; no longer C12.1, D4.C, U3.AHB
- net N$13: no longer IC1A.-IN
- net N$14: now also C14.1, IC1A.-IN, OK1A.EMIT, R11.2; no longer IC1B.-IN, IC1B.OUT, R106.1
- net N$16: now also Q3.G, U$3.HVG; no longer U$3.G, U3.AHO
- net N$17: now also Q4.G, U$3.LVG; no longer U$4.G, U3.ALO
- net N$18: now also R_SS2.2, U$3.CSS; no longer U$5.G, U3.BHO
- net N$19: now also C_BOOT.1, U$3.VBOOT; no longer U$6.G, U3.BLO
- net N$2: now also C3.2; no longer C3.1
- net N$20: now also C_DELAY.1, R_DELAY.2, U$3.DELAY; no longer SHUNT.2, U$4.S, U$4.S_2, U$4.S_3, U$6.S, U$6.S_2, U$6.S_3
- net N$21: now also OK1A.A, R105.2; no longer C14.1, D101.A, IC1B.+IN, R104.2
- net N$22: now also OK1A.C, OK1B.A; no longer D101.C, R102.1
- net N$25: now also IC1B.OUT; no longer R8.2
- net N$27: now also IC1B.-IN; no longer IC3B.-IN
- net N$29: now also IC1B.+IN, R5.1; no longer D5.A, IC3A.+IN, IC3B.+IN
- net N$3: now also C19.1, U3.CB; no longer C1.+, D1.C, F1.1, U2.VIN
- net N$30: now also F1.2; no longer D5.C, R5.1
- net N$7: now also CSS.1, R_SS.1, R_SS2.1; no longer C12.2, U$3.S, U$3.S_2, U$3.S_3, U$4.D, U3.AHS
- net N$8: now also RF_MAX.2, RF_MIN.2, R_SS.2, U$3.RFMIN; no longer C11.2, U$5.S, U$5.S_2, U$5.S_3, U$6.D, U3.BHS
- net NOTAUS: now also U$3.DIS; no longer Q2.G

Commit message: changes new rekick
Parts:
- added C26: 100p, rcl:C-EUC0603
- added IC3: 74HCT14D, 74xx-eu:74HCT14D
- added OK3: ILD213, optocoupler:ILD213
- added R12, R13: 12k, rcl:R-EU_R0805
- added R14: 380, rcl:R-EU_R0805
- added R15: 10k, rcl:R-EU_R0805
- added R16: 470k, rcl:R-EU_0207/15
- added U5: MC14025BDG, MC14025BDG:MC14025BDG
- Q2: value SiHB24N65E -> BUZ11BV; device transistor-power:IRG4BC15UD-S -> transistor-power:BUZ11BV
Connections:
- removed net MCU_UIN: IC2A.R0
- removed net U_IN: IC2A.S0
- new net N$37: IC2A.Q2, U5.IN_1A
- new net N$38: IC2A.Q3, U5.IN_1B
- new net N$41: C26.1, OK3A.COL, R15.1
- new net NOTAUS_PRI: OK3A.C, U5.OUTA
- net +5V: now also IC3P.VCC, R14.1, U5.VDD
- net BOOSTER_24V: now also R12.2
- net CAP_0V: now also C26.2, OK3A.EMIT, Q2.S; no longer Q2.E
- net GND: now also IC3P.GND, R13.1, U5.IN_1C, U5.VSS
- net N$24: now also Q2.D; no longer Q2.C
- net N$39: now also R12.1, R13.2; no longer IC2A.S1
- net N$40: now also OK3A.A, R14.2; no longer IC2A.R1

Commit message: update rekick 2015
Parts:
- removed C26: 100p, rcl:C-EUC0603
- removed OK3: ILD213, optocoupler:ILD213
- removed Q2: BUZ11BV, transistor-power:BUZ11BV
- added D5: SMD ZD 15, diode:BZX84CSMD
- added Q6: IRF840, transistor-power:IRF740
- added R17: 380, rcl:R-EU_R0805
- added R18: 10, rcl:R-EU_R0805
- added R19: 47k, rcl:R-EU_R0805
- added T1, T2: BC849, transistor:BC849
- added U$5, U$6: SI8261ABC, Si8261:SI8261ABC
- R15: value 10k -> 10
Connections:
- removed net VON_NOTAUS: Q2.G
- new net KICKER: R19.1
- new net N$42: T2.C, U$6.CATHODE
- new net N$43: R17.1, U$6.ANODE
- new net N$44: R18.1, U$6.VO@1, U$6.VO@2
- new net N$45: D5.C, Q6.G, R16.1, T1.C
- new net N$46: R15.2, T1.B
- new net N$47: R19.2, T2.B
- new net N$48: R18.2
- net +5V: now also R17.2
- net CAP_+12V: now also U$5.VDD, U$6.VDD
- net CAP_0V: now also D5.A, Q6.S, T1.E, U$5.GND, U$6.GND; no longer C26.2, OK3A.EMIT, Q2.S
- net CAP_330V: now also R16.2
- net GND: now also T2.E, U$5.NC@1, U$5.NC@2, U$6.NC@1, U$6.NC@2
- net N$24: now also Q6.D; no longer Q2.D
- net N$40: now also U$5.ANODE; no longer OK3A.A
- net N$41: now also U$5.VO@1, U$5.VO@2; no longer C26.1, OK3A.COL
- net NOTAUS_PRI: now also U$5.CATHODE; no longer OK3A.C

Commit message: changes rekick2015
Parts:
- added C26, C27, C28: 100n, rcl:C-EUC0603
- added COIL_IN, COIL_OUT: WIREPADSMD5-5, mywirepad:WIREPADSMD5-5
- added D12: 5KPXX, diode:5KPXX
- added Q2: IGW60T120, transistor-power:IRFPC40
- added R20: B72220S0321K101, varistor:S20K320
- added RJ_1: RJ10, ownParts:RJ10
- added X1, X2: (no value), con-ptr500:AK500/2-H
- L3, L4: device rcl:L-EUTJ9-U2 -> rcl:L-EULAL03
Connections:
- new net N$49: COIL_IN.P, D12.A, Q2.D, R20.2
- new net N$50: COIL_OUT.P, D12.C
- net +3V3: now also C26.2, C27.1, C27.2
- net +5V: now also C26.1, C28.1
- net BOOSTER_24V: now also X2-2.KL
- net CAN_H: now also RJ_1.P$3
- net CAN_L: now also RJ_1.P$2
- net CAP_0V: now also Q2.S, R20.1
- net GND: now also C28.2, RJ_1.P$4, X1-2.KL
- net GND1: now also X2-1.KL
- net N$30: now also X1-1.KL
- net N$48: now also Q2.G
Other:
- moved on the sheet: D1, F1, IC3C, IC3D, IC3E, IC3F

Commit message: changes rekick2015
Connections:
- net ZU-ADC_OPV renamed ADC_CAP
- removed net KICKER: R19.1
- removed net NOTAUS: U$3.DIS
- removed net ZU-NOTAUS-FF: C24.1, OK2A.EMIT, R10.2
- new net ACTIVATE_BOOSTER: IC3B.I, U$2.PB4
- new net KICK: R19.1, U$2.PB3
- new net N$51: IC3B.O, U5.IN_2B
- new net N$52: IC3A.O, U5.IN_2A
- net N$39: now also IC3A.I
- net NOTAUS_PRI: now also U$3.DIS
- net ÜBERSPANNUNG: now also C24.1, OK2A.EMIT, R10.2
Other:
- moved on the sheet: IC2, IC2P, IC3A, IC3B, IC3P, R12, R13, U5

Commit message: edit rekick2015
Parts:
- removed R103: 12k, rcl:R-EU_R0805
- added C29, C30: 47µF/35V, rcl:CPOL-EUD
- added C31, C32: 1µ, rcl:C-EUC0603
- added C33, C34: 100n, rcl:C-EUC0603
- added C35: 1µ/50V, rcl:C-EUC0603
- added C36, C37, C38, C39: 100p, rcl:C-EUC0603
- added D13: SMD ZD 12, diode:BZX84CSMD
- added D14: BZX84-A5V1, diode:BZX84CSMD
- added IC4: LM1458D, linear:LM1458D
- added Q5: IPD90P04P4L, transistor-power:IRFR5305
- added R200: 47k, rcl:R-EU_R0805
- added R21: 10k, 1%, rcl:R-EU_R0805
- added R22, R24, R25, R26, R27, R28: 10k, rcl:R-EU_R0805
- added R23: (no value), ptc-ntc:NTC644A
- added R29, R30: 1k, rcl:R-EU_R0805
- added S1: (no value), switch-omron:10-XX
- added T3, T4: BC849, transistor:BC849
- added U$7: DSEI30-12A, dsei30-12a:DSEI30-12A
- C10, C9: value 2200µ -> 2200µ/50V; device rcl:CPOL-EUE5-10.5 -> rcl:CPOL-EUE7.5-18
- C18, C2, C21: value 47µF/16V -> 47µF/35V
- D12: value 5KPXX -> BZX84-A5V1; device diode:5KPXX -> diode:BZX84CSMD
- L7: value (none) -> WE-LLCR
- Q3, Q4: value (none) -> IPP023N10N5
- R101: value 1M -> 1M, 1%
- R105: value 10 -> 750
- R11, R8: value 1k -> 2k, 1%
- R12: value 12k -> 70k
- R13: value 12k -> 10k
- R4: value 10k -> 10k, 1%
- R5: value 1M -> 3k, 1%; device rcl:R-EU_0207/15 -> rcl:R-EU_R0805; FARNELL 2396016 -> (none)
- R6: value 12k -> 12k, 1%
- R7: value 20k -> 2.37k, 1%
- R9: value 10k -> 2k
Connections:
- removed net SEK-FEEDBACK: C12.1, RF_MAX.1, U$3.STBY
- new net +5V/3: C39.1, D14.C, OK1B.COL, R27.2, R30.1, R5.2
- new net +5V/4: C16.1, D12.C, OK1A.COL, R29.1, R7.2
- new net N$53: IC4B.OUT, U5.IN_2C
- new net N$54: D13.C, Q5.G, R200.1
- new net N$55: D13.A
- new net N$56: R24.2, T3.B
- new net N$57: C10.+, C35.1, C9.+, Q3.D, Q5.D, R23.2
- new net N$58: R26.1, T4.C, U5.IN_2A
- new net N$59: C37.1, IC4B.+IN, R27.1, R28.2
- new net STBY: C12.1, RF_MAX.1, U$3.STBY, U5.OUTB
- net +12V: now also R30.2; no longer OK1B.COL
- net +5V: now also C34.1, IC4P.V+, R26.2, S1.S, S1.S1; no longer R14.1
- net ACTIVATE_BOOSTER: now also R24.1, R25.1; no longer IC3B.I
- net ADC_CAP: now also IC4A.+IN
- net BOOSTER_24V: now also Q5.S, R200.2, R23.1; no longer C10.+, C9.+, Q3.D
- net CAP_+12V: now also C29.+, C31.1, C32.1, R29.2; no longer OK1A.COL, R7.2
- net CAP_-12V: now also C30.-
- net CAP_0V: now also C29.-, C30.+, C31.2, C32.2, D12.A; no longer R103.1
- net CAP_330V: now also COIL_OUT.P, U$7.C; no longer R5.2
- net GND: now also C33.2, C34.2, C36.2, C37.2, C39.2, D14.A, IC4P.V-, R21.1, R22.1, R28.1, T4.E, U$5.CATHODE; no longer R13.1
- net GND1: now also C35.2, C38.2, R13.1, T3.E
- net N$15: now also IC1B.+IN, R6.2; no longer R103.2
- net N$29: now also C36.1, IC4A.-IN, R21.2; no longer C16.1, IC1B.+IN, R6.2
- net N$39: now also C38.1, IC4B.-IN; no longer IC3A.I
- net N$49: now also U$7.A; no longer D12.A
- net N$50: now also IC4A.OUT; no longer COIL_OUT.P, D12.C
- net N$51: no longer IC3B.O
- net N$52: now also R25.2, T4.B; no longer IC3A.O, U5.IN_2A
- net NOTAUS_PRI: now also R14.1; no longer U$5.CATHODE
- net TASTER: now also C33.1, R22.2, S1.P, S1.P1
Other:
- moved on the sheet: C10, C14, C15, C16, C23, C24, C26, C27, C28, C9, COIL_IN, COIL_OUT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
