File: msl_electronic_boards/rekick2015/pcb/rekick2015-001.sch (EAGLE design)
At the start: 145 parts, among them IC1 LM1458D, IC2 4043D, IC3 74HCT14D, IC4 LM1458D, Q1 16MHz, Q2 IGW60T120, Q3 IPP023N10N5, Q4 IPP023N10N5, Q5 IPD90P04P4L, Q6 IRF840, T1 BC849, T2 BC849, T3 BC849, T4 BC849, U1 TXB0108PWR, U2 LM2675, U3 LM2675, U4 LM2675, U5 MC14025BDG

Commit message: edit rekick2015
Parts:
- removed C3: 10nF/50V, rcl:C-EUC0603
- removed L1: 68µH, Inductor-Fastron:L-EUPISM
- removed L2: 10µH, rcl:L-EUL2012C
- removed U2: LM2675, LM2675M-3.3:LM2675M-3.3
- added CAP_0V, CAP_330V: WIREPADSMD5-5, mywirepad:WIREPADSMD5-5
- added H1, H2, H3, H4: MOUNT-PAD-ROUND3.0, holes:MOUNT-PAD-ROUND3.0
- added R31: 20k, rcl:R-EU_R0805
- added R32: 120, rcl:R-EU_R0805
- added RJ_2: RJ10, ownParts:RJ10
- added SJ1: (no value), jumper:SJ
- C13: device rcl:C-EUC1206 -> rcl:C-EUC2220K
- C16, C39: value 100p -> 100n
- IC3: value 74HCT14D -> LM1117; device 74xx-eu:74HCT14D -> v-reg:LM317MBSTT3
- L3, L4: device rcl:L-EULAL03 -> EagleLibrary_Wuerth_Elektronik_eiSos_rev16a:WE-HCI_1890
- R101: device rcl:R-EU_0207/15 -> rcl:R-EU_0207/10
- R12: value 70k -> 68k
Connections:
- removed net ADC8: U$2.PC4
- removed net D2A: U$2.PC7
- removed net N$12: C3.1, U2.CB
- removed net N$2: C3.2, D2.C, L1.2, U2.VSW
- new net RF: RF_MAX.1, U$2.PC7
- net +24V: no longer C1.+, U2.VIN
- net +3V3: now also D2.A, IC3.OUT; no longer L1.1, U2.FB
- net +5V: now also C1.+, D2.C, IC3.IN; no longer IC3P.VCC, L2.1
- net +5V/3: now also C7.2, U$2.AVCC
- net ACTIVATE_BOOSTER: now also R31.2
- net ADC_CAP: now also U$2.PC4
- net CAN_H: now also RJ_2.P$3, SJ1.2
- net CAN_L: now also R32.2, RJ_2.P$2
- net CAP_0V: now also CAP_0V.P
- net CAP_330V: now also CAP_330V.P
- net GND: now also H1.MOUNT, H2.MOUNT, H3.MOUNT, H4.MOUNT, IC3.ADJ, R31.1; no longer D2.A, IC3P.GND, U2.GND
- net N$9: now also R32.1, SJ1.1; no longer C7.2, L2.2, U$2.AVCC
- net STBY: no longer RF_MAX.1
Other:
- moved on the sheet: C1, C12, C14, C15, C16, C2, C23, C24, C29, C30, C7, C_ISEN_A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

Commit message: edit rekick2015
Parts:
- L7: device EagleLibrary_Wuerth_Elektronik_eiSos_rev15h:WE-LLCR_760895641 -> EagleLibrary_Wuerth_Elektronik_eiSos_rev15h:WE-LLCR_ETD34
- R2, R3: value 47 -> 100; device resistor-power:RHS50 -> resistor-power:RHS25
Connections:
- net N$55: now also T3.C
- net TRAFO1: now also L7.4; no longer L7.3
- net TRAFO2: now also L7.5; no longer L7.2
Changed lines of the file:
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@@
 <?xml version="1.0" encoding="utf-8"?>
 <!DOCTYPE eagle SYSTEM "eagle.dtd">
-<eagle version="7.5.0">
+<eagle version="7.2.0">
 <drawing>
 <settings>
@@
 <part name="R105" library="rcl" deviceset="R-EU_" device="R0805" value="750"/>
 <part name="FRAME6" library="frames" deviceset="A4L-LOC" device=""/>
-<part name="R2" library="resistor-power" deviceset="R" device="HS50" value="47"/>
-<part name="R3" library="resistor-power" deviceset="R" device="HS50" value="47"/>
+<part name="R2" library="resistor-power" deviceset="R" device="HS25" value="100"/>
+<part name="R3" library="resistor-power" deviceset="R" device="HS25" value="100"/>
 <part name="C15" library="rcl" deviceset="C-EU" device="C0603" value="100p"/>
 <part name="R6" library="rcl" deviceset="R-EU_" device="R0805" value="12k, 1%"/>
@@
 <part name="R_LINE" library="rcl" deviceset="R-EU_" device="R0805" value="10k"/>
 <part name="P+18" library="supply1" deviceset="+5V" device=""/>
-<part name="L7" library="EagleLibrary_Wuerth_Elektronik_eiSos_rev15h" deviceset="WE-LLCR" device="_760895641" value="WE-LLCR"/>
+<part name="L7" library="EagleLibrary_Wuerth_Elektronik_eiSos_rev15h" deviceset="WE-LLCR" device="_ETD34" value="WE-LLCR"/>
 <part name="IC1" library="linear" deviceset="*1458" device="D" technology="LM"/>
 <part name="SUPPLY13" library="supply2" deviceset="-12V" device="" value="CAP_-12V"/>
@@
 <junction x="134.62" y="121.92"/>
 <wire x1="154.94" y1="121.92" x2="167.64" y2="121.92" width="0.1524" layer="91"/>
-<wire x1="167.64" y1="121.92" x2="180.34" y2="121.92" width="0.1524" layer="91"/>
+<wire x1="167.64" y1="121.92" x2="175.26" y2="121.92" width="0.1524" layer="91"/>
+<wire x1="175.26" y1="121.92" x2="175.26" y2="116.84" width="0.1524" layer="91"/>
 <wire x1="167.64" y1="121.92" x2="167.64" y2="119.38" width="0.1524" layer="91"/>
 <junction x="167.64" y="121.92"/>
 <pinref part="L3" gate="G$1" pin="1"/>
-<wire x1="180.34" y1="121.92" x2="180.34" y2="111.76" width="0.1524" layer="91"/>
-<pinref part="L7" gate="G$1" pin="3"/>
-<wire x1="180.34" y1="111.76" x2="185.42" y2="111.76" width="0.1524" layer="91"/>
+<pinref part="L7" gate="G$1" pin="4"/>
+<wire x1="175.26" y1="116.84" x2="185.42" y2="116.84" width="0.1524" layer="91"/>
 </segment>
 </net>
@@
 <junction x="175.26" y="99.06"/>
 <pinref part="L4" gate="G$1" pin="1"/>
-<pinref part="L7" gate="G$1" pin="2"/>
-<wire x1="185.42" y1="106.68" x2="180.34" y2="106.68" width="0.1524" layer="91"/>
-<wire x1="180.34" y1="106.68" x2="180.34" y2="99.06" width="0.1524" layer="91"/>
+<wire x1="180.34" y1="121.92" x2="180.34" y2="99.06" width="0.1524" layer="91"/>
+<pinref part="L7" gate="G$1" pin="5"/>
+<wire x1="180.34" y1="121.92" x2="185.42" y2="121.92" width="0.1524" layer="91"/>
 </segment>
 </net>
@@
 <pinref part="D13" gate="G$1" pin="A"/>
 <wire x1="190.5" y1="165.1" x2="182.88" y2="165.1" width="0.1524" layer="91"/>
-</segment>
-</net>
+<pinref part="T3" gate="G$1" pin="C"/>
+</segment>
+</net>

Commit message: rekick2015
Parts:
- added VR1, VR2, VR3, VR4: TL431_SOT23, 1_USER:TL431_SOT23
Other:
- moved on the sheet: C16, C29, C30, D12, R29
Changed lines of the file:
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@@
 <layer number="131" name="tAdjust" color="15" fill="1" visible="no" active="no"/>
 <layer number="132" name="bAdjust" color="5" fill="1" visible="no" active="no"/>
+<layer number="200" name="200bmp" color="1" fill="10" visible="no" active="no"/>
 <layer number="250" name="Descript" color="3" fill="1" visible="no" active="no"/>
 <layer number="251" name="SMDround" color="12" fill="11" visible="no" active="no"/>
@@
 <part name="IC3" library="v-reg" deviceset="LM317?*" device="MBSTT3" value="LM1117"/>
 <part name="P+12" library="supply1" deviceset="+5V" device=""/>
+<part name="SUPPLY27" library="supply2" deviceset="+12V" device="" value="CAP_+12V"/>
+<part name="VR1" library="1_USER" deviceset="TL431" device="_SOT23"/>
+<part name="VR2" library="1_USER" deviceset="TL431" device="_SOT23"/>
+<part name="VR3" library="1_USER" deviceset="TL431" device="_SOT23"/>
+<part name="VR4" library="1_USER" deviceset="TL431" device="_SOT23"/>
 </parts>
 <sheets>
@@
 <instance part="GND9" gate="1" x="208.28" y="96.52"/>
 <instance part="SUPPLY10" gate="0V" x="129.54" y="58.42"/>
-<instance part="SUPPLY11" gate="+12V" x="20.32" y="88.9"/>
+<instance part="SUPPLY11" gate="+12V" x="15.24" y="121.92"/>
 <instance part="R9" gate="G$1" x="177.8" y="81.28"/>
 <instance part="OK2" gate="A" x="198.12" y="78.74"/>
 <instance part="OK2" gate="B" x="198.12" y="45.72"/>
-<instance part="U$4" gate="G$1" x="38.1" y="129.54"/>
-<instance part="P+9" gate="1" x="17.78" y="142.24"/>
-<instance part="GND8" gate="1" x="17.78" y="116.84"/>
-<instance part="SUPPLY2" gate="0V" x="81.28" y="129.54" rot="R90"/>
-<instance part="SUPPLY4" gate="G$1" x="60.96" y="121.92"/>
-<instance part="SUPPLY5" gate="+12V" x="60.96" y="137.16"/>
+<instance part="U$4" gate="G$1" x="33.02" y="149.86"/>
+<instance part="P+9" gate="1" x="12.7" y="162.56"/>
+<instance part="GND8" gate="1" x="12.7" y="137.16"/>
+<instance part="SUPPLY2" gate="0V" x="76.2" y="149.86" rot="R90"/>
+<instance part="SUPPLY4" gate="G$1" x="55.88" y="142.24"/>
+<instance part="SUPPLY5" gate="+12V" x="55.88" y="157.48"/>
 <instance part="R10" gate="G$1" x="208.28" y="68.58" rot="R90"/>
 <instance part="GND10" gate="1" x="208.28" y="58.42"/>
@@
 <instance part="SUPPLY14" gate="+12V" x="157.48" y="162.56"/>
 <instance part="P+19" gate="1" x="208.28" y="88.9"/>
-<instance part="C16" gate="G$1" x="27.94" y="58.42"/>
-<instance part="C29" gate="G$1" x="68.58" y="134.62"/>
-<instance part="C30" gate="G$1" x="68.58" y="127"/>
-<instance part="D12" gate="G$1" x="20.32" y="58.42" rot="R90"/>
-<instance part="R29" gate="G$1" x="20.32" y="78.74" rot="R90"/>
-<instance part="SUPPLY19" gate="0V" x="20.32" y="50.8"/>
-<instance part="SUPPLY20" gate="G$1" x="27.94" y="68.58"/>
+<instance part="C16" gate="G$1" x="22.86" y="91.44"/>
+<instance part="C29" gate="G$1" x="63.5" y="154.94"/>
+<instance part="C30" gate="G$1" x="63.5" y="147.32"/>
+<instance part="D12" gate="G$1" x="15.24" y="91.44" rot="R90"/>
+<instance part="R29" gate="G$1" x="15.24" y="111.76" rot="R90"/>
+<instance part="SUPPLY19" gate="0V" x="15.24" y="83.82"/>
+<instance part="SUPPLY20" gate="G$1" x="22.86" y="101.6"/>
 <instance part="SUPPLY21" gate="G$1" x="144.78" y="101.6"/>
 <instance part="SUPPLY22" gate="G$1" x="208.28" y="157.48"/>
 <instance part="SUPPLY7" gate="G$1" x="208.28" y="124.46"/>
+<instance part="SUPPLY27" gate="+12V" x="10.16" y="40.64"/>
+<instance part="VR1" gate="G$1" x="40.64" y="12.7" rot="R90"/>
+<instance part="VR2" gate="G$1" x="58.42" y="12.7" rot="R90"/>
+<instance part="VR3" gate="G$1" x="76.2" y="12.7" rot="R90"/>
+<instance part="VR4" gate="G$1" x="93.98" y="12.7" rot="R90"/>
 </instances>
 <busses>
@@
 <pinref part="R101" gate="G$1" pin="2"/>
 <wire x1="109.22" y1="154.94" x2="116.84" y2="154.94" width="0.1524" layer="91"/>
+</segment>
+<segment>
+<label x="27.94" y="50.8" size="1.778" layer="95" rot="R180" xref="yes"/>
+<wire x1="27.94" y1="50.8" x2="78.74" y2="50.8" width="0.1524" layer="91"/>
 </segment>
 </net>
@@
 <segment>
 <pinref part="GND8" gate="1" pin="GND"/>
-<wire x1="17.78" y1="119.38" x2="17.78" y2="124.46" width="0.1524" layer="91"/>
+<wire x1="12.7" y1="139.7" x2="12.7" y2="144.78" width="0.1524" layer="91"/>
 <pinref part="U$4" gate="G$1" pin="GND"/>
-<wire x1="17.78" y1="124.46" x2="22.86" y2="124.46" width="0.1524" layer="91"/>
+<wire x1="12.7" y1="144.78" x2="17.78" y2="144.78" width="0.1524" layer="91"/>
 </segment>
 <segment>
@@
 <pinref part="U$4" gate="G$1" pin="0V"/>
 <pinref part="SUPPLY2" gate="0V" pin="0V"/>
-<wire x1="53.34" y1="129.54" x2="68.58" y2="129.54" width="0.1524" layer="91"/>
+<wire x1="48.26" y1="149.86" x2="63.5" y2="149.86" width="0.1524" layer="91"/>
 <pinref part="C29" gate="G$1" pin="-"/>
-<wire x1="68.58" y1="129.54" x2="78.74" y2="129.54" width="0.1524" layer="91"/>
-<junction x="68.58" y="129.54"/>
+<wire x1="63.5" y1="149.86" x2="73.66" y2="149.86" width="0.1524" layer="91"/>
+<junction x="63.5" y="149.86"/>
 <pinref part="C30" gate="G$1" pin="+"/>
 </segment>
 <segment>
 <pinref part="SUPPLY19" gate="0V" pin="0V"/>
-<wire x1="20.32" y1="55.88" x2="20.32" y2="53.34" width="0.1524" layer="91"/>
+<wire x1="15.24" y1="88.9" x2="15.24" y2="86.36" width="0.1524" layer="91"/>
 <pinref part="D12" gate="G$1" pin="A"/>
 <pinref part="C16" gate="G$1" pin="2"/>
-<wire x1="20.32" y1="53.34" x2="27.94" y2="53.34" width="0.1524" layer="91"/>
-<junction x="20.32" y="53.34"/>
+<wire x1="15.24" y1="86.36" x2="22.86" y2="86.36" width="0.1524" layer="91"/>
+<junction x="15.24" y="86.36"/>
 </segment>
 </net>
@@
 <segment>
 <pinref part="SUPPLY11" gate="+12V" pin="+12V"/>
-<wire x1="20.32" y1="83.82" x2="20.32" y2="86.36" width="0.1524" layer="91"/>
+<wire x1="15.24" y1="116.84" x2="15.24" y2="119.38" width="0.1524" layer="91"/>
 <pinref part="R29" gate="G$1" pin="2"/>
 </segment>
@@
 <pinref part="U$4" gate="G$1" pin="+U_OUT"/>
 <pinref part="SUPPLY5" gate="+12V" pin="+12V"/>
-<wire x1="53.34" y1="134.62" x2="60.96" y2="134.62" width="0.1524" layer="91"/>
-<wire x1="60.96" y1="134.62" x2="63.5" y2="134.62" width="0.1524" layer="91"/>
-<wire x1="63.5" y1="134.62" x2="63.5" y2="137.16" width="0.1524" layer="91"/>
-<junction x="60.96" y="134.62"/>
-<wire x1="63.5" y1="137.16" x2="68.58" y2="137.16" width="0.1524" layer="91"/>
+<wire x1="48.26" y1="154.94" x2="55.88" y2="154.94" width="0.1524" layer="91"/>
+<wire x1="55.88" y1="154.94" x2="58.42" y2="154.94" width="0.1524" layer="91"/>
+<wire x1="58.42" y1="154.94" x2="58.42" y2="157.48" width="0.1524" layer="91"/>
+<junction x="55.88" y="154.94"/>
+<wire x1="58.42" y1="157.48" x2="63.5" y2="157.48" width="0.1524" layer="91"/>
 <pinref part="C29" gate="G$1" pin="+"/>
 </segment>
@@
 <pinref part="SUPPLY14" gate="+12V" pin="+12V"/>
 <pinref part="IC1" gate="P" pin="V+"/>
+</segment>
+<segment>
+<wire x1="10.16" y1="35.56" x2="10.16" y2="38.1" width="0.1524" layer="91"/>
+<pinref part="SUPPLY27" gate="+12V" pin="+12V"/>
+<wire x1="10.16" y1="35.56" x2="91.44" y2="35.56" width="0.1524" layer="91"/>
 </segment>
 </net>
@@
 <segment>
 <pinref part="P+9" gate="1" pin="+24V"/>
-<wire x1="17.78" y1="139.7" x2="17.78" y2="134.62" width="0.1524" layer="91"/>
+<wire x1="12.7" y1="160.02" x2="12.7" y2="154.94" width="0.1524" layer="91"/>
 <pinref part="U$4" gate="G$1" pin="U_IN"/>
-<wire x1="17.78" y1="134.62" x2="22.86" y2="134.62" width="0.1524" layer="91"/>
+<wire x1="12.7" y1="154.94" x2="17.78" y2="154.94" width="0.1524" layer="91"/>
 </segment>
 </net>
@@
 <pinref part="U$4" gate="G$1" pin="-U_OUT"/>
 <pinref part="SUPPLY4" gate="G$1" pin="-12V"/>
-<wire x1="53.34" y1="124.46" x2="60.96" y2="124.46" width="0.1524" layer="91"/>
-<wire x1="60.96" y1="124.46" x2="63.5" y2="124.46" width="0.1524" layer="91"/>
-<wire x1="63.5" y1="124.46" x2="63.5" y2="121.92" width="0.1524" layer="91"/>
-<junction x="60.96" y="124.46"/>
-<wire x1="63.5" y1="121.92" x2="68.58" y2="121.92" width="0.1524" layer="91"/>
+<wire x1="48.26" y1="144.78" x2="55.88" y2="144.78" width="0.1524" layer="91"/>
+<wire x1="55.88" y1="144.78" x2="58.42" y2="144.78" width="0.1524" layer="91"/>
+<wire x1="58.42" y1="144.78" x2="58.42" y2="142.24" width="0.1524" layer="91"/>
+<junction x="55.88" y="144.78"/>
+<wire x1="58.42" y1="142.24" x2="63.5" y2="142.24" width="0.1524" layer="91"/>
 <pinref part="C30" gate="G$1" pin="-"/>
 </segment>
@@
 <pinref part="R29" gate="G$1" pin="1"/>
 <pinref part="D12" gate="G$1" pin="C"/>
-<wire x1="20.32" y1="60.96" x2="20.32" y2="63.5" width="0.1524" layer="91"/>
-<wire x1="20.32" y1="63.5" x2="20.32" y2="73.66" width="0.1524" layer="91"/>
-<wire x1="20.32" y1="63.5" x2="27.94" y2="63.5" width="0.1524" layer="91"/>
-<wire x1="27.94" y1="63.5" x2="27.94" y2="66.04" width="0.1524" layer="91"/>
-<junction x="20.32" y="63.5"/>
+<wire x1="15.24" y1="93.98" x2="15.24" y2="96.52" width="0.1524" layer="91"/>
+<wire x1="15.24" y1="96.52" x2="15.24" y2="106.68" width="0.1524" layer="91"/>
+<wire x1="15.24" y1="96.52" x2="22.86" y2="96.52" width="0.1524" layer="91"/>
+<wire x1="22.86" y1="96.52" x2="22.86" y2="99.06" width="0.1524" layer="91"/>
+<junction x="15.24" y="96.52"/>
 <pinref part="C16" gate="G$1" pin="1"/>
-<wire x1="27.94" y1="60.96" x2="27.94" y2="63.5" width="0.1524" layer="91"/>
-<junction x="27.94" y="63.5"/>
+<wire x1="22.86" y1="93.98" x2="22.86" y2="96.52" width="0.1524" layer="91"/>
+<junction x="22.86" y="96.52"/>
 <pinref part="SUPPLY20" gate="G$1" pin="+5V/4"/>
 </segment>

Commit message: rekick 2015
Parts:
- added R33, R34, R35: 1M, rcl:R-EU_R2512
- added R36: 50k, rcl:R-EU_R0805
- added R37: 17k, rcl:R-EU_R0805
- added R38: 7.68k, rcl:R-EU_R0805
- R101: device rcl:R-EU_0207/10 -> rcl:R-EU_R2512
Changed lines of the file:
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@@
 <?xml version="1.0" encoding="utf-8"?>
 <!DOCTYPE eagle SYSTEM "eagle.dtd">
-<eagle version="7.2.0">
+<eagle version="7.5.0">
 <drawing>
 <settings>
@@
 <part name="SUPPLY3" library="supply2" deviceset="GND1" device=""/>
 <part name="FRAME5" library="frames" deviceset="A4L-LOC" device=""/>
-<part name="R101" library="rcl" deviceset="R-EU_" device="0207/10" value="1M, 1%">
+<part name="R101" library="rcl" deviceset="R-EU_" device="R2512" value="1M, 1%">
 <attribute name="FARNELL" value="2396016"/>
 </part>
@@
 <part name="VR3" library="1_USER" deviceset="TL431" device="_SOT23"/>
 <part name="VR4" library="1_USER" deviceset="TL431" device="_SOT23"/>
+<part name="R33" library="rcl" deviceset="R-EU_" device="R2512" value="1M"/>
+<part name="R34" library="rcl" deviceset="R-EU_" device="R2512" value="1M"/>
+<part name="R35" library="rcl" deviceset="R-EU_" device="R2512" value="1M"/>
+<part name="R36" library="rcl" deviceset="R-EU_" device="R0805" value="50k"/>
+<part name="R37" library="rcl" deviceset="R-EU_" device="R0805" value="17k"/>
+<part name="R38" library="rcl" deviceset="R-EU_" device="R0805" value="7.68k"/>
 </parts>
 <sheets>
@@
 <instance part="VR3" gate="G$1" x="76.2" y="12.7" rot="R90"/>
 <instance part="VR4" gate="G$1" x="93.98" y="12.7" rot="R90"/>
+<instance part="R33" gate="G$1" x="30.48" y="43.18" rot="R90"/>
+<instance part="R34" gate="G$1" x="50.8" y="43.18" rot="R90"/>
+<instance part="R35" gate="G$1" x="68.58" y="43.18" rot="R90"/>
+<instance part="R36" gate="G$1" x="30.48" y="12.7" rot="R90"/>
+<instance part="R37" gate="G$1" x="50.8" y="12.7" rot="R90"/>
+<instance part="R38" gate="G$1" x="68.58" y="12.7" rot="R90"/>
 </instances>
 <busses>

Commit message: rekick 2015
Parts:
- removed VR4: TL431_SOT23, 1_USER:TL431_SOT23
- added JP3: (no value), pinhead:PINHD-1X3
- added LED1, LED2, LED3: (no value), led:LEDCHIP-LED0805
- added R39, R40, R41: 50k, rcl:R-EU_R0805
Connections:
- removed net CS/OC1B: U$2.PC1
- removed net INT2: U$2.PB5
- new net +5V/1: JP3.2
- new net N$12: R33.1, R36.2, VR1.R
- new net N$2: LED1.C, VR1.C
- new net N$60: R34.1, R37.2, VR2.R
- new net N$61: R35.1, R38.2, VR3.R
- new net N$62: LED2.C, VR2.C
- new net N$63: LED3.C, VR3.C
- new net RESET_NOTAUS: IC2A.R2, IC2A.R3, U$2.PB5
- new net SERVO_PWM: JP3.1, U$2.PC1
- net CAP_0V: now also R36.1, R37.1, R38.1, VR1.A, VR2.A, VR3.A
- net CAP_330V: now also R33.2, R34.2, R35.2
- net GND: now also JP3.3, U$3.DIS; no longer IC2A.R2, IC2A.R3
- net NOTAUS_PRI: no longer U$3.DIS
Other:
- moved on the sheet: R33, R34, R35, R36, R37, R38, VR1, VR2, VR3

Commit message: rekick 2015
Parts:
- added C3, C40: 47µF/35V, rcl:CPOL-EUD
- added D15, D16, D17: ES1A, diode:GF1
- added L1: 68µH, Inductor-Fastron:L-EUPISM
- added LED10, LED4, LED5, LED6, LED7, LED8, LED9: (no value), led:LEDCHIP-LED0805
- added R42, R46: 680, rcl:R-EU_R0805
- added R43, R45: 1,5k, rcl:R-EU_R0805
- added R44, R49, R50: 4.7k, rcl:R-EU_R0805
- added R47: 1k, rcl:R-EU_R0805
- added R48: 10k, rcl:R-EU_R0805
- added T5: (no value), zetex:NMOSSOT23
- added U$8: LM2576, LM2576:LM2576
- C25: value 2200µ -> 2.2µ
- L3: device EagleLibrary_Wuerth_Elektronik_eiSos_rev16a:WE-HCI_1890 -> inductor-bourns:SRR1210
- R101: FARNELL 2396016 -> (none)
- R39, R40, R41: value 50k -> 4.7k
Connections:
- removed net INT1: U$2.PB2
- removed net NOTAUS_PRI: R14.1, U5.OUTA
- new net ACTIVATE_SERVO: R47.1, U$2.PB2
- new net BURST: D17.C, U5.OUTB
- new net N$64: LED1.A, R39.1
- new net N$65: LED2.A, R40.1
- new net N$66: LED3.A, R41.1
- new net N$67: LED4.A, R42.1
- new net N$68: C40.+, L1.1, R45.2, U$8.FB
- new net N$69: D15.C, L1.2, U$8.VOUT
- new net N$70: JP3.3, T5.D
- new net N$71: LED7.A, R45.1
- new net N$72: LED5.A, R43.1
- new net N$73: LED6.A, R44.1
- new net N$74: LED8.A, R46.1
- new net N$75: R47.2, T5.G
- new net N$76: LED9.A, R49.1
- new net N$77: LED10.A, R50.1
- new net NOTAUS: D16.C, R14.1, U5.OUTA
- net +12V: now also R44.2
- net +24V: now also C3.+, U$8.VIN
- net +3V3: now also R42.2
- net +5V: now also R43.2, R48.2
- net BOOSTER_24V: now also R46.2
- net CAP_+12V: now also R39.2, R40.2, R41.2, R49.2
- net CAP_-12V: now also LED10.C
- net CAP_0V: now also LED9.C, R50.2
- net GND: now also C3.-, C40.-, D15.A, LED4.C, LED5.C, LED6.C, LED7.C, T5.S, U$8.!ON!/OFF, U$8.GND, U5.IN_3A, U5.IN_3B, U5.IN_3C; no longer JP3.3
- net GND1: now also LED8.C
- net STBY: now also D16.A, D17.A, R48.1; no longer U5.OUTB
Other:
- moved on the sheet: D1, F1, H1, H2, H3, H4, R20, X1-1, X1-2

Commit message: rekick 2015
Connections:
- removed net N$29: C36.1, IC4A.-IN, R21.2, R5.1
- removed net RF: RF_MAX.1, U$2.PC7
- new net AN-AUSGANG-ODER-MCU-KOPPELN: RF_MAX.1
- new net D2A/KICK_VOLTAGE: C36.1, IC4A.-IN, R21.2, R5.1, U$2.PC7
Changed lines of the file:
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@@
 <?xml version="1.0" encoding="utf-8"?>
 <!DOCTYPE eagle SYSTEM "eagle.dtd">
-<eagle version="7.5.0">
+<eagle version="7.2.0">
 <drawing>
 <settings>
@@
 </segment>
 </net>
-<net name="RF" class="0">
+<net name="D2A/KICK_VOLTAGE" class="0">
 <segment>
 <pinref part="U$2" gate="G$1" pin="PC7"/>
@@
 </segment>
 </net>
-<net name="RF" class="0">
-<segment>
-<pinref part="RF_MAX" gate="G$1" pin="1"/>
-<wire x1="25.4" y1="99.06" x2="25.4" y2="104.14" width="0.1524" layer="91"/>
-<label x="25.4" y="99.06" size="1.778" layer="95" rot="R270" xref="yes"/>
-</segment>
-</net>
 <net name="N$74" class="0">
 <segment>
@@
 </segment>
 </net>
+<net name="AN-AUSGANG-ODER-MCU-KOPPELN" class="0">
+<segment>
+<pinref part="RF_MAX" gate="G$1" pin="1"/>
+<wire x1="25.4" y1="104.14" x2="25.4" y2="96.52" width="0.1524" layer="91"/>
+<label x="25.4" y="96.52" size="1.778" layer="95" rot="R270" xref="yes"/>
+</segment>
+</net>
 </nets>
 </sheet>
@@
 </segment>
 </net>
-<net name="N$29" class="0">
+<net name="D2A/KICK_VOLTAGE" class="0">
 <segment>
 <pinref part="R21" gate="G$1" pin="2"/>
@@
 <wire x1="96.52" y1="71.12" x2="88.9" y2="71.12" width="0.1524" layer="91"/>
 <junction x="96.52" y="71.12"/>
+<wire x1="88.9" y1="71.12" x2="78.74" y2="71.12" width="0.1524" layer="91"/>
+<label x="78.74" y="71.12" size="1.778" layer="95" rot="R180" xref="yes"/>
 </segment>
 </net>

Commit message: rekick 2015
Connections:
- removed net ADC2: U$2.PD5
- removed net AN-AUSGANG-ODER-MCU-KOPPELN: RF_MAX.1
- removed net N$51: U5.IN_2B
- removed net ZU_CR_LR-KNOTEN: C13.1, C_ISEN_A.2, L4.2
- new net N$29: L3.1, L4.1, L7.4
- new net RF_MAX: RF_MAX.1, U$2.PD5
- net GND: now also IC2A.R0, IC2A.R1, IC2A.S0, IC2A.S1
- net N$50: now also U5.IN_2B
- net TRAFO1: now also L4.2; no longer L3.1, L7.4
- net TRAFO2: now also C13.1, C_ISEN_A.2; no longer L4.1
Other:
- moved on the sheet: L3, L4
