File: msl_electronic_boards/rekick2015/pcb/rekick2015-001.sch (EAGLE design)
At the start: 191 parts, among them IC1 LM1458D, IC2 4043D, IC3 LM1117, IC4 LM1458D, Q1 16MHz, Q2 IGW60T120, Q3 IPP023N10N5, Q4 IPP023N10N5, Q5 IPD90P04P4L, Q6 IRF840, T1 BC849, T2 BC849, T3 BC849, T4 BC849, U1 TXB0108PWR, U3 LM2675, U4 LM2675, U5 MC14025BDG

Commit message: rekick 2015
Parts:
- added C41: 2.2µ / 100V, rcl:C-EUC1210K
- added C42: 47µF/35V, rcl:CPOL-EUD
- added R51: 12k, rcl:R-EU_R0805
- C10, C9: device rcl:CPOL-EUE7.5-18 -> rcl:CPOL-EUE5-13
- C13: value 2.2µ -> 2.2µ / 250V
- C25: device rcl:CPOL-EUE10-20 -> rcl:CPOL-EUE5-10.5
- R19: value 47k -> 3k
Connections:
- net +24V: now also C42.+
- net GND: now also C42.-, R51.1; no longer H1.MOUNT, H2.MOUNT, H3.MOUNT, H4.MOUNT
- net GND1: now also C41.2
- net N$47: now also R51.2
- net TRAFO2: now also C41.1

Commit message: rekick 2015
Parts:
- added C43, C44, C45: 100n, rcl:C-EUC0603
- added R52: 10k, rcl:R-EU_R0805
- added R53, R54: 100k, rcl:R-EU_R0805
- C1, C2: device rcl:CPOL-EUD -> rcl:C-EUC0603
- IC3: device v-reg:LM317MBSTT3 -> LM1117:LM1117
Connections:
- removed net ADC10: U$2.PC6
- removed net ADC3/INT0: U$2.PD6
- removed net ADC9: U$2.PC5
- removed net D2A/KICK_VOLTAGE: C36.1, IC4A.-IN, R21.2, R5.1, U$2.PC7
- removed net N$68: C40.+, L1.1, R45.2, U$8.FB
- removed net RF_MAX: RF_MAX.1, U$2.PD5
- new net D2A/RF_MAX: RF_MAX.1, U$2.PC7
- new net KICK_VOLTAGE: C36.1, IC4A.-IN, R21.2, R5.1, R52.2
- new net OC0A/MOSI_A/KICK_VOLTAGE: R52.1, U$2.(MOSI_A/TXD)PD3
- net +3V3: now also C2.1, IC3.OUT@1, IC3.OUT@2; no longer C2.+, C26.2, C27.2, IC3.OUT
- net +5V: now also C1.1, C44.1, C45.1; no longer C1.+
- net +5V/1: now also C40.+, L1.1, R45.2, U$8.FB
- net BURST: now also U$2.PD6
- net CAP_+12V: now also C43.1
- net CAP_-12V: now also C43.2
- net GND: now also C1.2, C2.2, C26.2, C27.2, C44.2, C45.2, IC3.GND; no longer C1.-, C2.-, IC3.ADJ
- net GND1: now also R54.2
- net N$16: now also R53.1
- net N$17: now also R54.1
- net NOTAUS: now also U$2.PD7
- net OC0A/MOSI_A: no longer U$2.(MOSI_A/TXD)PD3
- net STBY: now also U$2.PD5
- net TRAFO1: now also R53.2

Commit message: rekick 2015
Connections:
- new net FREI: U$2.PB2
- new net FREI2: U$2.PB6
- new net FREI3: U$2.PD7
- net ACTIVATE_BOOSTER: now also U$2.PB5; no longer U$2.PB4
- net ACTIVATE_SERVO: now also U$2.PD5; no longer U$2.PB2
- net ADC_CAP: now also U$2.PD6; no longer U$2.PC4
- net BURST: now also U$2.PC5; no longer U$2.PD6
- net NOTAUS: now also U$2.PC6; no longer U$2.PD7
- net RESET_NOTAUS: now also U$2.PB4; no longer U$2.PB5
- net STBY: now also U$2.PC4; no longer U$2.PD5
Changed lines of the file:
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@@
 <net name="ADC_CAP" class="0">
 <segment>
-<pinref part="U$2" gate="G$1" pin="PC4"/>
-<wire x1="124.46" y1="116.84" x2="129.54" y2="116.84" width="0.1524" layer="91"/>
-<label x="129.54" y="116.84" size="1.27" layer="95" xref="yes"/>
+<pinref part="U$2" gate="G$1" pin="PD6"/>
+<wire x1="124.46" y1="99.06" x2="129.54" y2="99.06" width="0.1524" layer="91"/>
+<label x="129.54" y="99.06" size="1.27" layer="95" xref="yes"/>
 </segment>
 </net>
@@
 <net name="RESET_NOTAUS" class="0">
 <segment>
-<pinref part="U$2" gate="G$1" pin="PB5"/>
-<wire x1="129.54" y1="142.24" x2="124.46" y2="142.24" width="0.1524" layer="91"/>
-<label x="129.54" y="142.24" size="1.27" layer="95" xref="yes"/>
-</segment>
-</net>
-<net name="ACTIVATE_SERVO" class="0">
-<segment>
-<pinref part="U$2" gate="G$1" pin="PB2"/>
-<wire x1="129.54" y1="134.62" x2="124.46" y2="134.62" width="0.1524" layer="91"/>
-<label x="129.54" y="134.62" size="1.27" layer="95" xref="yes"/>
+<label x="129.54" y="139.7" size="1.27" layer="95" xref="yes"/>
+<pinref part="U$2" gate="G$1" pin="PB4"/>
+<wire x1="124.46" y1="139.7" x2="129.54" y2="139.7" width="0.1524" layer="91"/>
 </segment>
 </net>
@@
 <wire x1="215.9" y1="147.32" x2="210.82" y2="147.32" width="0.1524" layer="91"/>
 <label x="210.82" y="147.32" size="1.27" layer="95" rot="R180" xref="yes"/>
-</segment>
-</net>
-<net name="ACTIVATE_BOOSTER" class="0">
-<segment>
-<label x="129.54" y="139.7" size="1.27" layer="95" xref="yes"/>
-<pinref part="U$2" gate="G$1" pin="PB4"/>
-<wire x1="124.46" y1="139.7" x2="129.54" y2="139.7" width="0.1524" layer="91"/>
 </segment>
 </net>
@@
 </segment>
 </net>
-<net name="BURST" class="0">
+<net name="FREI" class="0">
 <segment>
-<pinref part="U$2" gate="G$1" pin="PD6"/>
-<wire x1="124.46" y1="99.06" x2="129.54" y2="99.06" width="0.1524" layer="91"/>
-<label x="129.54" y="99.06" size="1.27" layer="95" xref="yes"/>
+<pinref part="U$2" gate="G$1" pin="PB2"/>
+<wire x1="129.54" y1="134.62" x2="124.46" y2="134.62" width="0.1524" layer="91"/>
+<label x="129.54" y="134.62" size="1.27" layer="95" xref="yes"/>
 </segment>
 </net>
-<net name="NOTAUS" class="0">
+<net name="ACTIVATE_BOOSTER" class="0">
+<segment>
+<pinref part="U$2" gate="G$1" pin="PB5"/>
+<wire x1="129.54" y1="142.24" x2="124.46" y2="142.24" width="0.1524" layer="91"/>
+<label x="129.54" y="142.24" size="1.27" layer="95" xref="yes"/>
+</segment>
+</net>
+<net name="FREI2" class="0">
+<segment>
+<pinref part="U$2" gate="G$1" pin="PB6"/>
+<wire x1="124.46" y1="144.78" x2="129.54" y2="144.78" width="0.1524" layer="91"/>
+<label x="129.54" y="144.78" size="1.27" layer="95" xref="yes"/>
+</segment>
+</net>
+<net name="ACTIVATE_SERVO" class="0">
+<segment>
+<pinref part="U$2" gate="G$1" pin="PD5"/>
+<wire x1="124.46" y1="96.52" x2="129.54" y2="96.52" width="0.1524" layer="91"/>
+<label x="129.54" y="96.52" size="1.27" layer="95" xref="yes"/>
+</segment>
+</net>
+<net name="FREI3" class="0">
 <segment>
 <pinref part="U$2" gate="G$1" pin="PD7"/>
@@
 </segment>
 </net>
+<net name="NOTAUS" class="0">
+<segment>
+<pinref part="U$2" gate="G$1" pin="PC6"/>
+<wire x1="129.54" y1="121.92" x2="124.46" y2="121.92" width="0.1524" layer="91"/>
+<label x="129.54" y="121.92" size="1.27" layer="95" xref="yes"/>
+</segment>
+</net>
+<net name="BURST" class="0">
+<segment>
+<pinref part="U$2" gate="G$1" pin="PC5"/>
+<wire x1="124.46" y1="119.38" x2="129.54" y2="119.38" width="0.1524" layer="91"/>
+<label x="129.54" y="119.38" size="1.27" layer="95" xref="yes"/>
+</segment>
+</net>
 <net name="STBY" class="0">
 <segment>
-<pinref part="U$2" gate="G$1" pin="PD5"/>
-<wire x1="124.46" y1="96.52" x2="129.54" y2="96.52" width="0.1524" layer="91"/>
-<label x="129.54" y="96.52" size="1.27" layer="95" xref="yes"/>
+<pinref part="U$2" gate="G$1" pin="PC4"/>
+<wire x1="124.46" y1="116.84" x2="129.54" y2="116.84" width="0.1524" layer="91"/>
+<label x="129.54" y="116.84" size="1.27" layer="95" xref="yes"/>
 </segment>
 </net>

Commit message: rekick 2015
Parts:
- added C46: 100p, rcl:C-EUC0603
Connections:
- net +12V: no longer R30.2
- net +24V: now also R30.2
- net CAP_0V: now also C46.2
- net GND: now also C38.2, R13.1
- net GND1: no longer C38.2, R13.1
- net N$27: now also C46.1
Changed lines of the file:
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@@
 <part name="R27" library="rcl" deviceset="R-EU_" device="R0805" value="10k"/>
 <part name="R28" library="rcl" deviceset="R-EU_" device="R0805" value="10k"/>
-<part name="SUPPLY18" library="supply2" deviceset="GND1" device=""/>
 <part name="P+20" library="supply1" deviceset="+5V" device=""/>
 <part name="C36" library="rcl" deviceset="C-EU" device="C0603" value="100p"/>
@@
 <part name="SUPPLY23" library="supply2" deviceset="+5V/3" device=""/>
 <part name="SUPPLY24" library="supply2" deviceset="+5V/3" device=""/>
-<part name="P+17" library="supply1" deviceset="+12V" device=""/>
 <part name="C39" library="rcl" deviceset="C-EU" device="C0603" value="100n"/>
 <part name="D14" library="diode" deviceset="BZX84CSMD" device="" value="BZX84-A5V1"/>
@@
 <part name="R54" library="rcl" deviceset="R-EU_" device="R0805" value="100k"/>
 <part name="SUPPLY30" library="supply2" deviceset="+5V/1" device=""/>
+<part name="C46" library="rcl" deviceset="C-EU" device="C0603" value="100p"/>
+<part name="GND38" library="supply1" deviceset="GND" device=""/>
+<part name="P+17" library="supply1" deviceset="+24V" device=""/>
 </parts>
 <sheets>
@@
 <instance part="R27" gate="G$1" x="99.06" y="38.1" rot="R90"/>
 <instance part="R28" gate="G$1" x="99.06" y="17.78" rot="R90"/>
-<instance part="SUPPLY18" gate="G$1" x="88.9" y="7.62"/>
 <instance part="P+20" gate="1" x="109.22" y="86.36"/>
 <instance part="C36" gate="G$1" x="96.52" y="68.58"/>
@@
 <instance part="SUPPLY23" gate="G$1" x="88.9" y="93.98"/>
 <instance part="SUPPLY24" gate="G$1" x="99.06" y="48.26"/>
-<instance part="P+17" gate="1" x="10.16" y="129.54"/>
 <instance part="C39" gate="G$1" x="17.78" y="99.06"/>
 <instance part="D14" gate="G$1" x="10.16" y="99.06" rot="R90"/>
@@
 <instance part="C45" gate="G$1" x="15.24" y="157.48"/>
 <instance part="R52" gate="G$1" x="81.28" y="71.12"/>
+<instance part="GND38" gate="1" x="88.9" y="7.62"/>
+<instance part="P+17" gate="1" x="10.16" y="129.54"/>
 </instances>
 <busses>
@@
 <junction x="129.54" y="152.4"/>
 </segment>
+<segment>
+<pinref part="R13" gate="G$1" pin="1"/>
+<wire x1="88.9" y1="12.7" x2="88.9" y2="10.16" width="0.1524" layer="91"/>
+<pinref part="C38" gate="G$1" pin="2"/>
+<wire x1="91.44" y1="12.7" x2="88.9" y2="12.7" width="0.1524" layer="91"/>
+<junction x="88.9" y="12.7"/>
+<pinref part="GND38" gate="1" pin="GND"/>
+</segment>
 </net>
 <net name="+5V" class="0">
@@
 </segment>
 </net>
-<net name="GND1" class="0">
-<segment>
-<pinref part="R13" gate="G$1" pin="1"/>
-<pinref part="SUPPLY18" gate="G$1" pin="GND1"/>
-<wire x1="88.9" y1="12.7" x2="88.9" y2="10.16" width="0.1524" layer="91"/>
-<pinref part="C38" gate="G$1" pin="2"/>
-<wire x1="91.44" y1="12.7" x2="88.9" y2="12.7" width="0.1524" layer="91"/>
-<junction x="88.9" y="12.7"/>
-</segment>
-</net>
 <net name="+5V/3" class="0">
 <segment>
@@
 <junction x="17.78" y="104.14"/>
 <pinref part="SUPPLY25" gate="G$1" pin="+5V/3"/>
-</segment>
-</net>
-<net name="+12V" class="0">
-<segment>
-<wire x1="10.16" y1="124.46" x2="10.16" y2="127" width="0.1524" layer="91"/>
-<pinref part="R30" gate="G$1" pin="2"/>
-<pinref part="P+17" gate="1" pin="+12V"/>
 </segment>
 </net>
@@
 <wire x1="76.2" y1="71.12" x2="73.66" y2="71.12" width="0.1524" layer="91"/>
 <label x="73.66" y="71.12" size="1.778" layer="95" rot="R180" xref="yes"/>
+</segment>
+</net>
+<net name="+24V" class="0">
+<segment>
+<wire x1="10.16" y1="124.46" x2="10.16" y2="127" width="0.1524" layer="91"/>
+<pinref part="R30" gate="G$1" pin="2"/>
+<pinref part="P+17" gate="1" pin="+24V"/>
 </segment>
 </net>
@@
 <instance part="C42" gate="G$1" x="12.7" y="149.86"/>
 <instance part="C43" gate="G$1" x="162.56" y="152.4"/>
+<instance part="C46" gate="G$1" x="149.86" y="71.12"/>
 </instances>
 <busses>
@@
 <junction x="144.78" y="78.74"/>
 <pinref part="IC1" gate="B" pin="-IN"/>
-<wire x1="152.4" y1="78.74" x2="144.78" y2="78.74" width="0.1524" layer="91"/>
+<wire x1="152.4" y1="78.74" x2="149.86" y2="78.74" width="0.1524" layer="91"/>
+<pinref part="C46" gate="G$1" pin="1"/>
+<wire x1="149.86" y1="78.74" x2="144.78" y2="78.74" width="0.1524" layer="91"/>
+<wire x1="149.86" y1="73.66" x2="149.86" y2="78.74" width="0.1524" layer="91"/>
+<junction x="149.86" y="78.74"/>
 </segment>
 </net>
@@
 <wire x1="129.54" y1="63.5" x2="144.78" y2="63.5" width="0.1524" layer="91"/>
 <junction x="129.54" y="63.5"/>
-<wire x1="144.78" y1="63.5" x2="182.88" y2="63.5" width="0.1524" layer="91"/>
+<wire x1="144.78" y1="63.5" x2="149.86" y2="63.5" width="0.1524" layer="91"/>
+<wire x1="149.86" y1="63.5" x2="182.88" y2="63.5" width="0.1524" layer="91"/>
 <wire x1="182.88" y1="63.5" x2="182.88" y2="76.2" width="0.1524" layer="91"/>
 <junction x="144.78" y="63.5"/>
 <pinref part="OK2" gate="A" pin="C"/>
 <wire x1="182.88" y1="76.2" x2="187.96" y2="76.2" width="0.1524" layer="91"/>
-</segment>
-<segment>
+<pinref part="C46" gate="G$1" pin="2"/>
+<wire x1="149.86" y1="66.04" x2="149.86" y2="63.5" width="0.1524" layer="91"/>
+<junction x="149.86" y="63.5"/>
+</segment>
+<segment>
