File: msl_electronic_boards/rekick2015/pcb/rekick2015-001.brd (EAGLE design)
At the start: 160 x 100 mm, 90 parts, among them IC1 LM1458D, IC2 4043D, Q1 16MHz, Q2 SiHB24N65E, U1 TXB0108PWR, U2 LM2675, U3 LM2675, U4 LM2675

Commit message: changes new rekick
Parts:
- added C26: 100p, rcl:C0603
- added IC3: 74HCT14D, 74xx-eu:SO14
- added OK3: ILD213, optocoupler:SOIC08
- added R12, R13: 12k, rcl:R0805
- added R14: 380, rcl:R0805
- added R15: 10k, rcl:R0805
- added R16: 470k, rcl:0207/15
- added U5: MC14025BDG, MC14025BDG:SOIC127P600X175-14N
- Q2: value SiHB24N65E -> BUZ11BV; device transistor-power:D2PACK -> transistor-power:TO220BV
- moved Q2 449.9 mm to (-126.2, -359.2)
Connections:
- removed net MCU_UIN: IC2.3
- removed net U_IN: IC2.4
- new net N$37: IC2.10, U5.1
- new net N$38: IC2.1, U5.3
- new net N$41: C26.1, OK3.8, R15.1
- new net NOTAUS_PRI: OK3.2, U5.9
- net +5V: now also IC3.14, R14.1, U5.14
- net BOOSTER_24V: now also R12.2
- net CAP_0V: now also C26.2, OK3.7, Q2.S; no longer Q2.3
- net GND: now also IC3.7, R13.1, U5.11, U5.7
- net N$24: now also Q2.D; no longer Q2.2
- net N$39: now also R12.1, R13.2; no longer IC2.6
- net N$40: now also OK3.1, R14.2; no longer IC2.7
- net VON_NOTAUS: now also Q2.G; no longer Q2.1
Changed lines of the file:
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@@
 <element name="R2" library="resistor-power" package="HS50" value="47" x="116.078" y="82.296"/>
 <element name="R3" library="resistor-power" package="HS50" value="47" x="117.602" y="56.388"/>
-<element name="Q2" library="transistor-power" package="D2PACK" value="SiHB24N65E" x="115.824" y="20.066"/>
 <element name="C15" library="rcl" package="C0603" value="100p" x="126.746" y="46.99"/>
 <element name="R6" library="rcl" package="R0805" value="12k" x="127.254" y="32.004"/>
@@
 <element name="C25" library="rcl" package="EB20D" value="2200µ" x="152.146" y="11.684"/>
 <element name="IC2" library="40xx" package="SO16" value="4043D" x="-124.714" y="-354.838"/>
+<element name="Q2" library="transistor-power" package="TO220BV" value="BUZ11BV" x="-126.238" y="-359.156"/>
+<element name="U5" library="MC14025BDG" package="SOIC127P600X175-14N" value="MC14025BDG" x="-140.716" y="-358.902">
+<attribute name="PACKAGE" value="SOIC-14" x="-140.716" y="-358.902" size="1.778" layer="27" display="off"/>
+<attribute name="OC_NEWARK" value="26K3933" x="-140.716" y="-358.902" size="1.778" layer="27" display="off"/>
+<attribute name="MPN" value="MC14025BDG" x="-140.716" y="-358.902" size="1.778" layer="27" display="off"/>
+<attribute name="SUPPLIER" value="ON SEMICONDUCTOR" x="-140.716" y="-358.902" size="1.778" layer="27" display="off"/>
+<attribute name="OC_FARNELL" value="1191824" x="-140.716" y="-358.902" size="1.778" layer="27" display="off"/>
+</element>
+<element name="R12" library="rcl" package="R0805" value="12k" x="-142.748" y="-370.332"/>
+<element name="R13" library="rcl" package="R0805" value="12k" x="-142.748" y="-376.428"/>
+<element name="IC3" library="74xx-eu" package="SO14" value="74HCT14D" x="-138.176" y="-384.556"/>
+<element name="OK3" library="optocoupler" package="SOIC08" value="ILD213" x="-149.606" y="-384.556"/>
+<element name="R14" library="rcl" package="R0805" value="380" x="-152.146" y="-391.922"/>
+<element name="R15" library="rcl" package="R0805" value="10k" x="-152.146" y="-398.018"/>
+<element name="C26" library="rcl" package="C0603" value="100p" x="-152.654" y="-403.606"/>
+<element name="R16" library="rcl" package="0207/15" value="470k" x="-145.542" y="-409.194"/>
 </elements>
 <signals>
@@
 <contactref element="IC2" pad="16"/>
 <contactref element="OK2" pad="8"/>
+<contactref element="U5" pad="14"/>
+<contactref element="IC3" pad="14"/>
+<contactref element="R14" pad="1"/>
+<wire x1="-129.159" y1="-351.7646" x2="-138.2522" y2="-355.092" width="0" layer="19" extent="1-1"/>
+<wire x1="-141.986" y1="-381.4826" x2="-138.2522" y2="-355.092" width="0" layer="19" extent="1-1"/>
+<wire x1="-153.096" y1="-391.922" x2="-141.986" y2="-381.4826" width="0" layer="19" extent="1-1"/>
 <wire x1="17.132" y1="44.704" x2="-129.159" y2="-351.7646" width="0" layer="19" extent="1-1"/>
 <wire x1="14.5542" y1="56.261" x2="17.132" y2="44.704" width="0" layer="19" extent="1-1"/>
@@
 <contactref element="IC2" pad="15"/>
 <contactref element="IC2" pad="11"/>
+<contactref element="U5" pad="11"/>
+<contactref element="U5" pad="7"/>
+<contactref element="R13" pad="1"/>
+<contactref element="IC3" pad="7"/>
+<wire x1="-138.2522" y1="-358.902" x2="-143.1798" y2="-362.712" width="0" layer="19" extent="1-1"/>
+<wire x1="-127.889" y1="-351.7646" x2="-138.2522" y2="-358.902" width="0" layer="19" extent="1-1"/>
 <wire x1="-122.809" y1="-351.7646" x2="-127.889" y2="-351.7646" width="0" layer="19" extent="1-1"/>
 <wire x1="-120.269" y1="-357.9114" x2="-122.809" y2="-351.7646" width="0" layer="19" extent="1-1"/>
+<wire x1="-143.698" y1="-376.428" x2="-143.1798" y2="-362.712" width="0" layer="19" extent="1-1"/>
+<wire x1="-134.366" y1="-387.6294" x2="-143.698" y2="-376.428" width="0" layer="19" extent="1-1"/>
 <wire x1="4.046" y1="3.81" x2="-122.809" y2="-351.7646" width="0" layer="19" extent="1-1"/>
 <wire x1="3.95" y1="12.7" x2="4.046" y2="3.81" width="0" layer="19" extent="1-1"/>
@@
 <contactref element="Q3" pad="D"/>
 <contactref element="C9" pad="+"/>
+<contactref element="R12" pad="2"/>
 <wire x1="72.898" y1="79.756" x2="72.39" y2="92.456" width="0" layer="19" extent="1-1"/>
 <wire x1="47.244" y1="92.202" x2="72.39" y2="92.456" width="0" layer="19" extent="1-1"/>
+<wire x1="-141.798" y1="-370.332" x2="72.898" y2="79.756" width="0" layer="19" extent="1-1"/>
 </signal>
 <signal name="N$16">
@@
 </signal>
 <signal name="N$24">
-<contactref element="Q2" pad="2"/>
 <contactref element="R3" pad="2"/>
-<wire x1="149.072" y1="56.388" x2="115.824" y2="22.606" width="0" layer="19" extent="1-1"/>
+<contactref element="Q2" pad="D"/>
+<wire x1="149.072" y1="56.388" x2="-126.238" y2="-361.696" width="0" layer="19" extent="1-1"/>
 </signal>
 <signal name="NOTAUS">
@@
 <contactref element="OK1" pad="4"/>
 <contactref element="C15" pad="2"/>
-<contactref element="Q2" pad="3"/>
 <contactref element="R4" pad="1"/>
 <contactref element="R6" pad="1"/>
@@
 <contactref element="D11" pad="A"/>
 <contactref element="C25" pad="-"/>
-<wire x1="127.596" y1="46.99" x2="118.364" y2="11.176" width="0" layer="19" extent="1-1"/>
-<wire x1="126.304" y1="32.004" x2="127.596" y2="46.99" width="0" layer="19" extent="1-1"/>
+<contactref element="Q2" pad="S"/>
+<contactref element="OK3" pad="7"/>
+<contactref element="C26" pad="2"/>
+<wire x1="-150.241" y1="-381.4826" x2="-123.698" y2="-361.696" width="0" layer="19" extent="1-1"/>
+<wire x1="-151.804" y1="-403.606" x2="-150.241" y2="-381.4826" width="0" layer="19" extent="1-1"/>
+<wire x1="104.736" y1="18.542" x2="-123.698" y2="-361.696" width="0" layer="19" extent="1-1"/>
+<wire x1="103.444" y1="24.13" x2="104.736" y2="18.542" width="0" layer="19" extent="1-1"/>
+<wire x1="106.299" y1="39.0906" x2="103.444" y2="24.13" width="0" layer="19" extent="1-1"/>
+<wire x1="126.304" y1="32.004" x2="106.299" y2="39.0906" width="0" layer="19" extent="1-1"/>
 <wire x1="133.184" y1="26.416" x2="126.304" y2="32.004" width="0" layer="19" extent="1-1"/>
+<wire x1="139.827" y1="37.5666" x2="133.184" y2="26.416" width="0" layer="19" extent="1-1"/>
+<wire x1="148.572" y1="40.894" x2="139.827" y2="37.5666" width="0" layer="19" extent="1-1"/>
+<wire x1="127.596" y1="46.99" x2="126.304" y2="32.004" width="0" layer="19" extent="1-1"/>
 <wire x1="126.304" y1="11.43" x2="133.184" y2="26.416" width="0" layer="19" extent="1-1"/>
-<wire x1="70.17" y1="51.816" x2="127.596" y2="46.99" width="0" layer="19" extent="1-1"/>
-<wire x1="139.827" y1="37.5666" x2="126.304" y2="11.43" width="0" layer="19" extent="1-1"/>
-<wire x1="76.454" y1="60.706" x2="139.827" y2="37.5666" width="0" layer="19" extent="1-1"/>
-<wire x1="106.299" y1="39.0906" x2="76.454" y2="60.706" width="0" layer="19" extent="1-1"/>
-<wire x1="103.444" y1="24.13" x2="106.299" y2="39.0906" width="0" layer="19" extent="1-1"/>
-<wire x1="104.736" y1="18.542" x2="103.444" y2="24.13" width="0" layer="19" extent="1-1"/>
-<wire x1="148.572" y1="40.894" x2="104.736" y2="18.542" width="0" layer="19" extent="1-1"/>
-<wire x1="148.572" y1="20.32" x2="148.572" y2="40.894" width="0" layer="19" extent="1-1"/>
+<wire x1="148.572" y1="20.32" x2="133.184" y2="26.416" width="0" layer="19" extent="1-1"/>
 <wire x1="157.226" y1="11.684" x2="148.572" y2="20.32" width="0" layer="19" extent="1-1"/>
+<wire x1="76.454" y1="60.706" x2="106.299" y2="39.0906" width="0" layer="19" extent="1-1"/>
+<wire x1="70.17" y1="51.816" x2="76.454" y2="60.706" width="0" layer="19" extent="1-1"/>
 </signal>
 <signal name="CAP_+12V">
@@
 <wire x1="106.299" y1="45.2374" x2="105.344" y2="30.226" width="0" layer="19" extent="1-1"/>
 </signal>
-<signal name="VON_NOTAUS">
-<contactref element="Q2" pad="1"/>
-</signal>
 <signal name="N$30">
 <contactref element="F1" pad="P$2"/>
@@
 <contactref element="IC2" pad="12"/>
 </signal>
-<signal name="U_IN">
-<contactref element="IC2" pad="4"/>
-</signal>
-<signal name="MCU_UIN">
-<contactref element="IC2" pad="3"/>
+<signal name="VON_NOTAUS">
+<contactref element="Q2" pad="G"/>
+</signal>
+<signal name="N$37">
+<contactref element="IC2" pad="10"/>
+<contactref element="U5" pad="1"/>
+<wire x1="-121.539" y1="-351.7646" x2="-143.1798" y2="-355.092" width="0" layer="19" extent="1-1"/>
+</signal>
+<signal name="N$38">
+<contactref element="IC2" pad="1"/>
+<contactref element="U5" pad="3"/>
+<wire x1="-129.159" y1="-357.9114" x2="-143.1798" y2="-357.632" width="0" layer="19" extent="1-1"/>
 </signal>
 <signal name="N$39">
-<contactref element="IC2" pad="6"/>
+<contactref element="R13" pad="2"/>
+<contactref element="R12" pad="1"/>
+<wire x1="-143.698" y1="-370.332" x2="-141.798" y2="-376.428" width="0" layer="19" extent="1-1"/>
+</signal>
+<signal name="NOTAUS_PRI">
+<contactref element="U5" pad="9"/>
+<contactref element="OK3" pad="2"/>
+<wire x1="-150.241" y1="-387.6294" x2="-138.2522" y2="-361.442" width="0" layer="19" extent="1-1"/>
 </signal>
 <signal name="N$40">
-<contactref element="IC2" pad="7"/>
+<contactref element="R14" pad="2"/>
+<contactref element="OK3" pad="1"/>
+<wire x1="-151.511" y1="-387.6294" x2="-151.196" y2="-391.922" width="0" layer="19" extent="1-1"/>
+</signal>
+<signal name="N$41">
+<contactref element="OK3" pad="8"/>
+<contactref element="R15" pad="1"/>
+<contactref element="C26" pad="1"/>
+<wire x1="-153.096" y1="-398.018" x2="-153.504" y2="-403.606" width="0" layer="19" extent="1-1"/>
+<wire x1="-151.511" y1="-381.4826" x2="-153.096" y2="-398.018" width="0" layer="19" extent="1-1"/>
 </signal>
 </signals>

Commit message: update rekick 2015
Parts:
- removed C26: 100p, rcl:C0603
- removed OK3: ILD213, optocoupler:SOIC08
- removed Q2: BUZ11BV, transistor-power:TO220BV
- added D5: SMD ZD 15, diode:TO236
- added Q6: IRF840, transistor-power:TO220BV
- added R17: 380, rcl:R0805
- added R18: 10, rcl:R0805
- added R19: 47k, rcl:R0805
- added T1, T2: BC849, transistor:SOT23
- added U$5, U$6: SI8261ABC, Si8261:SOIC-8
- R15: value 10k -> 10
- moved R15 38.3 mm to (-178.1, -426.2)
Connections:
- removed net VON_NOTAUS: Q2.G
- new net KICKER: R19.1
- new net N$42: T2.3, U$6.3
- new net N$43: R17.1, U$6.2
- new net N$44: R18.1, U$6.6, U$6.7
- new net N$45: D5.C, Q6.G, R16.1, T1.3
- new net N$46: R15.2, T1.1
- new net N$47: R19.2, T2.1
- new net N$48: R18.2
- net +5V: now also R17.2
- net CAP_+12V: now also U$5.8, U$6.8
- net CAP_0V: now also D5.A, Q6.S, T1.2, U$5.5, U$6.5; no longer C26.2, OK3.7, Q2.S
- net CAP_330V: now also R16.2
- net GND: now also T2.2, U$5.1, U$5.4, U$6.1, U$6.4
- net N$24: now also Q6.D; no longer Q2.D
- net N$40: now also U$5.2; no longer OK3.1
- net N$41: now also U$5.6, U$5.7; no longer C26.1, OK3.8
- net NOTAUS_PRI: now also U$5.3; no longer OK3.2

Commit message: changes rekick2015
Parts:
- added C26, C27, C28: 100n, rcl:C0603
- added COIL_IN, COIL_OUT: WIREPADSMD5-5, mywirepad:5-5
- added D12: 5KPXX, diode:P6T15
- added Q2: IGW60T120, transistor-power:TO247BV
- added R20: B72220S0321K101, varistor:S20K320
- added RJ_1: RJ10, ownParts:RJ10
- added X1, X2: (no value), con-ptr500:AK500/2-H
- L3, L4: device rcl:TJ9-U2 -> rcl:LAL03
- moved Q6 585.4 mm to (122.2, 70.6)
- moved R16 572.0 mm to (133.9, 89.9)
- moved D5 551.7 mm to (117.9, 11.2)
- moved R19 545.9 mm to (65.8, 21.3)
- moved T2 542.5 mm to (71.9, 21.3)
- moved IC3 541.5 mm to (152.4, 72.4)
- moved T1 536.0 mm to (96.0, 14.5), turned to 270 degrees
- moved U5 530.7 mm to (137.7, 93.0), turned to 90 degrees
- moved R18 527.2 mm to (88.9, 22.4)
- moved IC2 525.0 mm to (150.1, 92.5)
- moved R15 516.2 mm to (89.2, 15.5)
- moved U$6 508.5 mm to (81.5, 21.8)
- moved R13 499.3 mm to (137.2, 37.1), turned to 270 degrees
- moved R17 496.1 mm to (66.5, 25.1)
- moved U$5 495.8 mm to (81.5, 14.7)
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Connections:
- new net N$49: COIL_IN.P$1, D12.A, Q2.D, R20.2
- new net N$50: COIL_OUT.P$1, D12.C
- net +3V3: now also C26.2, C27.1, C27.2
- net +5V: now also C26.1, C28.1
- net BOOSTER_24V: now also X2.2
- net CAN_H: now also RJ_1.P$3
- net CAN_L: now also RJ_1.P$2
- net CAP_0V: now also Q2.S, R20.1
- net GND: now also C28.2, RJ_1.P$4, X1.2
- net GND1: now also X2.1
- net N$30: now also X1.1
- net N$48: now also Q2.G

Commit message: changes rekick2015
Connections:
- net ZU-ADC_OPV renamed ADC_CAP
- removed net KICKER: R19.1
- removed net NOTAUS: U$3.8
- removed net ZU-NOTAUS-FF: C24.1, OK2.7, R10.2
- new net ACTIVATE_BOOSTER: IC3.11, U$2.24
- new net KICK: R19.1, U$2.23
- new net N$51: IC3.10, U5.4
- new net N$52: IC3.12, U5.2
- net N$39: now also IC3.13
- net NOTAUS_PRI: now also U$3.8
- net ÜBERSPANNUNG: now also C24.1, OK2.7, R10.2
Changed lines of the file:
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@@
 <wire x1="122.174" y1="68.072" x2="149.072" y2="56.388" width="0" layer="19" extent="1-1"/>
-</signal>
-<signal name="NOTAUS">
-<contactref element="U$3" pad="8"/>
 </signal>
 <signal name="N$27">
@@
 <wire x1="128.524" y1="26.858" x2="115.884" y2="26.289" width="0" layer="19" extent="1-1"/>
 </signal>
-<signal name="ZU-ADC_OPV">
+<signal name="ADC_CAP">
 <contactref element="OK1" pad="5"/>
 <contactref element="R8" pad="2"/>
@@
 <contactref element="OK2" pad="1"/>
 <wire x1="78.2066" y1="30.353" x2="114.996" y2="40.894" width="0" layer="19" extent="1-1"/>
-</signal>
-<signal name="ZU-NOTAUS-FF">
-<contactref element="R10" pad="2"/>
-<contactref element="OK2" pad="7"/>
-<contactref element="C24" pad="1"/>
-<wire x1="72.71" y1="26.416" x2="84.3534" y2="29.083" width="0" layer="19" extent="1-1"/>
-<wire x1="70.27" y1="35.814" x2="72.71" y2="26.416" width="0" layer="19" extent="1-1"/>
 </signal>
 <signal name="N$30">
@@
 <signal name="ÜBERSPANNUNG">
 <contactref element="IC2" pad="12"/>
+<contactref element="R10" pad="2"/>
+<contactref element="OK2" pad="7"/>
+<contactref element="C24" pad="1"/>
+<wire x1="84.3534" y1="29.083" x2="150.749" y2="95.5294" width="0" layer="19" extent="1-1"/>
+<wire x1="72.71" y1="26.416" x2="84.3534" y2="29.083" width="0" layer="19" extent="1-1"/>
+<wire x1="70.27" y1="35.814" x2="72.71" y2="26.416" width="0" layer="19" extent="1-1"/>
 </signal>
 <signal name="N$37">
@@
 <contactref element="R13" pad="2"/>
 <contactref element="R12" pad="1"/>
+<contactref element="IC3" pad="13"/>
+<wire x1="137.16" y1="36.134" x2="149.86" y2="75.4634" width="0" layer="19" extent="1-1"/>
 <wire x1="137.16" y1="33.462" x2="137.16" y2="36.134" width="0" layer="19" extent="1-1"/>
 </signal>
@@
 <contactref element="U5" pad="9"/>
 <contactref element="U$5" pad="3"/>
-<wire x1="79.0702" y1="14.097" x2="140.208" y2="95.4278" width="0" layer="19" extent="1-1"/>
+<contactref element="U$3" pad="8"/>
+<wire x1="43.307" y1="73.6" x2="140.208" y2="95.4278" width="0" layer="19" extent="1-1"/>
+<wire x1="79.0702" y1="14.097" x2="43.307" y2="73.6" width="0" layer="19" extent="1-1"/>
 </signal>
 <signal name="N$40">
@@
 <wire x1="66.736" y1="21.336" x2="70.932" y2="20.236" width="0" layer="19" extent="1-1"/>
 </signal>
-<signal name="KICKER">
-<contactref element="R19" pad="1"/>
-</signal>
 <signal name="N$48">
 <contactref element="R18" pad="2"/>
@@
 <wire x1="-4.064" y1="-13.462" x2="-7.112" y2="-31.75" width="0" layer="19" extent="1-1"/>
 </signal>
+<signal name="ACTIVATE_BOOSTER">
+<contactref element="IC3" pad="11"/>
+<contactref element="U$2" pad="24"/>
+<wire x1="46.9646" y1="33.776" x2="152.4" y2="75.4634" width="0" layer="19" extent="1-16"/>
+</signal>
+<signal name="N$51">
+<contactref element="IC3" pad="10"/>
+<contactref element="U5" pad="4"/>
+<wire x1="137.668" y1="90.5002" x2="153.67" y2="75.4634" width="0" layer="19" extent="1-1"/>
+</signal>
+<signal name="N$52">
+<contactref element="U5" pad="2"/>
+<contactref element="IC3" pad="12"/>
+<wire x1="151.13" y1="75.4634" x2="135.128" y2="90.5002" width="0" layer="19" extent="1-1"/>
+</signal>
+<signal name="KICK">
+<contactref element="U$2" pad="23"/>
+<contactref element="R19" pad="1"/>
+<wire x1="46.9646" y1="34.576" x2="64.836" y2="21.336" width="0" layer="19" extent="1-16"/>
+</signal>
 </signals>

Commit message: edit rekick2015
Parts:
- removed R103: 12k, rcl:R0805
- added C29, C30: 47µF/35V, rcl:PANASONIC_D
- added C31, C32: 1µ, rcl:C0603
- added C33, C34: 100n, rcl:C0603
- added C35: 1µ/50V, rcl:C0603
- added C36, C37, C38, C39: 100p, rcl:C0603
- added D13: SMD ZD 12, diode:TO236
- added D14: BZX84-A5V1, diode:TO236
- added IC4: LM1458D, linear:SO08
- added Q5: IPD90P04P4L, transistor-power:D-PAK_TO252AA
- added R200: 47k, rcl:R0805
- added R21: 10k, 1%, rcl:R0805
- added R22, R24, R25, R26, R27, R28: 10k, rcl:R0805
- added R23: (no value), ptc-ntc:N644A
- added R29, R30: 1k, rcl:R0805
- added S1: (no value), switch-omron:B3F-10XX
- added T3, T4: BC849, transistor:SOT23
- added U$7: DSEI30-12A, dsei30-12a:TO247AD
- C10, C9: value 2200µ -> 2200µ/50V; device rcl:E5-10,5 -> rcl:E7,5-18
- C18, C2, C21: value 47µF/16V -> 47µF/35V
- D12: value 5KPXX -> BZX84-A5V1; device diode:P6T15 -> diode:TO236
- L7: value (none) -> WE-LLCR
- Q3, Q4: value (none) -> IPP023N10N5
- R101: value 1M -> 1M, 1%
- R105: value 10 -> 750
- R11, R8: value 1k -> 2k, 1%
- R12: value 12k -> 70k
- R13: value 12k -> 10k
- R4: value 10k -> 10k, 1%
- R5: value 1M -> 3k, 1%; device rcl:0207/15 -> rcl:R0805
- R6: value 12k -> 12k, 1%
- R7: value 20k -> 2.37k, 1%
- R9: value 10k -> 2k
- moved R5 181.2 mm to (-16.5, -83.8), turned to 0 degrees
- moved D12 173.9 mm to (-50.8, -197.9)
- moved C16 146.2 mm to (-8.13, -38.9), turned to 0 degrees
Connections:
- removed net SEK-FEEDBACK: C12.1, RF_MAX.1, U$3.5
- new net +5V/3: C39.1, D14.C, OK1.6, R27.2, R30.1, R5.2
- new net +5V/4: C16.1, D12.C, OK1.8, R29.1, R7.2
- new net N$53: IC4.7, U5.12
- new net N$54: D13.C, Q5.1, R200.1
- new net N$55: D13.A
- new net N$56: R24.2, T3.1
- new net N$57: C10.+, C35.1, C9.+, Q3.D, Q5.4, R23.2
- new net N$58: R26.1, T4.3, U5.2
- new net N$59: C37.1, IC4.5, R27.1, R28.2
- new net STBY: C12.1, RF_MAX.1, U$3.5, U5.6
- net +12V: now also R30.2; no longer OK1.6
- net +5V: now also C34.1, IC4.8, R26.2, S1.1, S1.2; no longer R14.1
- net ACTIVATE_BOOSTER: now also R24.1, R25.1; no longer IC3.11
- net ADC_CAP: now also IC4.3
- net BOOSTER_24V: now also Q5.3, R200.2, R23.1; no longer C10.+, C9.+, Q3.D
- net CAP_+12V: now also C29.+, C31.1, C32.1, R29.2; no longer OK1.8, R7.2
- net CAP_-12V: now also C30.-
- net CAP_0V: now also C29.-, C30.+, C31.2, C32.2, D12.A; no longer R103.1
- net CAP_330V: now also COIL_OUT.P$1, U$7.C; no longer R5.2
- net GND: now also C33.2, C34.2, C36.2, C37.2, C39.2, D14.A, IC4.4, R21.1, R22.1, R28.1, T4.2, U$5.3; no longer R13.1
- net GND1: now also C35.2, C38.2, R13.1, T3.2
- net N$15: now also IC1.5, R6.2; no longer R103.2
- net N$29: now also C36.1, IC4.2, R21.2; no longer C16.1, IC1.5, R6.2
- net N$39: now also C38.1, IC4.6; no longer IC3.13
- net N$49: now also U$7.A; no longer D12.A
- net N$50: now also IC4.1; no longer COIL_OUT.P$1, D12.C
- net N$51: no longer IC3.10
- net N$52: now also R25.2, T4.1; no longer IC3.12, U5.2
- net NOTAUS_PRI: now also R14.1; no longer U$5.3
- net TASTER: now also C33.1, R22.2, S1.3, S1.4

Commit message: edit rekick2015
Parts:
- removed C3: 10nF/50V, rcl:C0603
- removed L1: 68µH, Inductor-Fastron:PISM
- removed L2: 10µH, rcl:L2012C
- removed U2: LM2675, LM2675M-3.3:SOIC127P620X175-8N
- added CAP_0V, CAP_330V: WIREPADSMD5-5, mywirepad:5-5
- added H1, H2, H3, H4: MOUNT-PAD-ROUND3.0, holes:3,0-PAD
- added R31: 20k, rcl:R0805
- added R32: 120, rcl:R0805
- added RJ_2: RJ10, ownParts:RJ10
- added SJ1: (no value), jumper:SJ
- C13: device rcl:C1206 -> rcl:C2220K
- C16, C39: value 100p -> 100n
- IC3: value 74HCT14D -> LM1117; device 74xx-eu:SO14 -> v-reg:SOT223
- L3, L4: device rcl:LAL03 -> EagleLibrary_Wuerth_Elektronik_eiSos_rev16a:WE-HCI_1890
- R101: device rcl:0207/15 -> rcl:0207/10
- R12: value 70k -> 68k
- moved U$7 256.1 mm to (139.2, 47.5), turned to 270 degrees
- moved C31 209.5 mm to (122.2, 90.7)
- moved S1 186.3 mm to (14.0, 97.0)
- moved COIL_OUT 164.8 mm to (145.0, 56.6)
- moved COIL_IN 163.7 mm to (145.0, 46.5)
- moved R23 162.9 mm to (61.0, 20.3), turned to 90 degrees
- moved R20 153.0 mm to (145.5, 34.5), turned to 90 degrees
- moved IC3 152.3 mm to (5.59, 32.0), turned to 270 degrees
- moved Q2 140.4 mm to (145.0, 29.5)
- moved IC2 121.5 mm to (28.7, 96.8)
- moved U5 108.2 mm to (29.5, 96.0)
- moved R101 103.5 mm to (22.4, 66.8), turned to 180 degrees
- moved IC1 100.3 mm to (22.4, 66.8)
- moved D11 94.1 mm to (133.9, 10.2), turned to 270 degrees
- moved R4 93.4 mm to (73.4, 96.8), turned to 0 degrees
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Connections:
- removed net ADC8: U$2.17
- removed net D2A: U$2.25
- removed net N$12: C3.1, U2.1
- removed net N$2: C3.2, D2.K, L1.2, U2.8
- new net RF: RF_MAX.1, U$2.25
- net +24V: no longer C1.+, U2.7
- net +3V3: now also D2.A, IC3.4; no longer L1.1, U2.4
- net +5V: now also C1.+, D2.K, IC3.3; no longer IC3.14, L2.1
- net +5V/3: now also C7.2, U$2.19
- net ACTIVATE_BOOSTER: now also R31.2
- net ADC_CAP: now also U$2.17
- net CAN_H: now also RJ_2.P$3, SJ1.2
- net CAN_L: now also R32.2, RJ_2.P$2
- net CAP_0V: now also CAP_0V.P$1
- net CAP_330V: now also CAP_330V.P$1
- net GND: now also H1.B3,0, H2.B3,0, H3.B3,0, H4.B3,0, IC3.1, R31.1; no longer D2.A, IC3.7, U2.6
- net N$9: now also R32.1, SJ1.1; no longer C7.2, L2.2, U$2.19
- net STBY: no longer RF_MAX.1
