File: msl_electronic_boards/rekick2015/pcb/rekick2015-001.brd (EAGLE design)
At the start: 160 x 100 mm, 151 parts, among them IC1 LM1458D, IC2 4043D, IC3 LM1117, IC4 LM1458D, Q1 16MHz, Q2 IGW60T120, Q3 IPP023N10N5, Q4 IPP023N10N5, Q5 IPD90P04P4L, Q6 IRF840, T1 BC849, T2 BC849, T3 BC849, T4 BC849, U1 TXB0108PWR, U3 LM2675, U4 LM2675, U5 MC14025BDG

Commit message: edit rekick2015
Parts:
- L7: device EagleLibrary_Wuerth_Elektronik_eiSos_rev15h:WE-LLCR_ETD39 -> EagleLibrary_Wuerth_Elektronik_eiSos_rev15h:WE-LLCR_ETD34
- R2, R3: value 47 -> 100; device resistor-power:HS50 -> resistor-power:HS25
- moved C32 198.8 mm to (123.4, 70.7), turned to 90 degrees
- moved C30 179.3 mm to (70.2, 94.9), turned to 270 degrees
- moved C29 177.2 mm to (79.0, 94.7), turned to 90 degrees
- moved C16 167.4 mm to (94.2, 93.6), turned to 180 degrees
- moved D13 160.6 mm to (49.5, 12.1), flipped to the bottom, turned to 90 degrees
- moved R200 159.1 mm to (57.1, 18.5), flipped to the bottom
- moved T3 155.9 mm to (45.1, 2.67), flipped to the bottom, turned to 90 degrees
- moved R24 155.8 mm to (36.2, 1.78), flipped to the bottom, turned to 180 degrees
- moved Q5 145.4 mm to (47.1, 20.2), flipped to the bottom, turned to 270 degrees
- moved RJ_1 129.4 mm to (138.8, 80.5), turned to 90 degrees
- moved IC1 91.3 mm to (109.1, 95.4)
- moved R101 91.3 mm to (109.1, 95.4)
- moved L3 78.1 mm to (80.6, 10.2), turned to 0 degrees
- moved CAP_330V 77.0 mm to (103.3, 10.0), turned to 270 degrees
- moved R16 73.4 mm to (155.6, 20.8), turned to 270 degrees
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Connections:
- net N$55: now also T3.3
- net TRAFO1: now also L7.9; no longer L7.12
- net TRAFO2: now also L7.11; no longer L7.8

Commit message: edit rekick2015
Parts:
- moved R3 52.5 mm to (122.0, 74.0)
- moved L3 37.0 mm to (70.9, 45.8), turned to 270 degrees
- moved Q5 36.9 mm to (81.5, 6.99), turned to 90 degrees
- moved D13 35.1 mm to (84.6, 14.4)
- moved Q4 28.4 mm to (55.8, 40.0), turned to 90 degrees
- moved C10 23.8 mm to (71.2, 66.0), turned to 0 degrees
- moved C13 21.5 mm to (69.5, 5.46)
- moved R200 20.8 mm to (77.6, 14.9)
- moved L4 19.0 mm to (83.6, 10.4)
- moved L7 18.7 mm to (99.9, 39.9)
- moved Q3 14.0 mm to (55.8, 52.3), turned to 90 degrees
- moved C25 13.3 mm to (133.5, 40.5)
- moved C9 9.84 mm to (62.6, 24.8), turned to 0 degrees
- moved R2 0.18 mm to (144.8, 73.9), turned to 90 degrees
