File: msl_electronic_boards/rekick2015/pcb/rekick2015-001.brd (EAGLE design)
At the start: 160 x 100 mm, 151 parts, among them IC1 LM1458D, IC2 4043D, IC3 LM1117, IC4 LM1458D, Q1 16MHz, Q2 IGW60T120, Q3 IPP023N10N5, Q4 IPP023N10N5, Q5 IPD90P04P4L, Q6 IRF840, T1 BC849, T2 BC849, T3 BC849, T4 BC849, U1 TXB0108PWR, U3 LM2675, U4 LM2675, U5 MC14025BDG

Commit message: rekick2015
Parts:
- added VR1, VR2, VR3, VR4: TL431_SOT23, 1_USER:SOT23
Changed lines of the file:
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@@
 <?xml version="1.0" encoding="utf-8"?>
 <!DOCTYPE eagle SYSTEM "eagle.dtd">
-<eagle version="7.5.0">
+<eagle version="7.2.0">
 <drawing>
 <settings>
@@
 <layer number="131" name="tAdjust" color="15" fill="1" visible="no" active="no"/>
 <layer number="132" name="bAdjust" color="5" fill="1" visible="no" active="no"/>
+<layer number="200" name="200bmp" color="1" fill="10" visible="no" active="no"/>
 <layer number="250" name="Descript" color="3" fill="1" visible="no" active="no"/>
 <layer number="251" name="SMDround" color="12" fill="11" visible="no" active="no"/>
@@
 <element name="SJ1" library="jumper" package="SJ" value="" x="-61.976" y="-241.046"/>
 <element name="IC3" library="v-reg" package="SOT223" value="LM1117" x="5.588" y="32.004" rot="R270"/>
+<element name="VR1" library="1_USER" package="SOT23" value="TL431_SOT23" x="-61.849" y="-245.745"/>
+<element name="VR2" library="1_USER" package="SOT23" value="TL431_SOT23" x="-61.849" y="-253.111"/>
+<element name="VR3" library="1_USER" package="SOT23" value="TL431_SOT23" x="-61.849" y="-260.477"/>
+<element name="VR4" library="1_USER" package="SOT23" value="TL431_SOT23" x="-61.849" y="-267.843"/>
 </elements>
 <signals>

Commit message: rekick 2015
Parts:
- added R33, R34, R35: 1M, rcl:R2512
- added R36: 50k, rcl:R0805
- added R37: 17k, rcl:R0805
- added R38: 7.68k, rcl:R0805
- R101: device rcl:0207/10 -> rcl:R2512
Changed lines of the file:
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@@
 <?xml version="1.0" encoding="utf-8"?>
 <!DOCTYPE eagle SYSTEM "eagle.dtd">
-<eagle version="7.2.0">
+<eagle version="7.5.0">
 <drawing>
 <settings>
@@
 <element name="C9" library="rcl" package="E7,5-18" value="2200µ/50V" x="62.611" y="24.765"/>
 <element name="C10" library="rcl" package="E7,5-18" value="2200µ/50V" x="71.247" y="66.04"/>
-<element name="R101" library="rcl" package="0207/10" value="1M, 1%" x="109.093" y="95.377" rot="R180">
+<element name="R101" library="rcl" package="R2512" value="1M, 1%" x="109.093" y="95.377" rot="R180">
 <attribute name="FARNELL" value="2396016" x="109.093" y="95.377" size="1.778" layer="27" rot="R180" display="off"/>
 </element>
@@
 <element name="VR3" library="1_USER" package="SOT23" value="TL431_SOT23" x="-61.849" y="-260.477"/>
 <element name="VR4" library="1_USER" package="SOT23" value="TL431_SOT23" x="-61.849" y="-267.843"/>
+<element name="R33" library="rcl" package="R2512" value="1M" x="-60.325" y="-275.209"/>
+<element name="R34" library="rcl" package="R2512" value="1M" x="-60.325" y="-280.924"/>
+<element name="R35" library="rcl" package="R2512" value="1M" x="-60.325" y="-286.639"/>
+<element name="R36" library="rcl" package="R0805" value="50k" x="-62.23" y="-293.37"/>
+<element name="R37" library="rcl" package="R0805" value="17k" x="-62.23" y="-299.466"/>
+<element name="R38" library="rcl" package="R0805" value="7.68k" x="-62.23" y="-305.562"/>
 </elements>
 <signals>
@@
 <contactref element="IC1" pad="5"/>
 <contactref element="R6" pad="2"/>
-<wire x1="114.173" y1="95.377" x2="131.125" y2="94.361" width="0" layer="19" extent="1-1"/>
-<wire x1="111.693" y1="93.472" x2="114.173" y2="95.377" width="0" layer="19" extent="1-1"/>
+<wire x1="111.893" y1="95.377" x2="131.125" y2="94.361" width="0" layer="19" extent="1-1"/>
+<wire x1="111.693" y1="93.472" x2="111.893" y2="95.377" width="0" layer="19" extent="1-1"/>
 <wire x1="106.493" y1="94.742" x2="111.693" y2="93.472" width="0" layer="19" extent="1-1"/>
 <wire x1="64.428" y1="83.82" x2="106.493" y2="94.742" width="0" layer="19" extent="1-1"/>
@@
 <wire x1="103.251" y1="10.033" x2="114.427" y2="10.033" width="0" layer="19" extent="1-1"/>
 <wire x1="155.575" y1="13.208" x2="128.397" y2="40.513" width="0" layer="19" extent="1-1"/>
-<wire x1="104.013" y1="95.377" x2="126.891" y2="44.196" width="0" layer="19" extent="16-16"/>
+<wire x1="106.293" y1="95.377" x2="126.891" y2="44.196" width="0" layer="19" extent="16-16"/>
 </signal>
 <signal name="N$23">

Commit message: rekick 2015
Parts:
- removed VR4: TL431_SOT23, 1_USER:SOT23
- added JP3: (no value), pinhead:1X03
- added LED1, LED2, LED3: (no value), led:CHIP-LED0805
- added R39, R40, R41: 50k, rcl:R0805
Connections:
- removed net CS/OC1B: U$2.3
- removed net INT2: U$2.26
- new net +5V/1: JP3.2
- new net N$12: R33.1, R36.2, VR1.2
- new net N$2: LED1.C, VR1.1
- new net N$60: R34.1, R37.2, VR2.2
- new net N$61: R35.1, R38.2, VR3.2
- new net N$62: LED2.C, VR2.1
- new net N$63: LED3.C, VR3.1
- new net RESET_NOTAUS: IC2.11, IC2.15, U$2.26
- new net SERVO_PWM: JP3.1, U$2.3
- net CAP_0V: now also R36.1, R37.1, R38.1, VR1.3, VR2.3, VR3.3
- net CAP_330V: now also R33.2, R34.2, R35.2
- net GND: now also JP3.3, U$3.8; no longer IC2.11, IC2.15
- net NOTAUS_PRI: no longer U$3.8
Changed lines of the file:
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@@
 <?xml version="1.0" encoding="utf-8"?>
 <!DOCTYPE eagle SYSTEM "eagle.dtd">
-<eagle version="7.5.0">
+<eagle version="7.2.0">
 <drawing>
 <settings>
@@
 <element name="VR2" library="1_USER" package="SOT23" value="TL431_SOT23" x="-61.849" y="-253.111"/>
 <element name="VR3" library="1_USER" package="SOT23" value="TL431_SOT23" x="-61.849" y="-260.477"/>
-<element name="VR4" library="1_USER" package="SOT23" value="TL431_SOT23" x="-61.849" y="-267.843"/>
 <element name="R33" library="rcl" package="R2512" value="1M" x="-60.325" y="-275.209"/>
 <element name="R34" library="rcl" package="R2512" value="1M" x="-60.325" y="-280.924"/>
@@
 <element name="R37" library="rcl" package="R0805" value="17k" x="-62.23" y="-299.466"/>
 <element name="R38" library="rcl" package="R0805" value="7.68k" x="-62.23" y="-305.562"/>
+<element name="LED1" library="led" package="CHIP-LED0805" value="" x="-67.437" y="-306.832"/>
+<element name="LED2" library="led" package="CHIP-LED0805" value="" x="-73.533" y="-306.832"/>
+<element name="LED3" library="led" package="CHIP-LED0805" value="" x="-79.629" y="-306.832"/>
+<element name="JP3" library="pinhead" package="1X03" value="" x="-78.105" y="-312.166"/>
+<element name="R39" library="rcl" package="R0805" value="50k" x="-80.518" y="-317.246"/>
+<element name="R40" library="rcl" package="R0805" value="50k" x="-80.518" y="-323.342"/>
+<element name="R41" library="rcl" package="R0805" value="50k" x="-80.518" y="-329.438"/>
 </elements>
 <signals>
@@
 <contactref element="C23" pad="2"/>
 <contactref element="IC2" pad="8"/>
-<contactref element="IC2" pad="15"/>
-<contactref element="IC2" pad="11"/>
 <contactref element="U5" pad="11"/>
 <contactref element="U5" pad="7"/>
@@
 <contactref element="C1" pad="-"/>
 <contactref element="IC3" pad="1"/>
+<contactref element="U$3" pad="8"/>
+<contactref element="JP3" pad="3"/>
 <wire x1="129.721" y1="82.423" x2="155.575" y2="96.012" width="0" layer="19" extent="1-1"/>
 <wire x1="129.667" y1="68.4022" x2="129.721" y2="82.423" width="0" layer="19" extent="1-1"/>
@@
 <wire x1="61.7474" y1="99.187" x2="64.0588" y2="98.679" width="0" layer="19" extent="1-1"/>
 <wire x1="59.1312" y1="94.869" x2="61.7474" y2="99.187" width="0" layer="19" extent="1-1"/>
-<wire x1="55.6006" y1="96.647" x2="59.1312" y2="94.869" width="0" layer="19" extent="1-1"/>
-<wire x1="55.6006" y1="91.567" x2="59.1312" y2="94.869" width="0" layer="19" extent="1-1"/>
 <wire x1="66.128" y1="88.138" x2="59.1312" y2="94.869" width="0" layer="19" extent="1-1"/>
-<wire x1="42.037" y1="78.8" x2="55.6006" y2="91.567" width="0" layer="19" extent="1-1"/>
+<wire x1="42.037" y1="78.8" x2="59.1312" y2="94.869" width="0" layer="19" extent="1-1"/>
 <wire x1="42.506" y1="77.216" x2="42.037" y2="78.8" width="0" layer="19" extent="1-1"/>
 <wire x1="39.966" y1="76.2" x2="42.506" y2="77.216" width="0" layer="19" extent="1-1"/>
@@
 <wire x1="36.83" y1="74.808" x2="37.172" y2="75.184" width="0" layer="19" extent="1-1"/>
 <wire x1="35.372" y1="78.232" x2="38.696" y2="77.47" width="0" layer="19" extent="1-1"/>
+<wire x1="43.307" y1="73.6" x2="42.506" y2="77.216" width="0" layer="19" extent="1-1"/>
 <wire x1="24.804" y1="81.788" x2="35.372" y2="78.232" width="0" layer="19" extent="1-1"/>
 <wire x1="18.884" y1="81.788" x2="24.804" y2="81.788" width="0" layer="19" extent="1-1"/>
@@
 <wire x1="-45.124" y1="-217.17" x2="-51.8" y2="-212.074" width="0" layer="19" extent="1-1"/>
 <wire x1="-51.75" y1="-228.854" x2="-45.124" y2="-217.17" width="0" layer="19" extent="1-1"/>
+<wire x1="-75.565" y1="-312.166" x2="-51.75" y2="-228.854" width="0" layer="19" extent="1-1"/>
 </signal>
 <signal name="SCK_3V">
@@
 <wire x1="20.447" y1="30.2768" x2="18.8214" y2="71.126" width="0" layer="19" extent="16-16"/>
 </signal>
-<signal name="CS/OC1B">
-<contactref element="U$2" pad="3"/>
-</signal>
 <signal name="SCK">
 <contactref element="U1" pad="15"/>
@@
 <signal name="ADC10">
 <contactref element="U$2" pad="22"/>
-</signal>
-<signal name="INT2">
-<contactref element="U$2" pad="26"/>
 </signal>
 <signal name="INT1">
@@
 <contactref element="U$7" pad="C"/>
 <contactref element="CAP_330V" pad="P$1"/>
-<wire x1="126.891" y1="44.196" x2="144.78" y2="53.444" width="0" layer="19" extent="16-16"/>
+<contactref element="R35" pad="2"/>
+<contactref element="R34" pad="2"/>
+<contactref element="R33" pad="2"/>
+<wire x1="126.891" y1="44.196" x2="106.293" y2="95.377" width="0" layer="19" extent="1-16"/>
 <wire x1="126.891" y1="44.196" x2="126.891" y2="44.196" width="0" layer="19" extent="1-16"/>
 <wire x1="128.397" y1="40.513" x2="126.891" y2="44.196" width="0" layer="19" extent="16-16"/>
+<wire x1="144.78" y1="53.444" x2="126.891" y2="44.196" width="0" layer="19" extent="16-16"/>
 <wire x1="114.427" y1="17.018" x2="128.397" y2="40.513" width="0" layer="19" extent="1-1"/>
 <wire x1="114.427" y1="10.033" x2="114.427" y2="17.018" width="0" layer="19" extent="1-1"/>
 <wire x1="103.251" y1="10.033" x2="114.427" y2="10.033" width="0" layer="19" extent="1-1"/>
 <wire x1="155.575" y1="13.208" x2="128.397" y2="40.513" width="0" layer="19" extent="1-1"/>
-<wire x1="106.293" y1="95.377" x2="126.891" y2="44.196" width="0" layer="19" extent="16-16"/>
+<wire x1="-57.525" y1="-275.209" x2="103.251" y2="10.033" width="0" layer="19" extent="1-1"/>
+<wire x1="-57.525" y1="-280.924" x2="-57.525" y2="-275.209" width="0" layer="19" extent="1-1"/>
+<wire x1="-57.525" y1="-286.639" x2="-57.525" y2="-280.924" width="0" layer="19" extent="1-1"/>
 </signal>
 <signal name="N$23">
@@
 <contactref element="C16" pad="2"/>
 <contactref element="CAP_0V" pad="P$1"/>
+<contactref element="VR1" pad="3"/>
+<contactref element="VR2" pad="3"/>
+<contactref element="R38" pad="1"/>
+<contactref element="R36" pad="1"/>
+<contactref element="VR3" pad="3"/>
+<contactref element="R37" pad="1"/>
+<wire x1="-61.849" y1="-244.645" x2="-51.8" y2="-198.866" width="0" layer="19" extent="1-1"/>
+<wire x1="-61.849" y1="-252.011" x2="-61.849" y2="-244.645" width="0" layer="19" extent="1-1"/>
+<wire x1="-61.849" y1="-259.377" x2="-61.849" y2="-252.011" width="0" layer="19" extent="1-1"/>
+<wire x1="-63.18" y1="-293.37" x2="-61.849" y2="-259.377" width="0" layer="19" extent="1-1"/>
+<wire x1="-63.18" y1="-299.466" x2="-63.18" y2="-293.37" width="0" layer="19" extent="1-1"/>
+<wire x1="-63.18" y1="-305.562" x2="-63.18" y2="-299.466" width="0" layer="19" extent="1-1"/>
 <wire x1="136.779" y1="10.033" x2="-51.8" y2="-198.866" width="0" layer="19" extent="1-1"/>
 <wire x1="136.652" y1="16.891" x2="136.779" y2="10.033" width="0" layer="19" extent="1-1"/>
@@
 <signal name="NOTAUS_PRI">
 <contactref element="U5" pad="9"/>
-<contactref element="U$3" pad="8"/>
 <contactref element="R14" pad="1"/>
 <wire x1="59.1312" y1="97.409" x2="151.577" y2="33.655" width="0" layer="19" extent="1-1"/>
-<wire x1="43.307" y1="73.6" x2="59.1312" y2="97.409" width="0" layer="19" extent="1-1"/>
 </signal>
 <signal name="N$40">
@@
 <wire x1="25.914" y1="64.0334" x2="35.626" y2="77.216" width="0" layer="19" extent="1-16"/>
 </signal>
+<signal name="RESET_NOTAUS">
+<contactref element="IC2" pad="15"/>
+<contactref element="IC2" pad="11"/>
+<contactref element="U$2" pad="26"/>
+<wire x1="55.6006" y1="91.567" x2="55.6006" y2="96.647" width="0" layer="19" extent="1-1"/>
+<wire x1="25.114" y1="64.0334" x2="55.6006" y2="91.567" width="0" layer="19" extent="1-16"/>
+</signal>
+<signal name="N$12">
+<contactref element="R36" pad="2"/>
+<contactref element="R33" pad="1"/>
+<contactref element="VR1" pad="2"/>
+<wire x1="-63.125" y1="-275.209" x2="-61.28" y2="-293.37" width="0" layer="19" extent="1-1"/>
+<wire x1="-60.899" y1="-246.845" x2="-63.125" y2="-275.209" width="0" layer="19" extent="1-1"/>
+</signal>
+<signal name="N$60">
+<contactref element="R34" pad="1"/>
+<contactref element="R37" pad="2"/>
+<contactref element="VR2" pad="2"/>
+<wire x1="-63.125" y1="-280.924" x2="-61.28" y2="-299.466" width="0" layer="19" extent="1-1"/>
+<wire x1="-60.899" y1="-254.211" x2="-63.125" y2="-280.924" width="0" layer="19" extent="1-1"/>
+</signal>
+<signal name="N$61">
+<contactref element="R35" pad="1"/>
+<contactref element="R38" pad="2"/>
+<contactref element="VR3" pad="2"/>
+<wire x1="-63.125" y1="-286.639" x2="-61.28" y2="-305.562" width="0" layer="19" extent="1-1"/>
+<wire x1="-60.899" y1="-261.577" x2="-63.125" y2="-286.639" width="0" layer="19" extent="1-1"/>
+</signal>
+<signal name="N$2">
+<contactref element="VR1" pad="1"/>
+<contactref element="LED1" pad="C"/>
+<wire x1="-62.799" y1="-246.845" x2="-67.437" y2="-305.782" width="0" layer="19" extent="1-1"/>
+</signal>
+<signal name="N$62">
+<contactref element="VR2" pad="1"/>
+<contactref element="LED2" pad="C"/>
+<wire x1="-62.799" y1="-254.211" x2="-73.533" y2="-305.782" width="0" layer="19" extent="1-1"/>
+</signal>
+<signal name="N$63">
+<contactref element="LED3" pad="C"/>
+<contactref element="VR3" pad="1"/>
+<wire x1="-62.799" y1="-261.577" x2="-79.629" y2="-305.782" width="0" layer="19" extent="1-1"/>
+</signal>
+<signal name="+5V/1">
+<contactref element="JP3" pad="2"/>
+</signal>
+<signal name="SERVO_PWM">
+<contactref element="JP3" pad="1"/>
+<contactref element="U$2" pad="3"/>
+<wire x1="18.8214" y1="67.126" x2="-80.645" y2="-312.166" width="0" layer="19" extent="16-16"/>
+</signal>
 </signals>

Commit message: rekick 2015
Parts:
- added C3, C40: 47µF/35V, rcl:PANASONIC_D
- added D15, D16, D17: ES1A, diode:SMA-DO214AC
- added L1: 68µH, Inductor-Fastron:PISM
- added LED10, LED4, LED5, LED6, LED7, LED8, LED9: (no value), led:CHIP-LED0805
- added R42, R46: 680, rcl:R0805
- added R43, R45: 1,5k, rcl:R0805
- added R44, R49, R50: 4.7k, rcl:R0805
- added R47: 1k, rcl:R0805
- added R48: 10k, rcl:R0805
- added T5: (no value), zetex:SOT-23
- added U$8: LM2576, LM2576:TO220511
- C25: value 2200µ -> 2.2µ
- L3: device EagleLibrary_Wuerth_Elektronik_eiSos_rev16a:WE-HCI_1890 -> inductor-bourns:SRR1210
- R39, R40, R41: value 50k -> 4.7k
- moved C9 31.2 mm to (90.0, 9.91), turned to 270 degrees
- moved Q5 25.1 mm to (58.3, 16.5), turned to 270 degrees
- moved L4 17.2 mm to (71.4, 22.5), turned to 270 degrees
- moved L3 1.37 mm to (72.1, 45.3), turned to 0 degrees
Connections:
- removed net INT1: U$2.16
- removed net NOTAUS_PRI: R14.1, U5.9
- new net ACTIVATE_SERVO: R47.1, U$2.16
- new net BURST: D17.K, U5.6
- new net N$64: LED1.A, R39.1
- new net N$65: LED2.A, R40.1
- new net N$66: LED3.A, R41.1
- new net N$67: LED4.A, R42.1
- new net N$68: C40.+, L1.1, R45.2, U$8.4
- new net N$69: D15.K, L1.2, U$8.2
- new net N$70: JP3.3, T5.1
- new net N$71: LED7.A, R45.1
- new net N$72: LED5.A, R43.1
- new net N$73: LED6.A, R44.1
- new net N$74: LED8.A, R46.1
- new net N$75: R47.2, T5.3
- new net N$76: LED9.A, R49.1
- new net N$77: LED10.A, R50.1
- new net NOTAUS: D16.K, R14.1, U5.9
- net +12V: now also R44.2
- net +24V: now also C3.+, U$8.1
- net +3V3: now also R42.2
- net +5V: now also R43.2, R48.2
- net BOOSTER_24V: now also R46.2
- net CAP_+12V: now also R39.2, R40.2, R41.2, R49.2
- net CAP_-12V: now also LED10.C
- net CAP_0V: now also LED9.C, R50.2
- net GND: now also C3.-, C40.-, D15.A, LED4.C, LED5.C, LED6.C, LED7.C, T5.2, U$8.3, U$8.5, U5.13, U5.5, U5.8; no longer JP3.3
- net GND1: now also LED8.C
- net STBY: now also D16.A, D17.A, R48.1; no longer U5.6

Commit message: rekick 2015
Parts:
- moved RJ_1 126.8 mm to (12.6, 92.6)
- moved CAP_330V 90.8 mm to (145.5, 90.4), turned to 90 degrees
- moved R23 89.0 mm to (119.8, 9.65)
- moved R16 88.4 mm to (95.5, 85.7), turned to 90 degrees
- moved R20 87.7 mm to (102.4, 88.1), turned to 180 degrees
- moved D1 86.5 mm to (121.3, 12.7), turned to 270 degrees
- moved F1 84.6 mm to (119.0, 5.46), turned to 270 degrees
- moved CAP_0V 84.1 mm to (112.0, 90.4), turned to 90 degrees
- moved COIL_OUT 82.8 mm to (134.4, 90.4), turned to 90 degrees
- moved X2 81.8 mm to (142.4, 8.38)
- moved COIL_IN 80.4 mm to (123.2, 90.4), turned to 90 degrees
- moved Q5 69.6 mm to (127.0, 5.33)
- moved C25 67.8 mm to (83.1, 85.9), turned to 90 degrees
- moved Q6 65.3 mm to (102.6, 74.5), turned to 0 degrees
- moved C10 63.7 mm to (103.1, 10.9), turned to 270 degrees
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Connections:
- removed net N$29: C36.1, IC4.2, R21.2, R5.1
- removed net RF: RF_MAX.1, U$2.25
- new net AN-AUSGANG-ODER-MCU-KOPPELN: RF_MAX.1
- new net D2A/KICK_VOLTAGE: C36.1, IC4.2, R21.2, R5.1, U$2.25

Commit message: rekick 2015
Parts:
- moved CAP_330V 90.5 mm to (103.9, 10.0), turned to 270 degrees
- moved R20 88.0 mm to (147.1, 12.3), turned to 0 degrees
- moved R16 87.1 mm to (153.7, 20.8), turned to 270 degrees
- moved CAP_0V 84.3 mm to (137.4, 10.0), turned to 270 degrees
- moved COIL_OUT 82.7 mm to (115.1, 10.0), turned to 270 degrees
- moved COIL_IN 80.4 mm to (126.2, 10.0), turned to 270 degrees
- moved C25 78.3 mm to (149.0, 43.6)
- moved X2 73.8 mm to (68.6, 8.38)
- moved C10 67.9 mm to (35.2, 10.2)
- moved Q6 65.7 mm to (146.8, 25.9), turned to 180 degrees
- moved R200 64.8 mm to (65.2, 16.3), turned to 90 degrees
- moved Q2 63.6 mm to (140.2, 22.5), turned to 270 degrees
- moved Q5 61.5 mm to (67.9, 22.5), turned to 90 degrees
- moved U$7 61.1 mm to (120.7, 19.9), turned to 0 degrees
- moved D13 55.1 mm to (70.0, 15.7), turned to 270 degrees
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Connections:
- removed net ADC2: U$2.13
- removed net AN-AUSGANG-ODER-MCU-KOPPELN: RF_MAX.1
- removed net N$51: U5.4
- removed net ZU_CR_LR-KNOTEN: C13.1, C_ISEN_A.2, L4.2
- new net N$29: L3.1, L4.1, L7.9
- new net RF_MAX: RF_MAX.1, U$2.13
- net GND: now also IC2.3, IC2.4, IC2.6, IC2.7
- net N$50: now also U5.4
- net TRAFO1: now also L4.2; no longer L3.1, L7.9
- net TRAFO2: now also C13.1, C_ISEN_A.2; no longer L4.1

Commit message: rekick 2015
Parts:
- added C41: 2.2µ / 100V, rcl:C1210K
- added C42: 47µF/35V, rcl:PANASONIC_D
- added R51: 12k, rcl:R0805
- C10, C9: device rcl:E7,5-18 -> rcl:E5-13
- C13: value 2.2µ -> 2.2µ / 250V
- C25: device rcl:EB20D -> rcl:E5-10,5
- R19: value 47k -> 3k
- moved D17 571.5 mm to (96.8, 97.7)
- moved D16 562.8 mm to (96.8, 95.1)
- moved R50 509.8 mm to (88.0, 9.65), turned to 90 degrees
- moved LED10 499.8 mm to (88.0, 3.94), turned to 180 degrees
- moved LED9 494.7 mm to (90.6, 3.94), turned to 180 degrees
- moved R49 493.9 mm to (90.4, 9.65), turned to 90 degrees
- moved R45 423.1 mm to (26.5, 8.13), turned to 90 degrees
- moved R44 418.2 mm to (29.1, 8.13), turned to 90 degrees
- moved R43 413.2 mm to (31.6, 8.13), turned to 90 degrees
- moved R42 408.3 mm to (34.2, 8.13), turned to 90 degrees
- moved LED7 395.7 mm to (26.5, 2.54), turned to 180 degrees
- moved LED6 394.5 mm to (29.1, 2.54), turned to 180 degrees
- moved LED5 393.4 mm to (31.6, 2.54), turned to 180 degrees
- moved LED4 392.3 mm to (34.2, 2.54), turned to 180 degrees
- moved R41 380.9 mm to (93.1, 9.65), turned to 90 degrees
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Connections:
- net +24V: now also C42.+
- net GND: now also C42.-, R51.1; no longer H1.B3,0, H2.B3,0, H3.B3,0, H4.B3,0
- net GND1: now also C41.2
- net N$47: now also R51.2
- net TRAFO2: now also C41.1

Commit message: rekick 2015
Parts:
- added C43, C44, C45: 100n, rcl:C0603
- added R52: 10k, rcl:R0805
- added R53, R54: 100k, rcl:R0805
- C1, C2: device rcl:PANASONIC_D -> rcl:C0603
- IC3: device v-reg:SOT223 -> LM1117:SOT223
- moved R48 557.2 mm to (91.3, 96.9), turned to 90 degrees
- moved R47 520.3 mm to (42.4, 80.5), flipped to the bottom
- moved T5 515.5 mm to (37.3, 81.5), flipped to the bottom, turned to 180 degrees
- moved C40 471.0 mm to (34.7, 94.4), turned to 90 degrees
- moved D15 464.5 mm to (18.7, 84.7), turned to 180 degrees
- moved L1 451.2 mm to (25.9, 91.6), turned to 270 degrees
- moved LED8 450.7 mm to (80.6, 4.06), turned to 180 degrees
- moved R46 449.9 mm to (80.6, 9.65), turned to 90 degrees
- moved C3 449.6 mm to (6.22, 85.3), turned to 180 degrees
- moved U$8 435.3 mm to (20.7, 91.8), turned to 270 degrees
- moved JP3 413.4 mm to (34.8, 85.5)
- moved R30 340.6 mm to (83.6, 95.2)
- moved C39 338.3 mm to (83.3, 95.5)
- moved D14 335.1 mm to (83.1, 96.1)
- moved C38 302.9 mm to (99.8, 70.7)
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Connections:
- removed net ADC10: U$2.22
- removed net ADC3/INT0: U$2.14
- removed net ADC9: U$2.18
- removed net D2A/KICK_VOLTAGE: C36.1, IC4.2, R21.2, R5.1, U$2.25
- removed net N$68: C40.+, L1.1, R45.2, U$8.4
- removed net RF_MAX: RF_MAX.1, U$2.13
- new net D2A/RF_MAX: RF_MAX.1, U$2.25
- new net KICK_VOLTAGE: C36.1, IC4.2, R21.2, R5.1, R52.2
- new net OC0A/MOSI_A/KICK_VOLTAGE: R52.1, U$2.2
- net +3V3: now also C2.1, IC3.2; no longer C2.+, C26.2, C27.2
- net +5V: now also C1.1, C44.1, C45.1; no longer C1.+
- net +5V/1: now also C40.+, L1.1, R45.2, U$8.4
- net BURST: now also U$2.14
- net CAP_+12V: now also C43.1
- net CAP_-12V: now also C43.2
- net GND: now also C1.2, C2.2, C26.2, C27.2, C44.2, C45.2; no longer C1.-, C2.-
- net GND1: now also R54.2
- net N$16: now also R53.1
- net N$17: now also R54.1
- net NOTAUS: now also U$2.15
- net OC0A/MOSI_A: no longer U$2.2
- net STBY: now also U$2.13
- net TRAFO1: now also R53.2
Routing:
- net +5V: track 0.00 -> 156.6 mm, vias 0 -> 3
- net +5V/1: track 0.00 -> 149.0 mm, vias 0 -> 1
- net +24V: track 0.00 -> 145.1 mm, vias 0 -> 4
- net +3V3: track 0.00 -> 103.9 mm, vias 0 -> 3
- net BOOSTER_24V: track 0.00 -> 64.3 mm
- net GND1: track 0.00 -> 49.6 mm
- net N$57: track 0.00 -> 40.5 mm
- net +12V: track 0.00 -> 40.2 mm, vias 0 -> 1
- net ACTIVATE_BOOSTER: track 0.00 -> 39.4 mm
- net CAN_H: track 0.00 -> 31.8 mm
- net CAN_L: track 0.00 -> 25.4 mm
- net GND: track 0.00 -> 22.6 mm, vias 0 -> 1
- net N$54: track 0.00 -> 20.4 mm
- net SCK_3V: track 0.00 -> 19.7 mm
- net CLKOUT_ETH_3V: track 0.00 -> 18.1 mm, vias 0 -> 1
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