File: msl_electronic_boards/rekick2015/pcb/rekick2015-001.brd (EAGLE design)
At the start: 160 x 100 mm, 200 parts, among them IC1 LM1458D, IC2 4043D, IC3 LM1117, IC4 LM1458D, Q1 16MHz, Q2 IGW60T120, Q3 IPP023N10N5, Q4 IPP023N10N5, Q5 IPD90P04P4L, Q6 IRF840, T1 BC849, T2 BC849, T3 BC849, T4 BC849, U1 TXB0108PWR, U3 LM2675, U4 LM2675, U5 MC14025BDG

Commit message: rekick 2015
Parts:
- moved R_SS 39.6 mm to (29.7, 20.7), turned to 0 degrees
- moved T5 39.4 mm to (73.5, 97.0)
- moved CSS 39.3 mm to (29.7, 18.4)
- moved C13 36.1 mm to (89.2, 17.7)
- moved R47 34.4 mm to (74.5, 92.7), turned to 90 degrees
- moved JP3 34.1 mm to (67.3, 95.8), turned to 90 degrees
- moved R_LINE 30.0 mm to (29.7, 31.6), flipped to the top, turned to 0 degrees
- moved R_SS2 28.9 mm to (35.8, 20.7), turned to 180 degrees
- moved RF_MIN 28.4 mm to (29.7, 27.8)
- moved CF 24.7 mm to (35.8, 26.5), turned to 0 degrees
- moved C12 24.4 mm to (35.8, 29.1), turned to 0 degrees
- moved C_ISEN_B 24.2 mm to (31.0, 17.3), turned to 90 degrees
- moved C_DELAY 23.1 mm to (29.7, 23.0), turned to 0 degrees
- moved R48 21.9 mm to (110.2, 85.9)
- moved R_ISEN_B 21.2 mm to (33.5, 17.3), turned to 270 degrees
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Connections:
- new net FREI: U$2.16
- new net FREI2: U$2.27
- new net FREI3: U$2.15
- net ACTIVATE_BOOSTER: now also U$2.26; no longer U$2.24
- net ACTIVATE_SERVO: now also U$2.13; no longer U$2.16
- net ADC_CAP: now also U$2.14; no longer U$2.17
- net BURST: now also U$2.18; no longer U$2.14
- net NOTAUS: now also U$2.22; no longer U$2.15
- net RESET_NOTAUS: now also U$2.24; no longer U$2.26
- net STBY: now also U$2.17; no longer U$2.13
Routing:
- net CAP_-12V: track 0.00 -> 78.5 mm
- net CAP_+12V: track 0.00 -> 74.0 mm
- net CAP_330V: track 0.00 -> 60.9 mm, vias 0 -> 1
- net TRAFO2: track 0.00 -> 56.1 mm
- net N$24: track 0.00 -> 44.7 mm
- net ADC1/SCK_A: track 0.00 -> 39.5 mm, vias 0 -> 1
- net SERVO_PWM: track 0.00 -> 39.1 mm, vias 0 -> 2
- net CAN_RX: track 0.00 -> 37.8 mm, vias 0 -> 2
- net N$8: track 0.00 -> 36.0 mm
- net N$29: track 0.00 -> 35.3 mm
- net N$28: track 0.00 -> 32.7 mm, vias 0 -> 1
- net GND: track 22.6 -> 54.7 mm, vias 1 -> 4
- net RST: track 0.00 -> 31.3 mm, vias 0 -> 2
- net +12V: track 40.2 -> 70.7 mm, vias 1 -> 2
- net INT_ETH: track 3.56 -> 34.0 mm, vias 0 -> 1
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- added copper zone on layer 1, net CAP_0V
- added copper zone on layer 1, net CAP_330V
- added copper zone on layer 1, net GND1
- added copper zone on layer 1, net N$49
- added copper zone on layer 1, net TRAFO2

Commit message: rekick 2015
Parts:
- added C46: 100p, rcl:C0603
- moved T1 52.7 mm to (157.2, 49.3), flipped to the bottom, turned to 180 degrees
- moved R13 49.1 mm to (125.3, 82.9), flipped to the bottom
- moved R12 46.4 mm to (125.3, 80.6), flipped to the bottom
- moved R26 43.6 mm to (64.3, 52.8), turned to 180 degrees
- moved R15 43.4 mm to (155.4, 56.4), flipped to the bottom, turned to 180 degrees
- moved R14 39.3 mm to (153.3, 72.6), flipped to the bottom
- moved T4 36.3 mm to (69.1, 51.7)
- moved R25 35.9 mm to (64.3, 50.5)
- moved U$5 33.9 mm to (153.9, 64.9), turned to 270 degrees
- moved C44 29.5 mm to (119.3, 70.5), flipped to the bottom, turned to 0 degrees
- moved R18 29.5 mm to (146.7, 45.0)
- moved C38 29.3 mm to (125.3, 85.2), flipped to the bottom, turned to 180 degrees
- moved C37 25.3 mm to (119.3, 85.2), flipped to the bottom
- moved IC4 24.8 mm to (119.3, 74.3), flipped to the bottom, turned to 90 degrees
- moved R48 24.6 mm to (87.5, 95.1), flipped to the bottom, turned to 0 degrees
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Connections:
- net +12V: no longer R30.2
- net +24V: now also R30.2
- net CAP_0V: now also C46.2
- net GND: now also C38.2, R13.1
- net GND1: no longer C38.2, R13.1
- net N$27: now also C46.1
Routing:
- net +5V: track 182.2 -> 359.7 mm, vias 7 -> 10
- net CAP_0V: track 8.88 -> 146.6 mm, vias 0 -> 7
- net STBY: track 11.6 -> 119.2 mm, vias 0 -> 4
- net ADC_CAP: track 0.00 -> 85.4 mm, vias 0 -> 3
- net NOTAUS: track 0.00 -> 79.5 mm
- net ÜBERSPANNUNG: track 0.00 -> 76.8 mm, vias 0 -> 2
- net +24V: track 144.6 -> 208.3 mm, vias 3 -> 5
- net CAP_+12V: track 74.0 -> 135.4 mm, vias 0 -> 5
- net +5V/3: track 5.85 -> 61.2 mm, vias 0 -> 3
- net +5V/4: track 0.00 -> 47.3 mm, vias 0 -> 3
- net OC0A/MOSI_A/KICK_VOLTAGE: track 19.0 -> 64.6 mm, vias 1 -> 2
- net CAP_330V: track 60.9 -> 99.5 mm
- net CAP_-12V: track 78.5 -> 115.2 mm, vias 0 -> 1
- net N$50: track 0.00 -> 32.7 mm, vias 0 -> 2
- net N$53: track 0.00 -> 30.8 mm, vias 0 -> 2
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