File: msl_electronic_boards/rekick2015/pcb/rekick2015-003.brd (EAGLE design)
At the start: 160 x 100 mm, 200 parts, among them IC1 LM1458D, IC2 4043D, IC3 LM1117, IC4 LM1458D, Q1 16MHz, Q2 IGW60T120, Q3 IPP023N10N5, Q4 IPP023N10N5, Q5 IPD90P04P4L, Q6 IRF840, T1 BC849, T2 BC849, T3 BC849, T4 BC849, U1 TXB0108PWR, U3 LM2675, U4 LM2675, U5 MC14025BDG

Commit message: rekick 2015
Parts:
- moved C37 36.0 mm to (150.6, 79.5)
- moved R28 36.0 mm to (150.6, 77.2)
- moved R5 36.0 mm to (150.6, 72.6), turned to 0 degrees
- moved R27 36.0 mm to (150.6, 74.9)
- moved C33 23.1 mm to (100.5, 91.3), flipped to the top, turned to 90 degrees
- moved IC2 21.8 mm to (100.8, 87.1), turned to 90 degrees
- moved R22 21.2 mm to (98.2, 91.3), flipped to the top, turned to 270 degrees
- moved C45 20.8 mm to (100.8, 85.1), turned to 90 degrees
- moved C38 19.2 mm to (132.3, 78.7), turned to 90 degrees
- moved C42 18.6 mm to (106.7, 72.6), turned to 180 degrees
- moved R13 18.3 mm to (134.6, 78.7), turned to 270 degrees
- moved R12 17.8 mm to (136.9, 78.7), turned to 90 degrees
- moved D14 16.2 mm to (109.5, 97.4)
- moved R30 16.2 mm to (106.6, 97.4)
- moved C39 16.2 mm to (112.4, 97.3)
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Routing:
- net CAP_-12V: track 13.8 -> 149.2 mm, vias 1 -> 3
- net CAP_+12V: track 17.9 -> 149.3 mm, vias 1 -> 3
- net +5V: track 276.1 -> 211.9 mm, vias 10 -> 7
- net STBY: track 116.7 -> 57.5 mm, vias 3 -> 2
- net ADC_CAP: track 47.3 -> 8.85 mm
- net NOTAUS: track 66.5 -> 32.9 mm, vias 2 -> 1
- net BURST: track 54.8 -> 24.1 mm, vias 2 -> 1
- net +5V/4: track 22.3 -> 48.2 mm
- net TASTER: track 23.1 -> 0.00 mm
- net CAP_330V: track 123.5 -> 140.5 mm
- net N$58: track 51.3 -> 34.6 mm, vias 1 -> 0
- net ÜBERSPANNUNG: track 15.0 -> 0.00 mm, vias 2 -> 0
- net RESET_NOTAUS: track 39.8 -> 24.9 mm
- net N$37: track 13.5 -> 0.00 mm
- net N$38: track 11.4 -> 0.00 mm
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- added copper zone on layer 1, net CAP_0V
- added copper zone on layer 16, net CAP_0V
