File: msl_electronic_boards/rekick2015/pcb/rekick2015-Prototyp.brd (EAGLE design)
At the start: 160 x 100 mm, 200 parts, among them IC1 LM1458D, IC2 4043D, IC3 LM1117, IC4 LM1458D, Q1 16MHz, Q2 IGW60T120, Q3 IPP023N10N5, Q4 IPP023N10N5, Q5 IPD90P04P4L, Q6 IRF840, T1 BC849, T2 BC849, T3 BC849, T4 BC849, U1 TXB0108PWR, U3 LM2675, U4 LM2675, U5 MC14025BDG

Commit message: rekick2015 Prototyp
Routing:
- net N$14: track 43.8 -> 44.6 mm
- net GND1: vias 0 -> 3
- net CAP_0V: vias 3 -> 9
Changed lines of the file:
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@@
 <vertex x="75.311" y="47.498"/>
 <vertex x="95.123" y="67.31"/>
-<vertex x="115.443" y="67.31"/>
-<vertex x="115.443" y="57.912"/>
-<vertex x="138.938" y="57.912"/>
-<vertex x="138.938" y="64.008"/>
-<vertex x="160.02" y="64.008"/>
+<vertex x="116.078" y="67.31"/>
+<vertex x="116.078" y="58.547"/>
+<vertex x="138.811" y="58.547"/>
+<vertex x="138.811" y="64.77"/>
+<vertex x="160.02" y="64.77"/>
 <vertex x="160.02" y="100.076"/>
 <vertex x="0" y="100.076"/>
@@
 <vertex x="75.311" y="47.498"/>
 <vertex x="95.123" y="67.31"/>
-<vertex x="115.443" y="67.31"/>
-<vertex x="115.443" y="65.024"/>
-<vertex x="160.02" y="65.024"/>
+<vertex x="116.078" y="67.31"/>
+<vertex x="116.078" y="64.77"/>
+<vertex x="160.02" y="64.77"/>
 <vertex x="160.02" y="100.076"/>
 <vertex x="0" y="100.076"/>
@@
 <wire x1="74.158" y1="16.51" x2="74.158" y2="7.6554" width="1.778" layer="1"/>
 <wire x1="74.158" y1="7.6554" x2="74.1934" y2="7.62" width="1.778" layer="1"/>
-<polygon width="0.254" layer="16" rank="2">
+<polygon width="0.254" layer="16" isolate="0.4064" rank="2">
 <vertex x="42.799" y="0"/>
-<vertex x="95.123" y="0"/>
-<vertex x="95.123" y="67.31"/>
+<vertex x="94.488" y="0"/>
+<vertex x="94.488" y="66.675"/>
 <vertex x="75.311" y="47.498"/>
 <vertex x="51.435" y="47.498"/>
 <vertex x="42.799" y="38.862"/>
 </polygon>
-<polygon width="0.254" layer="1">
+<polygon width="0.254" layer="1" isolate="0.4064">
 <vertex x="42.799" y="0"/>
-<vertex x="95.123" y="0"/>
-<vertex x="95.123" y="67.31"/>
+<vertex x="94.488" y="0"/>
+<vertex x="94.488" y="66.675"/>
 <vertex x="75.311" y="47.498"/>
 <vertex x="51.435" y="47.498"/>
 <vertex x="42.799" y="38.862"/>
 </polygon>
+<via x="49.784" y="27.178" extent="1-16" drill="0.6"/>
+<via x="49.149" y="21.463" extent="1-16" drill="0.6"/>
+<via x="45.72" y="13.843" extent="1-16" drill="0.6"/>
 </signal>
 <signal name="BOOSTER_24V">
@@
 <contactref element="IC1" pad="2"/>
 <wire x1="153.67" y1="33.849" x2="153.67" y2="32.385" width="0.254" layer="16"/>
-<wire x1="153.67" y1="32.385" x2="154.051" y2="32.004" width="0.254" layer="16"/>
-<wire x1="154.051" y1="32.004" x2="156.337" y2="32.004" width="0.254" layer="16"/>
-<wire x1="156.337" y1="32.004" x2="156.972" y2="32.639" width="0.254" layer="16"/>
-<wire x1="156.972" y1="32.639" x2="156.972" y2="44.262" width="0.254" layer="16"/>
+<wire x1="153.67" y1="32.385" x2="154.178" y2="31.877" width="0.254" layer="16"/>
+<wire x1="154.178" y1="31.877" x2="156.718" y2="31.877" width="0.254" layer="16"/>
 <wire x1="156.972" y1="44.262" x2="157.033" y2="44.323" width="0.254" layer="16"/>
 <wire x1="157.033" y1="44.323" x2="157.033" y2="46.509" width="0.254" layer="16"/>
@@
 <wire x1="153.543" y1="61.087" x2="153.543" y2="59.016" width="0.254" layer="16"/>
 <wire x1="153.543" y1="59.016" x2="156.933" y2="55.626" width="0.254" layer="16"/>
+<wire x1="156.972" y1="44.262" x2="157.48" y2="43.754" width="0.254" layer="16"/>
+<wire x1="157.48" y1="43.754" x2="157.48" y2="32.639" width="0.254" layer="16"/>
+<wire x1="157.48" y1="32.639" x2="156.718" y2="31.877" width="0.254" layer="16"/>
 </signal>
 <signal name="N$21">
@@
 <via x="112.649" y="65.532" extent="1-16" drill="0.6"/>
 <via x="112.522" y="58.42" extent="1-16" drill="0.6"/>
-<wire x1="121.158" y1="10.033" x2="121.158" y2="14.605" width="2.1844" layer="1"/>
+<wire x1="121.158" y1="10.033" x2="121.158" y2="14.478" width="2.1844" layer="1"/>
+<wire x1="121.158" y1="14.478" x2="121.158" y2="14.605" width="2.1844" layer="1"/>
 <wire x1="121.158" y1="14.605" x2="124.587" y2="18.034" width="2.1844" layer="1"/>
 <wire x1="124.587" y1="18.034" x2="124.587" y2="23.368" width="2.1844" layer="1"/>
 <polygon width="0.254" layer="1" isolate="1.016">
-<vertex x="160.02" y="64.389"/>
+<vertex x="160.02" y="63.5"/>
 <vertex x="160.02" y="0"/>
 <vertex x="95.758" y="0"/>
-<vertex x="95.758" y="66.675"/>
-<vertex x="114.808" y="66.675"/>
-<vertex x="114.808" y="64.389"/>
+<vertex x="95.758" y="66.04"/>
+<vertex x="114.808" y="66.04"/>
+<vertex x="114.808" y="63.5"/>
 </polygon>
 <polygon width="0.254" layer="16" isolate="1.016">
@@
 <vertex x="160.02" y="0"/>
 <vertex x="95.758" y="0"/>
-<vertex x="95.758" y="66.675"/>
-<vertex x="114.808" y="66.675"/>
+<vertex x="95.758" y="66.04"/>
+<vertex x="114.808" y="66.04"/>
 <vertex x="114.808" y="57.277"/>
-<vertex x="139.573" y="57.277"/>
-<vertex x="139.573" y="63.373"/>
+<vertex x="140.208" y="57.277"/>
+<vertex x="140.208" y="63.373"/>
 </polygon>
 <wire x1="143.129" y1="61.6966" x2="143.129" y2="59.436" width="0.254" layer="16"/>
 <polygon width="0.254" layer="1">
-<vertex x="95.758" y="66.675"/>
+<vertex x="95.758" y="66.04"/>
 <vertex x="95.758" y="1.143"/>
 <vertex x="113.03" y="1.143"/>
@@
 <vertex x="126.238" y="57.277"/>
 <vertex x="126.238" y="47.371"/>
-<vertex x="140.208" y="47.371"/>
-<vertex x="140.208" y="57.277"/>
-<vertex x="149.479" y="57.277"/>
-<vertex x="149.479" y="19.177"/>
+<vertex x="140.843" y="47.371"/>
+<vertex x="140.843" y="57.277"/>
+<vertex x="147.701" y="57.277"/>
+<vertex x="147.701" y="19.177"/>
 <vertex x="160.02" y="19.177"/>
-<vertex x="160.02" y="64.389"/>
-<vertex x="114.808" y="64.389"/>
-<vertex x="114.808" y="66.675"/>
+<vertex x="160.02" y="63.5"/>
+<vertex x="114.808" y="63.5"/>
+<vertex x="114.808" y="66.04"/>
 </polygon>
 <polygon width="0.254" layer="16">
-<vertex x="149.479" y="57.277"/>
-<vertex x="149.479" y="19.177"/>
+<vertex x="147.701" y="57.277"/>
+<vertex x="147.701" y="19.177"/>
 <vertex x="160.02" y="19.177"/>
-<vertex x="160.02" y="63.373"/>
-<vertex x="139.573" y="63.373"/>
-<vertex x="139.573" y="57.277"/>
+<vertex x="160.02" y="63.5"/>
+<vertex x="140.208" y="63.5"/>
+<vertex x="140.208" y="57.277"/>
 <vertex x="126.238" y="57.277"/>
 <vertex x="126.238" y="47.371"/>
-<vertex x="140.208" y="47.371"/>
-<vertex x="140.208" y="57.277"/>
+<vertex x="140.843" y="47.371"/>
+<vertex x="140.843" y="57.277"/>
 </polygon>
 <via x="155.956" y="42.672" extent="1-16" drill="0.6"/>
 <polygon width="0.254" layer="16">
 <vertex x="114.808" y="57.277"/>
-<vertex x="114.808" y="66.675"/>
-<vertex x="95.758" y="66.675"/>
+<vertex x="114.808" y="66.04"/>
+<vertex x="95.758" y="66.04"/>
 <vertex x="95.758" y="1.143"/>
 <vertex x="113.03" y="1.143"/>
@@
 <vertex x="110.109" y="57.277"/>
 </polygon>
+<via x="152.908" y="50.038" extent="1-16" drill="0.6"/>
+<via x="97.409" y="2.794" extent="1-16" drill="0.6"/>
+<via x="121.158" y="14.478" extent="1-16" drill="0.6"/>
+<via x="118.364" y="14.478" extent="1-16" drill="0.6"/>
+<via x="123.825" y="14.478" extent="1-16" drill="0.6"/>
+<via x="156.972" y="58.674" extent="1-16" drill="0.6"/>
 </signal>
 <signal name="CAP_+12V">
@@
 <contactref element="R9" pad="2"/>
 <contactref element="OK2" pad="1"/>
-<wire x1="151.765" y1="58.547" x2="151.765" y2="54.163" width="0.254" layer="16"/>
+<wire x1="151.765" y1="58.293" x2="151.765" y2="54.163" width="0.254" layer="16"/>
 <wire x1="144.399" y1="61.6966" x2="144.399" y2="59.69" width="0.254" layer="16"/>
 <wire x1="144.399" y1="59.69" x2="145.034" y2="59.055" width="0.254" layer="16"/>
-<wire x1="145.034" y1="59.055" x2="151.257" y2="59.055" width="0.254" layer="16"/>
-<wire x1="151.257" y1="59.055" x2="151.765" y2="58.547" width="0.254" layer="16"/>
+<wire x1="145.034" y1="59.055" x2="151.003" y2="59.055" width="0.254" layer="16"/>
+<wire x1="151.003" y1="59.055" x2="151.765" y2="58.293" width="0.254" layer="16"/>
 </signal>
 <signal name="N$30">

Commit message: rekick2015 little changes
Parts:
- removed R31: 20k, rcl:R0805
Connections:
- net ACTIVATE_BOOSTER: no longer R31.2
- net GND1: no longer R31.1
Routing:
- net ACTIVATE_BOOSTER: track 80.2 -> 69.7 mm
- net CAP_0V: track 36.0 -> 37.0 mm
Changed lines of the file:
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@@
 <?xml version="1.0" encoding="utf-8"?>
 <!DOCTYPE eagle SYSTEM "eagle.dtd">
-<eagle version="7.5.0">
+<eagle version="7.2.0">
 <drawing>
 <settings>
@@
 <element name="R30" library="rcl" package="R0805" value="1k" x="102.743" y="76.835" rot="MR90"/>
 <element name="C7" library="rcl" package="C0603" value="100n" x="64.135" y="59.436" rot="MR180"/>
-<element name="R31" library="rcl" package="R0805" value="20k" x="69.215" y="16.129" rot="MR270"/>
 <element name="H1" library="holes" package="3,0-PAD" value="MOUNT-PAD-ROUND3.0" x="155.575" y="4.445"/>
 <element name="H2" library="holes" package="3,0-PAD" value="MOUNT-PAD-ROUND3.0" x="155.575" y="96.012"/>
@@
 <contactref element="LED8" pad="C"/>
 <contactref element="R54" pad="2"/>
-<contactref element="R31" pad="1"/>
 <wire x1="43.053" y1="4.699" x2="53.594" y2="4.699" width="2.1844" layer="16"/>
 <wire x1="53.594" y1="4.699" x2="57.531" y2="4.699" width="2.1844" layer="16"/>
@@
 <contactref element="R50" pad="2"/>
 <contactref element="C46" pad="2"/>
-<wire x1="121.412" y1="34.653" x2="124.605" y2="31.46" width="1.016" layer="16"/>
-<wire x1="124.605" y1="31.46" x2="124.605" y2="27.686" width="1.016" layer="16"/>
+<wire x1="124.605" y1="33.129" x2="124.605" y2="27.686" width="1.016" layer="16"/>
 <wire x1="124.605" y1="27.686" x2="124.587" y2="27.668" width="1.016" layer="16"/>
 <wire x1="124.587" y1="27.668" x2="124.587" y2="23.368" width="1.016" layer="16"/>
@@
 <via x="123.825" y="14.478" extent="1-16" drill="0.6"/>
 <via x="156.972" y="58.674" extent="1-16" drill="0.6"/>
+<wire x1="124.605" y1="33.129" x2="123.063" y2="34.671" width="1.016" layer="16"/>
+<wire x1="123.063" y1="34.671" x2="121.412" y2="34.671" width="1.016" layer="16"/>
+<wire x1="121.412" y1="34.653" x2="121.412" y2="34.671" width="1.016" layer="16"/>
 </signal>
 <signal name="CAP_+12V">
@@
 <contactref element="R24" pad="1"/>
 <contactref element="R25" pad="1"/>
-<contactref element="R31" pad="2"/>
 <contactref element="U$2" pad="26"/>
 <wire x1="55.1478875" y1="60.828459375" x2="53.882428125" y2="59.563" width="0.254" layer="16"/>
@@
 <wire x1="47.752" y1="14.859" x2="48.768" y2="13.843" width="0.254" layer="1"/>
 <wire x1="48.768" y1="13.843" x2="59.69" y2="13.843" width="0.254" layer="1"/>
-<wire x1="71.501" y1="15.179" x2="69.215" y2="15.179" width="0.3048" layer="16"/>
-<wire x1="69.215" y1="15.179" x2="61.026" y2="15.179" width="0.254" layer="16"/>
 <wire x1="61.026" y1="15.179" x2="59.69" y2="13.843" width="0.254" layer="16"/>
 <via x="59.69" y="13.843" extent="1-16" drill="0.6"/>
+<wire x1="61.026" y1="15.179" x2="71.501" y2="15.179" width="0" layer="19" extent="16-16"/>
 </signal>
 <signal name="KICK">

Commit message: rekick2015
Parts:
- removed T1: BC849, transistor:SOT23
- removed U5: MC14025BDG, MC14025BDG:SOIC127P600X175-14N
- added C41, C47: 100n, rcl:C0603
- added R31: 50k, rcl:R0805
- added R55, R56, R57, R58: 5,6k, rcl:R0805
- added R59: 11k, rcl:R0805
- added T6: BC859, transistor:SOT23-BEC
- added U2: SN74LVC2G02DCTR, SN74LVC2G02DCTR:SOP65P400X130-8N
- C14, C15, C23, C24, C36, C46: value 100p -> 100n
- C30: device rcl:PANASONIC_D -> rcl:E2-5
- C31: value 1µ -> 47µF/35V; device rcl:C0603 -> rcl:E2-5
- C32: value 1µ -> 100n
- C37, C38: value 100p -> 1µ/25V; device rcl:C0603 -> rcl:SMC_A
- D5: value SMD ZD 15 -> ES1A; device diode:TO236 -> diode:SMA-DO214AC
- R10, R47: value 1k -> 5,6k
- R105: value 750 -> 680
- R11, R8: value 2k, 1% -> 10k, 1%
- R12: value 68k -> 10k
- R13: value 10k -> 5
- R15: value 10 -> 10k
- R16: value 470k -> 50k; device rcl:0207/15 -> rcl:R0805
- R18: value 10 -> 5
- R19: value 3k -> 5,6k
- R20: value B72220S0321K101 -> ERZE07A621; device varistor:S20K320 -> varistor:S10K385
- R21: value 10k, 1% -> 33k, 1%
- R24, R28: value 10k -> 5,6k
- R25: value 10k -> 100k
- R26, R27: value 10k -> 50k
- R30: value 1k -> 3.3k
- R4: value 10k, 1% -> 24k, 1%
- R46: value 680 -> 11k
- R5: value 3k, 1% -> 10k, 1%
- R50: value 4.7k -> 5,6k
- R51: value 12k -> 50k
- R52: value 10k -> 10k, 1%
- R7: value 2.37k, 1% -> 5.6k, 1%
- moved LED10 87.8 mm to (13.0, 7.49), turned to 0 degrees
- moved R27 84.5 mm to (70.1, 49.3), flipped to the top, turned to 180 degrees
- moved R28 81.8 mm to (69.7, 65.0), flipped to the top
- moved R16 81.0 mm to (64.3, 83.7), turned to 0 degrees
- moved R50 65.9 mm to (69.6, 68.5), turned to 0 degrees
- moved C37 39.7 mm to (111.0, 76.8), turned to 90 degrees
- moved R12 36.2 mm to (137.5, 41.5), turned to 270 degrees
- moved R13 36.1 mm to (133.0, 41.5)
- moved C30 32.5 mm to (136.7, 53.1)
- moved C38 31.9 mm to (140.2, 47.2), flipped to the top, turned to 270 degrees
- moved R52 23.4 mm to (150.6, 75.2), turned to 0 degrees
- moved R21 20.2 mm to (150.6, 77.5), turned to 0 degrees
- moved C32 19.4 mm to (149.4, 48.0), turned to 270 degrees
- moved C36 17.0 mm to (150.6, 79.8), turned to 180 degrees
- moved C14 15.1 mm to (153.2, 61.5), turned to 180 degrees
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Connections:
- removed net ADC1/SCK_A: SV1.7, U$2.12
- removed net CAP_-12V: C30.-, C43.2, IC1.4, LED10.C, U$4.4
- removed net FREI3: U$2.15
- new net 24V_PRI: C10.+, C35.1, C9.+, Q3.D, Q5.4, R23.2, R27.2
- new net ADC_24V_LOGIK/SCK_A: R31.2, R50.1, SV1.7, U$2.12
- new net ADC_24V_PRI: R27.1, R28.2, U$2.13
- new net N$51: R55.1, U$2.22
- new net N$68: R58.1, U$2.3
- net +24V: now also R31.1
- net +5V: now also U2.8; no longer U5.14
- net +5V/3: now also C37.+; no longer R27.2
- net +5V/4: now also C38.+
- net ACTIVATE_SERVO: now also U$2.15; no longer U$2.13
- net ADC_CAP: now also C47.1
- net BOOSTER_24V: no longer R12.2
- net BURST: now also U2.3; no longer U$2.18, U5.6
- net CAP_+12V: now also C30.+, C31.+, T6.E; no longer C31.1, C32.1
- net CAP_0V: now also C30.-, C31.-, C38.-, C43.2, IC1.4, U$4.4; no longer C30.+, C31.2, D5.A, R50.2, T1.2, U$4.5
- net CAP_330V: no longer R16.2
- net GND: now also C37.-, C41.2, C47.2, LED10.C, R16.1, R50.2; no longer C37.2, C38.2, R13.1, U5.11, U5.13, U5.5, U5.7, U5.8
- net N$15: now also C32.1
- net N$30: now also R59.2
- net N$37: now also U2.1; no longer U5.1
- net N$38: now also U2.5; no longer U5.3
- net N$39: now also Q6.G, R12.2, T6.C; no longer C38.1, IC4.6, R12.1, R13.2
- net N$44: now also D5.K
- net N$45: now also R56.2; no longer D5.C, Q6.G, R16.1, T1.3
- net N$46: now also T6.B; no longer T1.1
- net N$48: now also R13.2
- net N$50: now also U2.6; no longer U5.4
- net N$53: now also D5.A, R13.1; no longer IC4.7, U5.12
- net N$57: now also R56.1, U$2.18; no longer C10.+, C35.1, C9.+, Q3.D, Q5.4, R23.2
- net N$58: now also U2.2; no longer U5.2
- net N$59: now also R57.1, U$2.17; no longer C37.1, IC4.5, R27.1, R28.2
- net N$75: now also R16.2
- net N$77: now also R59.1; no longer R50.1
- net NOTAUS: now also R55.2, U2.7; no longer U$2.22, U5.9
- net SERVO_PWM: now also R58.2; no longer U$2.3
- net STBY: now also R57.2; no longer U$2.17
- net ÜBERSPANNUNG: now also C41.1
Routing:
- net CAP_-12V: track 149.4 -> 0.00 mm, vias 3 -> 0
- net BOOSTER_24V: track 147.0 -> 29.8 mm, vias 2 -> 0
- net N$53: track 60.9 -> 3.59 mm, vias 2 -> 0
- net N$50: track 78.0 -> 31.9 mm, vias 4 -> 1
- net N$57: track 40.6 -> 0.00 mm
- net 24V_PRI: track 0.00 -> 40.6 mm
- net ADC_24V_LOGIK/SCK_A: track 0.00 -> 39.5 mm, vias 0 -> 1
- net ADC1/SCK_A: track 39.5 -> 0.00 mm, vias 1 -> 0
- net KICK_VOLTAGE: track 39.3 -> 12.0 mm
- net N$45: track 21.8 -> 0.00 mm
- net N$59: track 15.0 -> 0.00 mm
- net N$39: track 22.2 -> 8.06 mm, vias 2 -> 0
- net OC0A/MOSI_A/KICK_VOLTAGE: track 95.6 -> 109.2 mm
- net ACTIVATE_SERVO: track 20.0 -> 7.11 mm
- net N$38: track 28.3 -> 16.2 mm, vias 2 -> 0
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
Commit message: rekick2015
Parts:
- moved R31 63.9 mm to (11.2, 50.3), flipped to the bottom
- moved R50 29.4 mm to (44.3, 53.5), flipped to the bottom, turned to 315 degrees
- moved R58 13.7 mm to (51.3, 80.3), flipped to the bottom, turned to 90 degrees
- moved R55 11.1 mm to (70.5, 56.0), flipped to the bottom, turned to 180 degrees
- moved R59 9.67 mm to (7.11, 11.0)
- moved C6 9.25 mm to (58.2, 64.5), flipped to the top, turned to 225 degrees
- moved R28 8.52 mm to (66.2, 72.8), flipped to the bottom
- moved C47 8.32 mm to (75.7, 74.4), flipped to the bottom, turned to 270 degrees
- moved R56 7.65 mm to (71.0, 62.0), flipped to the bottom, turned to 180 degrees
- moved R57 7.58 mm to (71.0, 64.3), flipped to the bottom, turned to 180 degrees
- moved R27 5.35 mm to (64.8, 49.7)
- moved R24 5.08 mm to (66.4, 16.3), turned to 270 degrees
- moved LED10 4.46 mm to (12.6, 3.05), turned to 180 degrees
- moved R16 3.99 mm to (67.9, 85.2), flipped to the bottom, turned to 90 degrees
- moved R22 2.41 mm to (100.2, 94.5), turned to 180 degrees
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Connections:
- removed net N$45: R56.2
- net BURST: now also R56.2
Routing:
- net OC0A/MOSI_A/KICK_VOLTAGE: track 109.2 -> 36.4 mm, vias 4 -> 1
- net ACTIVATE_BOOSTER: track 69.7 -> 0.00 mm, vias 4 -> 0
- net N$58: track 47.7 -> 3.89 mm, vias 1 -> 0
- net N$50: track 31.9 -> 73.3 mm, vias 1 -> 2
- net BURST: track 46.3 -> 8.66 mm
- net NOTAUS: track 107.4 -> 79.4 mm, vias 3 -> 2
- net STBY: track 98.3 -> 76.4 mm
- net +5V/3: track 103.5 -> 81.7 mm
- net ADC_24V_LOGIK/SCK_A: track 39.5 -> 60.8 mm, vias 1 -> 3
- net ADC_CAP: track 107.5 -> 89.4 mm, vias 6 -> 2
- net SERVO_PWM: track 30.9 -> 16.2 mm, vias 2 -> 0
- net N$68: track 0.00 -> 12.9 mm, vias 0 -> 2
- net GND: track 51.8 -> 38.9 mm
- net RESET_NOTAUS: track 81.0 -> 70.0 mm, vias 4 -> 3
- net ACTIVATE_SERVO: track 7.11 -> 0.00 mm
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
Commit message: rekick2015
Parts:
- removed R_SS2: (no value), rcl:R0805
Connections:
- removed net N$7: CSS.1, R_SS.1, R_SS2.1
- net N$18: now also CSS.1, R_SS.1; no longer R_SS2.2
Routing:
- net N$7: track 6.52 -> 0.00 mm
- net N$18: track 6.86 -> 3.49 mm
Changed lines of the file:
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@@
 <?xml version="1.0" encoding="utf-8"?>
 <!DOCTYPE eagle SYSTEM "eagle.dtd">
-<eagle version="7.5.0">
+<eagle version="7.2.0">
 <drawing>
 <settings>
@@
 <element name="C12" library="rcl" package="C0603" value="" x="35.814" y="29.083" rot="MR0"/>
 <element name="C_BOOT" library="rcl" package="C0603" value="100n" x="49.276" y="24.511" rot="MR90"/>
-<element name="R_SS2" library="rcl" package="R0805" value="" x="35.814" y="20.701" rot="MR180"/>
 <element name="R_DELAY" library="rcl" package="R0805" value="" x="29.718" y="25.273" rot="MR180"/>
 <element name="C_DELAY" library="rcl" package="C0603" value="" x="29.718" y="22.987" rot="MR0"/>
@@
 <vertex x="138.811" y="64.77"/>
 <vertex x="160.02" y="64.77"/>
-<vertex x="160.02" y="100.076"/>
+<vertex x="160.02" y="92.075"/>
+<vertex x="119.888" y="92.075"/>
+<vertex x="119.888" y="100.076"/>
 <vertex x="0" y="100.076"/>
 </polygon>
@@
 <vertex x="116.078" y="64.77"/>
 <vertex x="160.02" y="64.77"/>
-<vertex x="160.02" y="100.076"/>
+<vertex x="160.02" y="92.075"/>
+<vertex x="119.888" y="92.075"/>
+<vertex x="119.888" y="100.076"/>
 <vertex x="0" y="100.076"/>
 </polygon>
@@
 <via x="43.307" y="27.813" extent="1-16" drill="0.6"/>
 </signal>
-<signal name="N$7">
-<contactref element="R_SS" pad="1"/>
-<contactref element="CSS" pad="1"/>
-<contactref element="R_SS2" pad="1"/>
-<wire x1="30.668" y1="20.701" x2="34.864" y2="20.701" width="0.254" layer="16"/>
-<wire x1="30.668" y1="20.701" x2="30.568" y2="20.601" width="0.254" layer="16"/>
-<wire x1="30.568" y1="20.601" x2="30.568" y2="18.415" width="0.254" layer="16"/>
-</signal>
 <signal name="N$11">
 <contactref element="U$3" pad="3"/>
@@
 <signal name="N$18">
 <contactref element="U$3" pad="1"/>
-<contactref element="R_SS2" pad="2"/>
-<wire x1="36.764" y1="20.701" x2="40.132" y2="20.701" width="0.254" layer="16"/>
 <wire x1="40.132" y1="20.701" x2="40.513" y2="21.082" width="0.254" layer="16"/>
 <wire x1="40.513" y1="21.082" x2="40.513" y2="23.936" width="0.254" layer="16"/>
 <wire x1="40.513" y1="23.936" x2="40.58" y2="24.003" width="0.254" layer="16"/>
+<contactref element="CSS" pad="1"/>
+<contactref element="R_SS" pad="1"/>
+<wire x1="30.668" y1="20.701" x2="40.132" y2="20.701" width="0" layer="19" extent="16-16"/>
+<wire x1="30.568" y1="18.415" x2="30.668" y2="20.701" width="0" layer="19" extent="16-16"/>
 </signal>
 <signal name="N$8">
