File: msl_electronic_boards/rekick2015/pcb/rekick2015-Prototyp.brd (EAGLE design)
At the start: 160 x 100 mm, 206 parts, among them IC1 LM1458D, IC2 4043D, IC3 LM1117, IC4 LM1458D, Q1 16MHz, Q2 IGW60T120, Q3 IPP023N10N5, Q4 IPP023N10N5, Q5 IPD90P04P4L, Q6 IRF840, T2 BC849, T3 BC849, T4 BC849, T6 BC859, U1 TXB0108PWR, U2 SN74LVC2G02DCTR, U3 LM2675, U4 LM2675

Commit message: rekick2015 finished prototyp
Parts:
- removed D16, D17: ES1A, diode:SMA-DO214AC
- removed R56: 5,6k, rcl:R0805
- added C48: 100n, rcl:C0603
- added C49: 10µ, rcl:C0603
- added C50: 1µ/50V, rcl:C1206
- added JP4: (no value), pinhead:1X03
- added R61: 5,6k, rcl:R0805
- added T1, T8: BC849, transistor:SOT23
- C12: value (none) -> 100n
- C35: device rcl:C0603 -> rcl:C1206
- R48: value 10k -> 5,6k
- R52: value 10k, 1% -> 5,6k, 1%
- R58: value 5,6k -> 10k
- moved R48 66.9 mm to (30.4, 53.3), turned to 90 degrees
- moved R58 41.5 mm to (92.5, 85.6), flipped to the top
- moved R27 20.6 mm to (44.3, 52.5), turned to 270 degrees
- moved R31 11.9 mm to (11.2, 38.4)
- moved C47 9.52 mm to (66.3, 72.9), flipped to the top, turned to 180 degrees
- moved T5 7.96 mm to (72.1, 88.4)
- moved JP3 7.91 mm to (69.6, 91.9)
- moved R55 6.54 mm to (64.0, 56.9), turned to 225 degrees
- moved RF_MAX 5.75 mm to (33.4, 39.2)
- moved D14 5.61 mm to (106.3, 71.2)
- moved R30 5.61 mm to (103.3, 71.2)
- moved C37 5.61 mm to (111.5, 71.2)
- moved C39 5.61 mm to (109.3, 71.2)
- moved R57 4.89 mm to (66.5, 62.2), turned to 135 degrees
- moved R25 4.55 mm to (50.7, 52.8)
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- renumbered R_LINE to R70
Connections:
- removed net 1.25V-BIS-6V: R70.2, U$3.7
- removed net BURST: D17.K, R56.2, U2.3
- removed net D2A/RF_MAX: RF_MAX.1, U$2.25
- removed net N$57: R56.1, U$2.18
- removed net N$68: R58.1, U$2.3
- removed net OC0A/MOSI_A/KICK_VOLTAGE: R52.1, U$2.2
- removed net OC1A/MISO_A: SV1.9, U$2.1
- new net ADC9/FREI: U$2.18
- new net D2A: R52.1, U$2.25
- new net LINE: C48.1, R70.2, T1.3, T2.3, U$3.7, U$6.3
- new net N$7: RF_MAX.1, T8.3
- new net N$78: R61.2, T1.1
- new net N$79: C49.1, R48.2, T8.1
- new net OC1A_FREQ/MISO_A: R48.1, SV1.9, U$2.1
- net +5V: now also R58.2; no longer R48.2
- net +5V/1: now also JP4.2
- net 24V_PRI: now also C50.1
- net CAP_0V: now also R12.1
- net GND: now also C48.2, C49.2, H2.B3,0, H3.B3,0, H4.B3,0, IC4.5, IC4.6, JP4.3, T1.2, T8.2, U2.4
- net GND1: now also C50.2
- net N$42: now also IC2.5, R58.1; no longer T2.3, U$6.3
- net NOTAUS: now also R61.1; no longer D16.K
- net OC0A/MOSI_A: now also JP4.1, U$2.2
- net SERVO_PWM: now also U$2.3; no longer R58.2
- net STBY: now also U2.3; no longer D16.A, D17.A, R48.1
Routing:
- net LINE: track 0.00 -> 130.6 mm, vias 0 -> 2
- net D2A: track 0.00 -> 110.6 mm, vias 0 -> 4
- net OC0A/MOSI_A: track 0.00 -> 68.2 mm, vias 0 -> 2
- net ACTIVATE_BOOSTER: track 0.00 -> 56.1 mm, vias 0 -> 2
- net NOTAUS: track 79.4 -> 135.3 mm, vias 2 -> 3
- net N$58: track 3.89 -> 46.7 mm, vias 0 -> 1
- net 24V_PRI: track 40.6 -> 81.2 mm, vias 0 -> 4
- net OC0A/MOSI_A/KICK_VOLTAGE: track 36.4 -> 0.00 mm, vias 1 -> 0
- net ADC_24V_PRI: track 0.00 -> 34.6 mm, vias 0 -> 1
- net OC1A_FREQ/MISO_A: track 0.00 -> 33.9 mm, vias 0 -> 1
- net OC1A/MISO_A: track 29.7 -> 0.00 mm, vias 2 -> 0
- net D2A/RF_MAX: track 24.5 -> 0.00 mm
- net +5V/3: track 81.7 -> 104.3 mm
- net ACTIVATE_SERVO: track 0.00 -> 20.2 mm
- net ADC_CAP: track 89.4 -> 108.5 mm, vias 2 -> 4
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
Commit message: rekick2015 Prototyp ordered
Parts:
- added C51: 100n, rcl:C0603
- C1, C2: value 47µF/35V -> 10µ/10V
- C13: value 2.2µ / 250V -> 2.2µ/250V
- C17, C18, C20, C21, C29, C3, C30, C31, C40, C42: value 47µF/35V -> 47µ/35V
- C19, C22: value 10nF/50V -> 10n/35V
- C25: value 2.2µ -> 10µ/450V
- C49: value 10µ -> 10µ/10V
- CF: value (none) -> 470p
- CSS: value (none) -> 1µ/10V
- C_DELAY: value (none) -> 10µ/10V
- C_ISEN_A: value (none) -> 22n/50V
- C_ISEN_B: value (none) -> 62n/10V
- D1: value GF1 -> ES1A
- F1: value 1812L -> FUSETE5; device ptc-littlefuse:1812L -> fuse:TE5
- L3: value 20µ -> 3.3UH; device inductor-bourns:SRR1210 -> Panasonic-ELL:IND_ELLATP-B
- R13, R18: device rcl:R0805 -> rcl:R2512
- R14, R17: value 380 -> 390
- R200: value 47k -> 50k
- R37: value 17k -> 16.9k
- R46, R59: value 11k -> 10k
- RF_MAX, R_ISEN_A: value (none) -> 33k
- RF_MIN: value (none) -> 12k
- R_ISEN_B: value (none) -> 2k
- R_SS: value (none) -> 3.3k, 1%
- T5: value (none) -> IRLML6344TRPBF
- moved R18 5.97 mm to (129.3, 41.3), turned to 180 degrees
- moved R13 5.48 mm to (129.3, 45.6), turned to 180 degrees
- moved D5 3.45 mm to (128.5, 49.9), turned to 180 degrees
- moved L3 3.18 mm to (57.7, 35.8), turned to 270 degrees
- moved D6 2.03 mm to (43.4, 92.6)
- moved D7 2.03 mm to (15.7, 19.1)
- moved F1 0.57 mm to (11.4, 9.65)
Connections:
- net +24V: now also F1.1; no longer F1.P$1
- net CAP_0V: now also C51.2, H1.B3,0
- net N$14: now also C51.1
- net N$30: now also F1.2; no longer F1.P$2
Routing:
- net GND: track 38.9 -> 43.0 mm, vias 14 -> 16
- net N$48: track 20.0 -> 23.8 mm
- net N$53: track 3.59 -> 7.11 mm
- net N$1: track 9.89 -> 12.5 mm
- net N$26: track 9.96 -> 12.6 mm
- net N$29: track 39.2 -> 36.6 mm
- net N$14: track 33.1 -> 35.5 mm
- net N$44: track 16.2 -> 18.4 mm
- net TRAFO2: track 69.9 -> 68.3 mm
- net N$30: track 9.99 -> 11.1 mm
- net +24V: vias 4 -> 3
- net CAP_0V: vias 6 -> 7

Commit message: rekick2015 - values for prototyp
Parts:
- C_DELAY: value 10µ/10V -> 1µ/10V
- C_ISEN_A: value 22n/50V -> 10n/50V
- C_ISEN_B: value 62n/10V -> 24nF/10V
- R_DELAY: value (none) -> 33k
- R_ISEN_B: value 2k -> 6,8k
Changed lines of the file:
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@@
 <element name="C12" library="rcl" package="C0603" value="100n" x="35.814" y="29.083" rot="MR0"/>
 <element name="C_BOOT" library="rcl" package="C0603" value="100n" x="49.276" y="24.511" rot="MR90"/>
-<element name="R_DELAY" library="rcl" package="R0805" value="" x="29.718" y="25.273" rot="MR180"/>
-<element name="C_DELAY" library="rcl" package="C0603" value="10µ/10V" x="29.718" y="22.987" rot="MR0"/>
+<element name="R_DELAY" library="rcl" package="R0805" value="33k" x="29.718" y="25.273" rot="MR180"/>
+<element name="C_DELAY" library="rcl" package="C0603" value="1µ/10V" x="29.718" y="22.987" rot="MR0"/>
 <element name="C11" library="rcl" package="C0603" value="100n" x="43.307" y="30.226" rot="R90"/>
-<element name="C_ISEN_A" library="rcl" package="C0603" value="22n/50V" x="43.815" y="17.526" rot="R90"/>
+<element name="C_ISEN_A" library="rcl" package="C0603" value="10n/50V" x="43.815" y="17.526" rot="R90"/>
 <element name="R_ISEN_A" library="rcl" package="R0805" value="33k" x="41.275" y="17.653" rot="R270"/>
 <element name="D3" library="diode" package="SOD123" value="MBR0520LT" x="38.989" y="17.272" rot="R90"/>
 <element name="D4" library="diode" package="SOD123" value="MBR0520LT" x="36.449" y="17.272" rot="R90"/>
-<element name="R_ISEN_B" library="rcl" package="R0805" value="2k" x="33.528" y="17.272" rot="R270"/>
-<element name="C_ISEN_B" library="rcl" package="C0603" value="62n/10V" x="30.988" y="17.272" rot="R90"/>
+<element name="R_ISEN_B" library="rcl" package="R0805" value="6,8k" x="33.528" y="17.272" rot="R270"/>
+<element name="C_ISEN_B" library="rcl" package="C0603" value="24nF/10V" x="30.988" y="17.272" rot="R90"/>
 <element name="L3" library="Panasonic-ELL" package="IND_ELLATP-B" value=" 3.3UH " x="57.658" y="35.814" rot="R270">
 <attribute name="PACKAGE" value="SMD-ELLATP-B" x="57.658" y="35.814" size="1.778" layer="27" rot="R270" display="off"/>
