File: msl_electronic_boards/rekick2015/pcb/rekick2015-Prototyp.sch (EAGLE design)
At the start: 200 parts, among them IC1 LM1458D, IC2 4043D, IC3 LM1117, IC4 LM1458D, Q1 16MHz, Q2 IGW60T120, Q3 IPP023N10N5, Q4 IPP023N10N5, Q5 IPD90P04P4L, Q6 IRF840, T1 BC849, T2 BC849, T3 BC849, T4 BC849, U1 TXB0108PWR, U3 LM2675, U4 LM2675, U5 MC14025BDG

Commit message: rekick2015 little changes
Parts:
- removed R31: 20k, rcl:R-EU_R0805
Connections:
- net ACTIVATE_BOOSTER: no longer R31.2
- net GND1: no longer R31.1
Changed lines of the file:
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@@
 <?xml version="1.0" encoding="utf-8"?>
 <!DOCTYPE eagle SYSTEM "eagle.dtd">
-<eagle version="7.5.0">
+<eagle version="7.2.0">
 <drawing>
 <settings>
@@
 <part name="C7" library="rcl" deviceset="C-EU" device="C0603" value="100n"/>
 <part name="SUPPLY26" library="supply2" deviceset="+5V/3" device=""/>
-<part name="R31" library="rcl" deviceset="R-EU_" device="R0805" value="20k"/>
 <part name="H1" library="holes" deviceset="MOUNT-PAD-ROUND" device="3.0"/>
 <part name="H2" library="holes" deviceset="MOUNT-PAD-ROUND" device="3.0"/>
@@
 <part name="GND38" library="supply1" deviceset="GND" device=""/>
 <part name="P+17" library="supply1" deviceset="+24V" device=""/>
-<part name="SUPPLY18" library="supply2" deviceset="GND1" device=""/>
 </parts>
 <sheets>
@@
 <instance part="R24" gate="G$1" x="167.64" y="160.02"/>
 <instance part="C35" gate="G$1" x="157.48" y="147.32"/>
-<instance part="R31" gate="G$1" x="144.78" y="152.4" rot="R90"/>
 <instance part="CAP_330V" gate="G$1" x="254" y="116.84" rot="R180"/>
 <instance part="CAP_0V" gate="G$1" x="254" y="101.6" rot="R180"/>
@@
 <instance part="R53" gate="G$1" x="144.78" y="124.46"/>
 <instance part="R54" gate="G$1" x="144.78" y="104.14"/>
-<instance part="SUPPLY18" gate="G$1" x="144.78" y="142.24"/>
 </instances>
 <busses>
@@
 <junction x="231.14" y="147.32"/>
 </segment>
-<segment>
-<pinref part="R31" gate="G$1" pin="1"/>
-<wire x1="144.78" y1="144.78" x2="144.78" y2="147.32" width="0.1524" layer="91"/>
-<pinref part="SUPPLY18" gate="G$1" pin="GND1"/>
-</segment>
 </net>
 <net name="BOOSTER_24V" class="0">
@@
 <segment>
 <pinref part="R24" gate="G$1" pin="1"/>
-<wire x1="162.56" y1="160.02" x2="144.78" y2="160.02" width="0.1524" layer="91"/>
+<wire x1="162.56" y1="160.02" x2="139.7" y2="160.02" width="0.1524" layer="91"/>
 <label x="139.7" y="160.02" size="1.778" layer="95" rot="R180" xref="yes"/>
-<pinref part="R31" gate="G$1" pin="2"/>
-<wire x1="144.78" y1="160.02" x2="139.7" y2="160.02" width="0.1524" layer="91"/>
-<wire x1="144.78" y1="157.48" x2="144.78" y2="160.02" width="0.1524" layer="91"/>
-<junction x="144.78" y="160.02"/>
-</segment>
-</net>
+</segment>
+</net>

Commit message: rekick2015
Parts:
- removed T1: BC849, transistor:BC849
- removed U5: MC14025BDG, MC14025BDG:MC14025BDG
- added C41, C47: 100n, rcl:C-EUC0603
- added R31: 50k, rcl:R-EU_R0805
- added R55, R56, R57, R58: 5,6k, rcl:R-EU_R0805
- added R59: 11k, rcl:R-EU_R0805
- added T6: BC859, transistor:BC858C-PNP-SOT23-BEC
- added U2: SN74LVC2G02DCTR, SN74LVC2G02DCTR:SN74LVC2G02DCTR
- C14, C15, C23, C24, C36, C46: value 100p -> 100n
- C30: device rcl:CPOL-EUD -> rcl:CPOL-EUE2-5
- C31: value 1µ -> 47µF/35V; device rcl:C-EUC0603 -> rcl:CPOL-EUE2-5
- C32: value 1µ -> 100n
- C37, C38: value 100p -> 1µ/25V; device rcl:C-EUC0603 -> rcl:CPOL-EUSMCA
- D5: value SMD ZD 15 -> ES1A; device diode:BZX84CSMD -> diode:GF1
- R10, R47: value 1k -> 5,6k
- R105: value 750 -> 680
- R11, R8: value 2k, 1% -> 10k, 1%
- R12: value 68k -> 10k
- R13: value 10k -> 5
- R15: value 10 -> 10k
- R16: value 470k -> 50k; device rcl:R-EU_0207/15 -> rcl:R-EU_R0805
- R18: value 10 -> 5
- R19: value 3k -> 5,6k
- R20: value B72220S0321K101 -> ERZE07A621; device varistor:S20K320 -> varistor:S10K385
- R21: value 10k, 1% -> 33k, 1%
- R24, R28: value 10k -> 5,6k
- R25: value 10k -> 100k
- R26, R27: value 10k -> 50k
- R30: value 1k -> 3.3k
- R4: value 10k, 1% -> 24k, 1%
- R46: value 680 -> 11k
- R5: value 3k, 1% -> 10k, 1%
- R50: value 4.7k -> 5,6k
- R51: value 12k -> 50k
- R52: value 10k -> 10k, 1%
- R7: value 2.37k, 1% -> 5.6k, 1%
Connections:
- removed net ADC1/SCK_A: SV1.7, U$2.(RXD)PD4
- removed net CAP_-12V: C30.-, C43.2, IC1P.V-, LED10.C, U$4.-U_OUT
- removed net FREI3: U$2.PD7
- new net 24V_PRI: C10.+, C35.1, C9.+, Q3.D, Q5.D, R23.2, R27.2
- new net ADC_24V_LOGIK/SCK_A: R31.2, R50.1, SV1.7, U$2.(RXD)PD4
- new net ADC_24V_PRI: R27.1, R28.2, U$2.PD5
- new net N$51: R55.1, U$2.PC6
- new net N$68: R58.1, U$2.PC1
- net +24V: now also R31.1
- net +5V: now also U2.VCC; no longer U5.VDD
- net +5V/3: now also C37.+; no longer R27.2
- net +5V/4: now also C38.+
- net ACTIVATE_SERVO: now also U$2.PD7; no longer U$2.PD5
- net ADC_CAP: now also C47.1
- net BOOSTER_24V: no longer R12.2
- net BURST: now also U2.2Y; no longer U$2.PC5, U5.OUTB
- net CAP_+12V: now also C30.+, C31.+, T6.E; no longer C31.1, C32.1
- net CAP_0V: now also C30.-, C31.-, C38.-, C43.2, IC1P.V-, U$4.-U_OUT; no longer C30.+, C31.2, D5.A, R50.2, T1.E, U$4.0V
- net CAP_330V: no longer R16.2
- net GND: now also C37.-, C41.2, C47.2, LED10.C, R16.1, R50.2; no longer C37.2, C38.2, R13.1, U5.IN_1C, U5.IN_3A, U5.IN_3B, U5.IN_3C, U5.VSS
- net N$15: now also C32.1
- net N$30: now also R59.2
- net N$37: now also U2.1A; no longer U5.IN_1A
- net N$38: now also U2.2A; no longer U5.IN_1B
- net N$39: now also Q6.G, R12.2, T6.C; no longer C38.1, IC4B.-IN, R12.1, R13.2
- net N$44: now also D5.C
- net N$45: now also R56.2; no longer D5.C, Q6.G, R16.1, T1.C
- net N$46: now also T6.B; no longer T1.B
- net N$48: now also R13.2
- net N$50: now also U2.2B; no longer U5.IN_2B
- net N$53: now also D5.A, R13.1; no longer IC4B.OUT, U5.IN_2C
- net N$57: now also R56.1, U$2.PC5; no longer C10.+, C35.1, C9.+, Q3.D, Q5.D, R23.2
- net N$58: now also U2.1B; no longer U5.IN_2A
- net N$59: now also R57.1, U$2.PC4; no longer C37.1, IC4B.+IN, R27.1, R28.2
- net N$75: now also R16.2
- net N$77: now also R59.1; no longer R50.1
- net NOTAUS: now also R55.2, U2.1Y; no longer U$2.PC6, U5.OUTA
- net SERVO_PWM: now also R58.2; no longer U$2.PC1
- net STBY: now also R57.2; no longer U$2.PC4
- net ÜBERSPANNUNG: now also C41.1
Other:
- moved on the sheet: C29, C36, COIL_IN, COIL_OUT, JP3, LED9, Q2, Q6, R15, R18, R2, R20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

Commit message: rekick2015
Connections:
- removed net N$45: R56.2
- net BURST: now also R56.2
Changed lines of the file:
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@@
 <net name="BURST" class="0">
 <segment>
-<wire x1="160.02" y1="119.38" x2="162.56" y2="119.38" width="0.1524" layer="91"/>
 <label x="162.56" y="119.38" size="1.27" layer="95" xref="yes"/>
+<pinref part="R56" gate="G$1" pin="2"/>
+<wire x1="157.48" y1="119.38" x2="162.56" y2="119.38" width="0.1524" layer="91"/>
 </segment>
 </net>
@@
 </segment>
 </net>
-<net name="N$45" class="0">
-<segment>
-<pinref part="R56" gate="G$1" pin="2"/>
-<wire x1="157.48" y1="119.38" x2="160.02" y2="119.38" width="0.1524" layer="91"/>
-</segment>
-</net>

Commit message: rekick2015
Parts:
- removed R_SS2: (no value), rcl:R-EU_R0805
Connections:
- removed net N$7: CSS.1, R_SS.1, R_SS2.1
- net N$18: now also CSS.1, R_SS.1; no longer R_SS2.2
Changed lines of the file:
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@@
 <?xml version="1.0" encoding="utf-8"?>
 <!DOCTYPE eagle SYSTEM "eagle.dtd">
-<eagle version="7.5.0">
+<eagle version="7.2.0">
 <drawing>
 <settings>
@@
 <part name="C12" library="rcl" deviceset="C-EU" device="C0603"/>
 <part name="C_BOOT" library="rcl" deviceset="C-EU" device="C0603" value="100n"/>
-<part name="R_SS2" library="rcl" deviceset="R-EU_" device="R0805"/>
 <part name="R_DELAY" library="rcl" deviceset="R-EU_" device="R0805"/>
 <part name="C_DELAY" library="rcl" deviceset="C-EU" device="C0603"/>
@@
 <instance part="C12" gate="G$1" x="55.88" y="104.14"/>
 <instance part="C_BOOT" gate="G$1" x="134.62" y="129.54"/>
-<instance part="R_SS2" gate="G$1" x="78.74" y="142.24" rot="R270"/>
 <instance part="R_DELAY" gate="G$1" x="63.5" y="129.54" rot="R90"/>
 <instance part="C_DELAY" gate="G$1" x="68.58" y="129.54"/>
@@
 </segment>
 </net>
-<net name="N$7" class="0">
-<segment>
+<net name="N$11" class="0">
+<segment>
+<pinref part="U$3" gate="L6599" pin="CF"/>
+<pinref part="CF" gate="G$1" pin="1"/>
+<wire x1="91.44" y1="121.92" x2="86.36" y2="121.92" width="0.1524" layer="91"/>
+</segment>
+</net>
+<net name="N$19" class="0">
+<segment>
+<pinref part="U$3" gate="L6599" pin="VBOOT"/>
+<pinref part="C_BOOT" gate="G$1" pin="1"/>
+<wire x1="127" y1="132.08" x2="134.62" y2="132.08" width="0.1524" layer="91"/>
+</segment>
+</net>
+<net name="N$18" class="0">
+<segment>
+<pinref part="U$3" gate="L6599" pin="CSS"/>
+<wire x1="78.74" y1="132.08" x2="91.44" y2="132.08" width="0.1524" layer="91"/>
 <pinref part="R_SS" gate="G$1" pin="1"/>
 <wire x1="45.72" y1="152.4" x2="45.72" y2="129.54" width="0.1524" layer="91"/>
@@
 <wire x1="78.74" y1="152.4" x2="88.9" y2="152.4" width="0.1524" layer="91"/>
 <wire x1="88.9" y1="152.4" x2="88.9" y2="149.86" width="0.1524" layer="91"/>
-<pinref part="R_SS2" gate="G$1" pin="1"/>
-<wire x1="78.74" y1="147.32" x2="78.74" y2="152.4" width="0.1524" layer="91"/>
 <junction x="78.74" y="152.4"/>
-</segment>
-</net>
-<net name="N$11" class="0">
-<segment>
-<pinref part="U$3" gate="L6599" pin="CF"/>
-<pinref part="CF" gate="G$1" pin="1"/>
-<wire x1="91.44" y1="121.92" x2="86.36" y2="121.92" width="0.1524" layer="91"/>
-</segment>
-</net>
-<net name="N$19" class="0">
-<segment>
-<pinref part="U$3" gate="L6599" pin="VBOOT"/>
-<pinref part="C_BOOT" gate="G$1" pin="1"/>
-<wire x1="127" y1="132.08" x2="134.62" y2="132.08" width="0.1524" layer="91"/>
-</segment>
-</net>
-<net name="N$18" class="0">
-<segment>
-<pinref part="U$3" gate="L6599" pin="CSS"/>
-<wire x1="78.74" y1="132.08" x2="91.44" y2="132.08" width="0.1524" layer="91"/>
-<pinref part="R_SS2" gate="G$1" pin="2"/>
-<wire x1="78.74" y1="132.08" x2="78.74" y2="137.16" width="0.1524" layer="91"/>
-</segment>
-</net>
+<wire x1="78.74" y1="132.08" x2="78.74" y2="152.4" width="0.1524" layer="91"/>
+</segment>
+</net>

Commit message: rekick2015 finished prototyp
Parts:
- removed D16, D17: ES1A, diode:GF1
- removed R56: 5,6k, rcl:R-EU_R0805
- removed R_LINE: 10k, rcl:R-EU_R0805
- added C48: 100n, rcl:C-EUC0603
- added C49: 10µ, rcl:C-EUC0603
- added C50: 1µ/50V, rcl:C-EUC1206
- added JP4: (no value), pinhead:PINHD-1X3
- added R61: 5,6k, rcl:R-EU_R0805
- added R70: 10k, rcl:R-EU_R0805
- added T1, T8: BC849, transistor:BC849
- C12: value (none) -> 100n
- C35: device rcl:C-EUC0603 -> rcl:C-EUC1206
- R48: value 10k -> 5,6k
- R52: value 10k, 1% -> 5,6k, 1%
- R58: value 5,6k -> 10k
Connections:
- removed net 1.25V-BIS-6V: R_LINE.2, U$3.LINE
- removed net BURST: D17.C, R56.2, U2.2Y
- removed net D2A/RF_MAX: RF_MAX.1, U$2.PC7
- removed net N$57: R56.1, U$2.PC5
- removed net N$68: R58.1, U$2.PC1
- removed net OC0A/MOSI_A/KICK_VOLTAGE: R52.1, U$2.(MOSI_A/TXD)PD3
- removed net OC1A/MISO_A: SV1.9, U$2.(MISO_A)PD2
- new net ADC9/FREI: U$2.PC5
- new net D2A: R52.1, U$2.PC7
- new net LINE: C48.1, R70.2, T1.C, T2.C, U$3.LINE, U$6.CATHODE
- new net N$7: RF_MAX.1, T8.C
- new net N$78: R61.2, T1.B
- new net N$79: C49.1, R48.2, T8.B
- new net OC1A_FREQ/MISO_A: R48.1, SV1.9, U$2.(MISO_A)PD2
- net +5V: now also R58.2, R70.1; no longer R48.2, R_LINE.1
- net +5V/1: now also JP4.2
- net 24V_PRI: now also C50.1
- net CAP_0V: now also R12.1
- net GND: now also C48.2, C49.2, H2.MOUNT, H3.MOUNT, H4.MOUNT, IC4B.+IN, IC4B.-IN, JP4.3, T1.E, T8.E, U2.GND
- net GND1: now also C50.2
- net N$42: now also IC2A.EN, R58.1; no longer T2.C, U$6.CATHODE
- net NOTAUS: now also R61.1; no longer D16.C
- net OC0A/MOSI_A: now also JP4.1, U$2.(MOSI_A/TXD)PD3
- net SERVO_PWM: now also U$2.PC1; no longer R58.2
- net STBY: now also U2.2Y; no longer D16.A, D17.A, R48.1
Other:
- moved on the sheet: C10, C12, C30, C31, C33, C34, C36, C37, C39, C41, C44, C45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

Commit message: rekick2015 Prototyp ordered
Parts:
- added C51: 100n, rcl:C-EUC0603
- C1, C2: value 47µF/35V -> 10µ/10V
- C13: value 2.2µ / 250V -> 2.2µ/250V
- C17, C18, C20, C21, C29, C3, C30, C31, C40, C42: value 47µF/35V -> 47µ/35V
- C19, C22: value 10nF/50V -> 10n/35V
- C25: value 2.2µ -> 10µ/450V
- C49: value 10µ -> 10µ/10V
- CF: value (none) -> 470p
- CSS: value (none) -> 1µ/10V
- C_DELAY: value (none) -> 10µ/10V
- C_ISEN_A: value (none) -> 22n/50V
- C_ISEN_B: value (none) -> 62n/10V
- D1: value GF1 -> ES1A
- F1: value 1812L -> FUSETE5; device ptc-littlefuse:1812L -> fuse:FUSETE5
- L3: value 20µ -> 3.3UH; device inductor-bourns:SRR1210 -> Panasonic-ELL:ELLATP3R3NB-ATP-B
- R13, R18: device rcl:R-EU_R0805 -> rcl:R-EU_R2512
- R14, R17: value 380 -> 390
- R200: value 47k -> 50k
- R37: value 17k -> 16.9k
- R46, R59: value 11k -> 10k
- RF_MAX, R_ISEN_A: value (none) -> 33k
- RF_MIN: value (none) -> 12k
- R_ISEN_B: value (none) -> 2k
- R_SS: value (none) -> 3.3k, 1%
- T5: value (none) -> IRLML6344TRPBF
Connections:
- net CAP_0V: now also C51.2, H1.MOUNT
- net N$14: now also C51.1

Commit message: rekick2015 - values for prototyp
Parts:
- C_DELAY: value 10µ/10V -> 1µ/10V
- C_ISEN_A: value 22n/50V -> 10n/50V
- C_ISEN_B: value 62n/10V -> 24nF/10V
- R_DELAY: value (none) -> 33k
- R_ISEN_B: value 2k -> 6,8k
Changed lines of the file:
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@@
 <part name="C12" library="rcl" deviceset="C-EU" device="C0603" value="100n"/>
 <part name="C_BOOT" library="rcl" deviceset="C-EU" device="C0603" value="100n"/>
-<part name="R_DELAY" library="rcl" deviceset="R-EU_" device="R0805"/>
-<part name="C_DELAY" library="rcl" deviceset="C-EU" device="C0603" value="10µ/10V"/>
+<part name="R_DELAY" library="rcl" deviceset="R-EU_" device="R0805" value="33k"/>
+<part name="C_DELAY" library="rcl" deviceset="C-EU" device="C0603" value="1µ/10V"/>
 <part name="C11" library="rcl" deviceset="C-EU" device="C0603" value="100n"/>
-<part name="C_ISEN_A" library="rcl" deviceset="C-EU" device="C0603" value="22n/50V"/>
+<part name="C_ISEN_A" library="rcl" deviceset="C-EU" device="C0603" value="10n/50V"/>
 <part name="R_ISEN_A" library="rcl" deviceset="R-EU_" device="R0805" value="33k"/>
 <part name="D3" library="diode" deviceset="MBR0520LT" device=""/>
 <part name="D4" library="diode" deviceset="MBR0520LT" device=""/>
-<part name="R_ISEN_B" library="rcl" deviceset="R-EU_" device="R0805" value="2k"/>
-<part name="C_ISEN_B" library="rcl" deviceset="C-EU" device="C0603" value="62n/10V"/>
+<part name="R_ISEN_B" library="rcl" deviceset="R-EU_" device="R0805" value="6,8k"/>
+<part name="C_ISEN_B" library="rcl" deviceset="C-EU" device="C0603" value="24nF/10V"/>
 <part name="L3" library="Panasonic-ELL" deviceset="ELL" device="-ATP-B" technology="ATP3R3NB" value=" 3.3UH "/>
 <part name="L4" library="EagleLibrary_Wuerth_Elektronik_eiSos_rev16a" deviceset="WE-HCI" device="_1890" value="820n"/>
