File: msl_electronic_boards/rekick2015/pcb/rekick2015-Prototyp-Flyback.brd (EAGLE design)
At the start: 160 x 100 mm, 193 parts, among them IC1 LM1458D, IC2 4043D, IC3 LM1117, IC4 LM1458D, Q1 16MHz, Q2 IGW60T120, Q3 IPP023N10N5, Q5 IPD90P04P4L, Q6 IRF840, T2 BC849, T3 BC849, T4 BC849, T5 IRLML6344TRPBF, T6 BC859, U1 TXB0108PWR, U2 SN74LVC2G02DCTR, U3 LM2675, U4 LM2675

Commit message: rekick flyback
Parts:
- removed C14, C15, C16, C23, C24, C32, C36, C43, C44, C46, C47, C51: 100n, rcl:C0603
- removed C38: 1µ/25V, rcl:SMC_A
- removed D12: BZX84-A5V1, diode:TO236
- removed IC1, IC4: LM1458D, linear:SO08
- removed OK1, OK2: ILD213, optocoupler:SOIC08
- removed R105: 680, rcl:R0805
- removed R12: 10k, rcl:R0805
- removed R21: 33k, 1%, rcl:R0805
- removed R25: 100k, rcl:R0805
- removed R26: 50k, rcl:R0805
- removed R29: 1k, rcl:R0805
- removed R52: 5,6k, 1%, rcl:R0805
- removed T6: BC859, transistor:SOT23-BEC
- added D3: SMD ZD 12, diode:TO236
- added R68: 150k, rcl:R0805
- added R69, R70, R71: 50k, rcl:R0805
- added T1, T7: BC859, transistor:SOT23-BEC
- added U5, U6: ADUM4190BRIZ, adum4190:SOIC127P1032X265-16N
- R10: value 5,6k -> 910k, 1%; device rcl:R0805 -> rcl:R2512
- R101: value 1M, 1% -> 910k, 1%
- R11: value 10k, 1% -> 100k
- R13, R18, R66: value 5 -> 4.7
- R4: value 24k, 1% -> 75k
- R48: value 375k -> 220k
- R5: value 10k, 1% -> 0
- R53: value 575k -> 560k
- R54: value 135k -> 130k
- R56: value 375k -> 360k
- R6: value 12k, 1% -> 11k
- R60: value 732 -> 0
- R67: value 375k -> 40.2k
- R7: value 5.6k, 1% -> 0
- R8: value 10k, 1% -> 261
- R9: value 2k -> 3,74k
- moved R11 347.1 mm to (-24.0, -242.1), flipped to the top, turned to 0 degrees
- moved R10 342.6 mm to (-22.0, -228.2), flipped to the top, turned to 0 degrees
- moved R8 329.9 mm to (-24.0, -208.0), flipped to the top, turned to 0 degrees
- moved R9 322.4 mm to (-24.0, -214.1), flipped to the top, turned to 0 degrees
- moved R5 315.2 mm to (-24.0, -189.7), flipped to the top
- moved R7 312.8 mm to (-24.0, -201.9)
- moved R4 295.9 mm to (-24.0, -183.6), turned to 0 degrees
- moved R6 292.9 mm to (-24.0, -195.8), flipped to the top, turned to 0 degrees
- moved T4 285.9 mm to (-23.6, -220.9)
Connections:
- net N$68 renamed FB
- removed net +5V/4: C16.1, C38.+, D12.C, OK1.8, R29.1, R7.2
- removed net CHARGE: U$9.8
- removed net KICK_VOLTAGE: C36.1, IC4.2, R21.2, R5.1, R52.2
- removed net N$35: OK2.1, R9.2
- removed net N$50: IC4.1, U2.6
- removed net N$52: R25.2, T4.1
- removed net N$58: R26.1, T4.3, U2.5
- new net 0V: R7.2
- new net N$78: R48.1, R68.2, T7.E
- new net N$79: R71.1, T7.B
- new net N$80: R69.1, T1.E, U$9.8
- new net N$81: R70.1, T1.B
- new net VDD1: U5.1, U6.1
- new net VDD2: U5.16, U6.16
- new net VREG1: U5.3, U6.3
- new net VREG2: U5.14, U6.14
- net +5V: no longer C44.1, IC4.8, OK2.8, R26.2
- net +5V/3: no longer OK1.6, R5.2
- net ACTIVATE_BOOSTER: now also R69.2; no longer R25.1
- net ADC_CAP: no longer C23.1, C47.1, IC4.3, OK1.5, R8.2
- net CAP_+12V: no longer C43.1, IC1.8, R29.2, T6.E
- net CAP_0V: now also D3.A, T4.2; no longer C14.2, C15.2, C16.2, C32.2, C38.-, C43.2, C46.2, C51.2, D12.A, IC1.4, OK1.4, OK2.2, R12.1, R4.1, R6.1
- net CAP_330V: now also R10.1
- net D2A: no longer R52.1
- net GND: now also T1.C, T7.C; no longer C23.2, C24.2, C36.2, C44.2, C47.2, IC4.4, IC4.5, IC4.6, R10.1, R21.1, R8.1, T4.2
- net N$13: now also R7.1, R9.2; no longer IC1.1, R105.1
- net N$14: now also R5.2, R6.1, U5.12; no longer C14.1, C51.1, IC1.2, OK1.7, R11.2
- net N$15: now also R4.2, R5.1; no longer C15.1, C32.1, IC1.3, IC1.5, R101.1, R6.2
- net N$21: now also R101.1, R4.1; no longer OK1.1, R105.2
- net N$22: now also U5.10, U5.11; no longer OK1.2, OK1.3
- net N$25: now also R8.2; no longer IC1.7
- net N$27: now also R6.2, R8.1; no longer C46.1, IC1.6, R4.2, R7.1
- net N$34: now also R68.1; no longer R48.1
- net N$39: now also D3.C, R10.2, T4.3; no longer R12.2, T6.C
- net N$46: now also R11.2, T4.1; no longer T6.B
- net NOTAUS: now also R70.2, R71.2
- net ÜBERSPANNUNG: no longer C24.1, OK2.7, R10.2
Routing:
- net ADC_CAP: track 108.5 -> 6.41 mm, vias 4 -> 1
- net N$50: track 75.0 -> 0.00 mm, vias 2 -> 0
- net N$58: track 45.3 -> 0.00 mm, vias 1 -> 0
- net +5V/4: track 38.9 -> 0.00 mm, vias 1 -> 0
- net N$14: track 35.5 -> 0.00 mm
- net CAP_+12V: track 141.6 -> 110.9 mm, vias 2 -> 0
- net N$15: track 19.6 -> 0.00 mm
- net N$13: track 15.3 -> 0.00 mm
- net KICK_VOLTAGE: track 12.0 -> 0.00 mm
- net N$27: track 11.1 -> 0.00 mm, vias 1 -> 0
- net N$25: track 10.6 -> 0.00 mm
- net ÜBERSPANNUNG: track 58.5 -> 48.8 mm
- net +5V: track 380.2 -> 372.2 mm
- net N$35: track 7.41 -> 0.00 mm
- net N$39: track 8.06 -> 2.24 mm
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
Commit message: rekick flyback
Parts:
- removed LED1: (no value), led:CHIP-LED0805
- removed R3: 100, resistor-power:HS25
- removed R33, R34: 1M, rcl:R2512
- removed R36, R71: 50k, rcl:R0805
- removed R37: 16.9k, rcl:R0805
- removed R39: 4.7k, rcl:R0805
- removed R68: 150k, rcl:R0805
- removed R7: 0, rcl:R0805
- removed R8: 261, rcl:R0805
- removed T7: BC859, transistor:SOT23-BEC
- removed U2: SN74LVC2G02DCTR, SN74LVC2G02DCTR:SOP65P400X130-8N
- removed VR1: TL431_SOT23, 1_USER:SOT23
- added C13, C14, C15, C16, C23, C24, C32, C36: 1µ, rcl:C0603
- added C38, C43, C49, C57, C58, C59: 100n, rcl:C0603
- added C44, C46, C47, C48: 10p, rcl:C0603
- added C51: 10µ/50V, rcl:C1206
- added C52, C53, C54, C55, C56: (no value), rcl:E2,5-7
- added D4, D8: BZX84-A5V1, diode:TO236
- added IC1: 74LVC1G02GW, 74xx-little-de:SOT23-5
- added IC4: LM1458D, linear:SO08
- added KK1, KK2, KK3: SK104, heatsink:SK104
- added LED11: (no value), led:CHIPLED_0603
- added Q4: PSMN7R8-120PS, transistor-power:TO220BV
- added R12, R21, R25: 1k, rcl:R0805
- added R26, R29: 100k, rcl:R0805
- added R52, R72: 10k, rcl:R0805
- added R73: 10m, R2818:R2818
- added R74: 2, R2818:R2818
- added U$10, U$11: RTO50, RTO50:TO220ACS
- C10, C9: value 2200µ/50V -> 10µ/50V; device rcl:E5-13 -> rcl:C1206
- C11: device rcl:C1206 -> rcl:C2220K
- C12: value 100n -> 10µ/50V; device rcl:C0603 -> rcl:C1206
- C30, C31: device rcl:E2-5 -> rcl:C1206
- C35, C50: value 1µ/50V -> 10µ/50V
- C41: value 100n -> 22n; device rcl:C0603 -> rcl:C1206
- D9: value STTH1R06A -> STTH810D; device diode:SMA-DO214AC -> diode:TO220ACS
- Q3: value IPP023N10N5 -> PSMN7R8-120PS
- R10, R101: value 910k, 1% -> 1M, 1%; device rcl:R2512 -> rcl:R1206
- R13, R18: device rcl:R2512 -> rcl:R0805
- R2: value 100 -> 1M, 1%; device resistor-power:HS25 -> rcl:R1206
- R35: value 1M -> 4.7k; device rcl:R2512 -> rcl:R0805
- R38: value 7.68k -> 5.6k
- R4: value 75k -> 140k
- R40, R41: value 4.7k -> 1k
- R43, R45: value 1,5k -> 1k
- R57: value 5,6k -> 3.2k
- R6: value 11k -> 12.4k
- R63: value 6m -> 10m; device rcl:R0805 -> R2818:R2818
- R9: value 3,74k -> 4,7k
- moved R11 351.7 mm to (97.5, 88.0), flipped to the bottom, turned to 90 degrees
- moved D3 348.2 mm to (104.9, 88.0), flipped to the bottom, turned to 180 degrees
- moved R10 336.9 mm to (88.6, 90.0), flipped to the bottom, turned to 180 degrees
- moved T4 333.0 mm to (100.8, 88.0), flipped to the bottom, turned to 180 degrees
- moved R9 324.3 mm to (90.3, 89.4), turned to 90 degrees
- moved R6 304.9 mm to (83.7, 89.4), turned to 90 degrees
- moved R5 298.3 mm to (81.2, 89.4), turned to 270 degrees
- moved R4 291.7 mm to (78.6, 89.4), turned to 270 degrees
- moved U5 269.2 mm to (64.8, 89.8), flipped to the bottom, turned to 180 degrees
- moved U6 259.5 mm to (81.3, 69.2), turned to 90 degrees
- moved C11 238.4 mm to (145.7, 70.4), flipped to the bottom, turned to 270 degrees
- moved R70 207.6 mm to (81.7, 27.6)
- moved T1 207.6 mm to (82.0, 34.3)
- moved R67 203.5 mm to (101.3, 39.1)
- moved R63 202.5 mm to (136.3, 49.7), flipped to the bottom, turned to 180 degrees
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Connections:
- removed net 0V: R7.2
- removed net ADC9/FREI: U$2.18
- removed net ADC_24V_PRI: U$2.13
- removed net D2A: U$2.25
- removed net FREI: U$2.16
- removed net FREI2: U$2.27
- removed net N$12: R33.1, R36.2, VR1.2
- removed net N$13: R7.1, R9.2
- removed net N$2: LED1.C, VR1.1
- removed net N$25: R8.2, R9.1
- removed net N$34: R68.1, U$9.2
- removed net N$60: R34.1, R37.2, VR2.2
- removed net N$64: LED1.A, R39.1
- removed net N$79: R71.1, T7.B
- removed net N$80: R69.1, T1.E, U$9.8
- removed net STBY: R57.2, U2.3
- removed net VDD1: U5.1, U6.1
- removed net VDD2: U5.16, U6.16
- removed net VREG1: U5.3, U6.3
- removed net VREG2: U5.14, U6.14
- new net !CHARGE: R69.1, T1.E, U$2.17, U$9.8
- new net ADC_CAP_OV: IC4.3, R52.1, U5.7
- new net N$35: R12.1, S1.3, S1.4
- new net N$50: C15.1, U5.3
- new net N$52: C16.1, U5.14
- new net N$58: C36.1, U6.14
- new net N$68: C32.1, U6.3
- new net N$82: R21.2, R26.2, U6.12
- new net N$83: R29.1, U6.10
- new net N$84: C47.1, R25.1, U6.13
- new net N$85: R25.2, R29.2, U6.11
- new net N$86: C41.2, R74.P$1
- new net N$89: C44.1, U5.13
- new net N$90: C46.1, U5.4
- new net N$91: R72.1, U6.7
- new net N$93: C48.1, U6.4
- net !FAULT: now also U$2.18
- net +12V: now also C13.1, C23.1, U5.1, U6.1
- net +5V: now also C49.1, IC1.5, IC4.8, R12.2, R40.2, R41.2, R57.1; no longer S1.1, S1.2, U2.8
- net +5V/3: now also IC4.2
- net ADC_24V_BOOSTER: now also C58.2, U$2.13
- net ADC_24V_LOGIK/SCK_A: now also C59.2
- net ADC_CAP: now also C57.1, D8.C, R35.2, R52.2, VR2.2
- net CAP_+12V: now also C14.1, C24.1, C30.1, C31.1, U5.16, U6.16; no longer C30.+, C31.+, R39.2, R40.2, R41.2
- net CAP_0V: now also C14.2, C16.2, C24.2, C30.2, C31.2, C36.2, C38.2, C43.2, C44.2, C47.2, R26.1, R9.2, U5.15, U5.9, U6.15, U6.9; no longer C30.-, C31.-, R36.1, R37.1, VR1.3
- net CAP_330V: now also D9.C, U$10.A; no longer D9.K, R33.2, R34.2, R35.2
- net CLKOUT_ETH: now also U1.14; no longer U1.12
- net CLKOUT_ETH_3V: now also U1.7; no longer U1.9
- net FB: now also D4.C, R72.2
- net GND: now also C13.2, C15.2, C23.2, C32.2, C46.2, C48.2, C49.2, C57.2, C58.1, C59.1, D4.A, D8.A, IC1.3, IC4.4, U5.2, U5.5, U5.8, U6.2, U6.5, U6.8; no longer C41.2, T7.C, U2.4
- net GND1: now also C10.2, C51.2, C52.-, C53.-, C54.-, C55.-, C56.-, C9.2, R63.P$2, R73.P$2; no longer C10.-, C9.-, R63.2
- net N$14: now also C43.1
- net N$16: now also Q4.D, R74.P$2
- net N$17: now also Q4.S, R63.P$1, R73.P$1; no longer R63.1
- net N$18: now also Q4.G
- net N$23: now also U$10.C, U$11.A; no longer R2.2, R3.1
- net N$24: now also U$11.C; no longer R3.2
- net N$27: now also C38.1, R21.1, R9.1; no longer R8.1
- net N$37: now also IC1.1; no longer U2.1
- net N$38: now also IC1.2; no longer U2.2
- net N$39: now also R2.2
- net N$59: now also R48.1, U$9.2; no longer R57.1, U$2.17
- net N$78: now also LED11.A, R57.2; no longer R48.1, R68.2, T7.E
- net N$8: now also C10.1, C41.1, C51.1, C52.+, C53.+, C54.+, C55.+, C56.+, C9.1; no longer C10.+, C9.+
- net NOTAUS: now also IC1.4, LED11.C; no longer R71.2, U2.7
- net RST_ETH: now also U1.12; no longer U1.14
- net RST_ETH_3V: now also U1.9; no longer U1.7
- net TASTER: now also S1.1, S1.2; no longer S1.3, S1.4
- net ÜBERSPANNUNG: now also IC4.1; no longer C41.1
Routing:
- net +5V: track 372.2 -> 15.4 mm, vias 10 -> 1
- net +24V: track 228.8 -> 0.00 mm, vias 3 -> 0
- net +5V/1: track 182.2 -> 0.00 mm, vias 2 -> 0
- net NOTAUS: track 132.4 -> 0.00 mm, vias 3 -> 0
- net D2A: track 109.1 -> 0.00 mm, vias 4 -> 0
- net +3V3: track 101.7 -> 0.00 mm, vias 3 -> 0
- net +5V/3: track 98.8 -> 13.4 mm, vias 2 -> 1
- net CAP_+12V: track 110.9 -> 34.7 mm, vias 0 -> 1
- net RESET_NOTAUS: track 75.8 -> 0.00 mm, vias 3 -> 0
- net KICK: track 74.9 -> 0.00 mm, vias 2 -> 0
- net STBY: track 70.6 -> 0.00 mm, vias 2 -> 0
- net +12V: track 70.3 -> 4.15 mm, vias 2 -> 0
- net ACTIVATE_BOOSTER: track 53.6 -> 0.00 mm, vias 2 -> 0
- net ÜBERSPANNUNG: track 48.8 -> 0.00 mm, vias 3 -> 0
- net ADC_24V_LOGIK/SCK_A: track 63.0 -> 24.1 mm, vias 5 -> 1
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- removed copper zone on layer 1, net CAP_0V
- removed copper zone on layer 16, net CAP_0V
- removed copper zone on layer 1, net GND
- removed copper zone on layer 16, net GND
- removed copper zone on layer 1, net GND1
- removed copper zone on layer 16, net GND1
