File: msl_electronic_boards/rekick2015/pcb/rekick2016-Flyback-Prototyp-Final.brd (EAGLE design)
At the start: 160 x 100 mm, 203 parts, among them IC1 74LVC1G02GW, IC2 4043D, IC3 LM1117, IC4 LM1458D, Q1 16MHz, Q2 IKW 25N120, Q3 PSMN7R8-120PS, Q4 PSMN7R8-120PS, Q5 IPD90P04P4L, Q6 IRF840, T1 BC859, T2 BC849, T3 BC849, T4 BC849, T5 IRLML6344TRPBF, U1 TXB0108PWR, U3 LM2675, U4 LM2675, U5 ADUM4190BRIZ, U6 ADUM4190BRIZ

Commit message: rekick 2016 little changes in layout
Routing:
- net NOTAUS: track 67.6 -> 68.2 mm
- net GND: vias 18 -> 19
Changed lines of the file:
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@@
 <via x="106.426" y="34.417" extent="1-16" drill="0.6"/>
 <via x="106.426" y="32.639" extent="1-16" drill="0.6"/>
+<via x="34.925" y="32.258" extent="1-16" drill="0.6"/>
 </signal>
 <signal name="SCK_3V">
@@
 <contactref element="R9" pad="2"/>
 <contactref element="H2" pad="B3,0"/>
-<wire x1="132.715" y1="64.77" x2="140.589" y2="64.77" width="3.81" layer="1"/>
-<wire x1="140.589" y1="64.77" x2="143.637" y2="61.722" width="3.81" layer="1"/>
-<wire x1="143.637" y1="61.722" x2="146.304" y2="61.722" width="3.81" layer="1"/>
 <wire x1="146.304" y1="67.808" x2="146.304" y2="63.373" width="1.4224" layer="16"/>
 <via x="146.304" y="63.373" extent="1-16" drill="1"/>
@@
 <via x="75.184" y="78.359" extent="1-16" drill="0.6"/>
 <via x="65.913" y="71.628" extent="1-16" drill="0.6"/>
+<wire x1="132.715" y1="64.77" x2="140.589" y2="64.77" width="2.54" layer="1"/>
+<wire x1="140.589" y1="64.77" x2="143.637" y2="61.722" width="2.54" layer="1"/>
+<wire x1="143.637" y1="61.722" x2="146.304" y2="61.722" width="2.54" layer="1"/>
 </signal>
 <signal name="CAP_+12V">
@@
 <contactref element="LED11" pad="C"/>
 <wire x1="50.927" y1="46.924" x2="50.866" y2="46.924" width="0.3048" layer="1"/>
-<wire x1="50.866" y1="46.924" x2="48.1965" y2="49.5935" width="0.3048" layer="1"/>
-<wire x1="47.0535" y1="50.7365" x2="46.355" y2="51.435" width="0.3048" layer="1"/>
+<wire x1="50.866" y1="46.924" x2="47.752" y2="50.038" width="0.3048" layer="1"/>
+<wire x1="47.752" y1="50.038" x2="46.355" y2="51.435" width="0.3048" layer="1"/>
 <wire x1="46.355" y1="51.435" x2="41.783" y2="51.435" width="0.3048" layer="1"/>
 <wire x1="41.783" y1="51.435" x2="28.575" y2="51.435" width="0.3048" layer="1"/>
@@
 <wire x1="59.69" y1="49.022" x2="59.055" y2="49.657" width="0.3048" layer="1"/>
 <via x="59.055" y="49.657" extent="1-16" drill="0.6"/>
-<wire x1="59.055" y1="49.657" x2="48.26" y2="49.657" width="0.3048" layer="16"/>
-<wire x1="48.26" y1="49.657" x2="48.1965" y2="49.5935" width="0.3048" layer="16"/>
-<via x="48.1965" y="49.5935" extent="1-16" drill="0.6"/>
-<wire x1="48.1965" y1="49.5935" x2="47.0535" y2="50.7365" width="0.3048" layer="1"/>
+<wire x1="59.055" y1="49.657" x2="48.133" y2="49.657" width="0.3048" layer="16"/>
 <wire x1="69.977" y1="60.391" x2="69.977" y2="50.419" width="0.3048" layer="16"/>
 <wire x1="69.977" y1="50.419" x2="69.215" y2="49.657" width="0.3048" layer="16"/>
 <wire x1="69.215" y1="49.657" x2="59.055" y2="49.657" width="0.3048" layer="16"/>
+<wire x1="48.133" y1="49.657" x2="47.752" y2="50.038" width="0.3048" layer="16"/>
+<via x="47.752" y="50.038" extent="1-16" drill="0.6"/>
 </signal>
 <signal name="N$40">
@@
 <contactref element="COIL_IN" pad="P$1"/>
 <contactref element="U$7" pad="A"/>
-<wire x1="132.715" y1="70.358" x2="138.938" y2="70.358" width="3.81" layer="1"/>
-<wire x1="138.938" y1="70.358" x2="146.304" y2="70.358" width="3.81" layer="1"/>
 <wire x1="132.715" y1="59.182" x2="128.905" y2="59.182" width="0.8128" layer="16"/>
 <wire x1="128.905" y1="59.182" x2="127.635" y2="60.452" width="0.8128" layer="16"/>
@@
 <wire x1="127.635" y1="69.088" x2="128.905" y2="70.358" width="0.8128" layer="16"/>
 <wire x1="128.905" y1="70.358" x2="132.715" y2="70.358" width="0.8128" layer="16"/>
+<wire x1="138.938" y1="70.358" x2="146.304" y2="70.358" width="2.54" layer="1"/>
+<wire x1="138.938" y1="70.358" x2="132.715" y2="70.358" width="2.54" layer="1"/>
 </signal>
 <signal name="ACTIVATE_BOOSTER">
