File: msl_electronic_boards/rekick2015/pcb/rekick2016-Flyback-v2-extra-boards.brd (EAGLE design)
At the start: 160 x 100 mm, 14 parts, among them J3 79109-12, P1 87759-12, Q1 PSMN7R8-120PS, Q2 PSMN7R8-120PS, X1 79109-12, X2 87832-04

Commit message: rekick 2016 + extra boards
Parts:
- removed J3: 79109-12, con-molex-milli-grid:79109-12
- removed P1: 87759-12, con-molex-milli-grid:87759-12
- X1: value 79109-12 -> 87759-12; device con-molex-milli-grid:79109-12 -> con-molex-milli-grid:87759-12
- X2: value 87832-04 -> 87759-04; device con-molex:87832-04 -> con-molex-milli-grid:87759-04
- moved R6 42.0 mm to (15.1, 27.2), turned to 180 degrees
- moved R3 40.0 mm to (3.17, 29.5)
- moved R5 37.8 mm to (15.1, 24.9), turned to 180 degrees
- moved R2 35.0 mm to (3.17, 27.2)
- moved R1 30.2 mm to (3.17, 24.9)
- moved X2 29.0 mm to (9.14, 26.0)
- moved R4 24.1 mm to (3.17, 22.6)
- moved U$1 0.36 mm to (20.8, 5.59)
- moved U$2 0.36 mm to (14.5, 5.59)
- moved Q1 0.25 mm to (5.59, 10.2)
- moved Q2 0.25 mm to (5.59, 5.08)
- moved X1 0.25 mm to (7.62, 15.5)
Routing:
- net CSN/GND1: track 0.00 -> 37.5 mm, vias 0 -> 1
- net CSP: track 0.00 -> 34.1 mm
- net DRAIN_MOSFET: track 0.00 -> 20.0 mm
- net GATE_MOSFET: track 0.00 -> 15.8 mm
- net FB_SPANNUNGSTEILER: track 0.00 -> 12.6 mm
- net N$5: track 0.00 -> 7.75 mm
- net ADC_SPANNUNGSTEILER: track 0.00 -> 6.24 mm
- net START_SPANNUNGSTEILER: track 0.00 -> 4.44 mm
- net MASSE_SPANNUNGSTEILER: track 0.00 -> 4.44 mm
- net N$6: track 0.00 -> 2.29 mm
- net N$1: track 0.00 -> 2.29 mm
Other:
- board size 160 x 100 mm -> 24.4 x 31.7 mm
