File: msl_electronic_boards/rekick2015/pcb/rekick2016-Flyback-v2.brd (EAGLE design)
At the start: 160 x 100 mm, 201 parts, among them IC1 74LVC1G02GW, IC2 4043D, IC3 LM1117, IC4 LM1458D, P1 39-30-06?_S, P2 39-30-08?_S, Q1 16MHz, Q2 IKW 25N120, Q3 PSMN7R8-120PS, Q5 IPD90P04P4L, Q6 IRF840, T1 BC859, T2 BC849, T3 BC849, T4 BC849, T5 IRLML6344TRPBF, T6 BC859, U1 TXB0108PWR, U3 LM2675, U4 LM2675, U5 ADUM4190BRIZ, U6 ADUM4190BRIZ, X1 87832-12, X2 87832-04

Commit message: rekick 2016 layout
Parts:
- moved R45 65.9 mm to (51.3, 38.6), turned to 270 degrees
- moved LED7 65.8 mm to (51.3, 43.7), turned to 0 degrees
- moved D15 61.4 mm to (48.6, 41.4), turned to 90 degrees
- moved U$8 54.3 mm to (47.5, 41.4)
- moved C3 52.3 mm to (41.5, 50.0), turned to 0 degrees
- moved L1 52.2 mm to (47.5, 41.4), flipped to the bottom
- moved C40 52.1 mm to (41.5, 32.8)
- moved R8 51.2 mm to (50.9, 52.8), flipped to the top
- moved R7 46.1 mm to (53.2, 52.8), flipped to the top, turned to 90 degrees
- moved JP4 37.8 mm to (41.5, 65.5)
- moved R47 37.8 mm to (44.3, 58.5)
- moved JP3 37.8 mm to (45.3, 59.1)
- moved R16 37.8 mm to (44.3, 56.3)
- moved T5 37.8 mm to (44.3, 61.7)
- moved SV1 22.6 mm to (91.4, 15.4), turned to 180 degrees
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Connections:
- removed net N$23: R26.2, R29.2
- removed net N$25: R34.2, R36.2
- net N$13: now also R26.2, R29.2, R34.2, R36.2
Routing:
- net +5V: track 49.5 -> 285.0 mm, vias 4 -> 11
- net +24V: track 121.3 -> 199.9 mm, vias 0 -> 2
- net +12V: track 99.2 -> 177.3 mm, vias 4 -> 6
- net CAP_330V: track 0.00 -> 68.3 mm
- net +5V/1: track 0.00 -> 64.1 mm, vias 0 -> 1
- net CAP_+12V: track 4.36 -> 63.5 mm, vias 0 -> 1
- net NOTAUS: track 0.00 -> 58.0 mm, vias 0 -> 2
- net TRIGGER_NOTAUS: track 0.00 -> 40.6 mm
- net ADC_CAP: track 80.7 -> 113.2 mm, vias 3 -> 5
- net N$27: track 0.00 -> 31.3 mm
- net +3V3: track 31.7 -> 60.4 mm, vias 2 -> 4
- net N$51: track 0.00 -> 27.1 mm
- net KICK: track 0.00 -> 24.5 mm
- net OC0A/MOSI_A: track 45.7 -> 69.4 mm, vias 1 -> 2
- net RST: track 29.8 -> 50.5 mm
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
Commit message: rekick 2016 v2 done for robocup workshop
Parts:
- moved R101 5.19 mm to (110.5, 97.9), turned to 180 degrees
- moved R4 3.43 mm to (109.1, 96.0), turned to 270 degrees
- moved R5 3.05 mm to (105.3, 96.0), turned to 90 degrees
- moved R2 2.68 mm to (110.5, 93.3), turned to 0 degrees
- moved R10 2.57 mm to (110.5, 95.6), turned to 0 degrees
- moved R6 2.54 mm to (102.5, 96.0), turned to 270 degrees
- moved C24 2.29 mm to (99.3, 80.3)
- moved R9 2.03 mm to (99.7, 96.0), turned to 90 degrees
- moved C57 0.76 mm to (81.2, 92.7)
- moved C10 0.38 mm to (134.0, 39.8)
- moved C35 0.38 mm to (134.0, 44.6)
- moved C50 0.38 mm to (134.0, 47.0)
- moved C51 0.38 mm to (134.0, 42.2)
- moved C9 0.38 mm to (134.0, 37.3)
Connections:
- removed net N$49: Q2.D, U$7.A
- new net COIL_IN: P2.3, P2.7, Q2.D, U$7.A
- net CAP_0V: now also P2.4, P2.8
- net CAP_330V: now also P2.1, P2.2, P2.5, P2.6
Routing:
- net CAP_330V: track 68.3 -> 113.5 mm
- net CHARGE: track 45.8 -> 75.2 mm, vias 2 -> 4
- net COIL_IN: track 0.00 -> 25.6 mm
- net N$17: track 39.6 -> 56.8 mm, vias 0 -> 1
- net 24V_BOOSTER: track 177.7 -> 192.8 mm
- net N$48: track 0.00 -> 14.5 mm
- net GND1: track 56.2 -> 68.7 mm, vias 1 -> 7
- net N$39: track 13.5 -> 25.8 mm
- net N$44: track 6.64 -> 16.8 mm
- net +5V/3: track 10.3 -> 18.5 mm
- net +3V3: track 60.4 -> 66.9 mm
- net +5V: track 285.0 -> 289.0 mm
- net N$53: track 0.00 -> 3.86 mm
- net N$27: track 31.3 -> 29.3 mm
- net N$9: track 0.00 -> 1.84 mm
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- added copper zone on layer 1, net CAP_0V
- added copper zone on layer 16, net CAP_0V
- added copper zone on layer 1, net GND
- added copper zone on layer 16, net GND
- added copper zone on layer 1, net GND1
- added copper zone on layer 16, net GND1

Commit message: rekick2016 robocup workshop
Parts:
- moved X1 1.02 mm to (121.4, 23.6)
- moved X2 0.64 mm to (103.9, 88.5), turned to 180 degrees
Connections:
- removed net N$15: R4.2, R5.1
- removed net N$17: Q3.S, R63.P$1, U$9.12
- removed net N$18: Q3.G, R66.2
- removed net N$24: Q3.D, R3.2, R61.1, R62.1, R74.2, U$3.10, U$3.11, U$3.12, U$3.9
- removed net N$27: R6.2, R9.1, U6.12
- removed net N$8: C38.1, R5.2, R6.1, U5.12
- new net ADC_SPANNUNGSTEILER: C38.1, R5.2, R6.1, U5.12, X2.2
- new net AFTER_1MOHM_SPANNUNGSTEILER: R4.2, R5.1, X2.1
- new net BEFORE_MOSFET: Q3.D, R3.2, R61.1, R62.1, R74.2, U$3.10, U$3.11, U$3.12, U$3.9, X1.5, X1.6, X1.7, X1.8
- new net CSP: Q3.S, R63.P$1, U$9.12, X1.2
- new net FB_SPANNUNGSTEILER: R6.2, R9.1, U6.12, X2.3
- new net GATE: Q3.G, R66.2, X1.3, X1.4
- net CAP_0V: now also X2.4
- net GND1: now also X1.1, X1.10, X1.11, X1.12, X1.9
Routing:
- net BEFORE_MOSFET: track 0.00 -> 71.7 mm, vias 0 -> 2
- net CSP: track 0.00 -> 59.3 mm, vias 0 -> 2
- net N$24: track 57.3 -> 0.00 mm, vias 2 -> 0
- net N$17: track 56.8 -> 0.00 mm, vias 1 -> 0
- net GND1: track 68.7 -> 103.5 mm, vias 7 -> 8
- net FB_SPANNUNGSTEILER: track 0.00 -> 33.8 mm
- net N$27: track 29.3 -> 0.00 mm
- net ADC_SPANNUNGSTEILER: track 0.00 -> 20.1 mm, vias 0 -> 1
- net GATE: track 0.00 -> 15.6 mm
- net N$8: track 13.6 -> 0.00 mm, vias 1 -> 0
- net AFTER_1MOHM_SPANNUNGSTEILER: track 0.00 -> 8.37 mm
- net N$18: track 6.10 -> 0.00 mm
- net N$15: track 3.81 -> 0.00 mm
- net INT_ETH: track 29.5 -> 28.4 mm
- net ADC_24V_BOOSTER: track 28.4 -> 29.1 mm
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
Commit message: rekick 2016 + extra boards
Parts:
- X1: value 87832-12 -> 79109-12; device con-molex:87832-12 -> con-molex-milli-grid:79109-12
- X2: value 87832-04 -> 79109-04; device con-molex:87832-04 -> con-molex-milli-grid:79109-04
Connections:
- net BEFORE_MOSFET renamed DRAIN_MOSFET
Routing:
- net GND1: track 103.5 -> 124.9 mm
- net DRAIN_MOSFET: track 71.7 -> 85.1 mm
- net GATE: track 15.6 -> 21.2 mm
- net FB_SPANNUNGSTEILER: track 33.8 -> 38.6 mm
- net AFTER_1MOHM_SPANNUNGSTEILER: track 8.37 -> 13.1 mm
- net ADC_SPANNUNGSTEILER: track 20.1 -> 23.8 mm
- net CSP: track 59.3 -> 62.3 mm
Changed lines of the file:
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@@
 <attribute name="OC_NEWARK" value="unknown" x="135.89" y="88.646" size="1.778" layer="27" rot="R90" display="off"/>
 </element>
-<element name="X1" library="con-molex" package="87832-12" value="87832-12" x="121.412" y="23.622">
-<attribute name="OC_FARNELL" value="1756948" x="121.412" y="23.622" size="1.778" layer="27" display="off"/>
-<attribute name="MPN" value="" x="121.412" y="23.622" size="1.778" layer="27" display="off"/>
-<attribute name="MF" value="" x="121.412" y="23.622" size="1.778" layer="27" display="off"/>
-<attribute name="OC_NEWARK" value="unknown" x="121.412" y="23.622" size="1.778" layer="27" display="off"/>
-</element>
+<element name="X1" library="con-molex-milli-grid" package="79109-12" value="79109-12" x="121.412" y="23.622"/>
 <element name="C43" library="rcl" package="C1206" value="10µ/50V" x="100.584" y="55.626" rot="MR270"/>
 <element name="C29" library="rcl" package="C1206" value="10µ/50V" x="100.584" y="46.355" rot="MR90"/>
-<element name="X2" library="con-molex" package="87832-04" value="87832-04" x="103.886" y="88.519" rot="R180">
-<attribute name="OC_FARNELL" value="unknown" x="103.886" y="88.519" size="1.778" layer="27" rot="R180" display="off"/>
-<attribute name="MF" value="" x="103.886" y="88.519" size="1.778" layer="27" rot="R180" display="off"/>
-<attribute name="OC_NEWARK" value="unknown" x="103.886" y="88.519" size="1.778" layer="27" rot="R180" display="off"/>
-<attribute name="MPN" value="" x="103.886" y="88.519" size="1.778" layer="27" rot="R180" display="off"/>
-</element>
+<element name="X2" library="con-molex-milli-grid" package="79109-04" value="79109-04" x="103.886" y="88.519" rot="R180"/>
 </elements>
 <signals>
@@
 <contactref element="X1" pad="10"/>
 <contactref element="X1" pad="12"/>
-<wire x1="116.412" y1="21.472" x2="114.672" y2="21.472" width="0.254" layer="1"/>
+<wire x1="116.412" y1="26.222" x2="114.672" y2="21.472" width="0.254" layer="1"/>
 <wire x1="114.672" y1="21.472" x2="112.522" y2="23.622" width="0.254" layer="1"/>
 <wire x1="112.522" y1="23.622" x2="112.522" y2="26.416" width="0.254" layer="1"/>
@@
 <via x="112.141" y="26.797" extent="1-16" drill="0.5"/>
 <wire x1="112.141" y1="26.797" x2="111.633" y2="27.305" width="0.254" layer="16"/>
-<wire x1="124.412" y1="21.472" x2="125.34" y2="21.472" width="0.4064" layer="1"/>
+<wire x1="124.412" y1="26.222" x2="125.34" y2="21.472" width="0.4064" layer="1"/>
 <wire x1="125.34" y1="21.472" x2="125.349" y2="21.463" width="0.4064" layer="1"/>
-<wire x1="126.403" y1="25.781" x2="126.412" y2="25.772" width="0.4064" layer="1"/>
-<wire x1="126.412" y1="21.472" x2="125.358" y2="21.472" width="0.4064" layer="1"/>
+<wire x1="126.403" y1="25.781" x2="126.412" y2="21.022" width="0.4064" layer="1"/>
+<wire x1="126.412" y1="26.222" x2="125.358" y2="21.472" width="0.4064" layer="1"/>
 <wire x1="125.358" y1="21.472" x2="125.349" y2="21.463" width="0.4064" layer="1"/>
 <wire x1="125.349" y1="21.463" x2="138.5062" y2="21.463" width="2.54" layer="1"/>
@@
 <wire x1="134.112" y1="25.527" x2="134.872" y2="25.527" width="0.254" layer="1"/>
 <wire x1="134.872" y1="25.527" x2="135.763" y2="24.636" width="0.254" layer="1"/>
-<wire x1="124.412" y1="25.772" x2="124.412" y2="21.472" width="0.8128" layer="1"/>
+<wire x1="124.412" y1="21.022" x2="124.412" y2="26.222" width="0.8128" layer="1"/>
 <wire x1="126.403" y1="25.781" x2="126.403" y2="21.481" width="0.8128" layer="1"/>
-<wire x1="126.403" y1="21.481" x2="126.412" y2="21.472" width="0.8128" layer="1"/>
+<wire x1="126.403" y1="21.481" x2="126.412" y2="26.222" width="0.8128" layer="1"/>
 </signal>
 <signal name="CAP_330V">
@@
 <wire x1="134.62" y1="30.226" x2="134.62" y2="30.734" width="0.254" layer="1"/>
 <contactref element="X1" pad="2"/>
-<wire x1="116.412" y1="25.772" x2="114.055" y2="25.772" width="0.254" layer="1"/>
+<wire x1="116.412" y1="21.022" x2="114.055" y2="25.772" width="0.254" layer="1"/>
 <wire x1="114.055" y1="25.772" x2="114.046" y2="25.781" width="0.254" layer="1"/>
 <via x="114.046" y="25.781" extent="1-16" drill="0.5"/>
@@
 <contactref element="X1" pad="4"/>
 <contactref element="X1" pad="3"/>
-<wire x1="118.412" y1="21.472" x2="118.412" y2="25.772" width="0.4064" layer="1"/>
-<wire x1="118.412" y1="25.772" x2="118.412" y2="30.274" width="0.4064" layer="1"/>
+<wire x1="118.412" y1="26.222" x2="118.412" y2="21.022" width="0.4064" layer="1"/>
+<wire x1="118.412" y1="21.022" x2="118.412" y2="30.274" width="0.4064" layer="1"/>
 <wire x1="118.412" y1="30.274" x2="118.872" y2="30.734" width="0.4064" layer="1"/>
 </signal>
@@
 <contactref element="X2" pad="1"/>
 <wire x1="105.283" y1="95.062" x2="104.886" y2="94.665" width="0.254" layer="1"/>
-<wire x1="104.886" y1="94.665" x2="104.886" y2="90.669" width="0.254" layer="1"/>
+<wire x1="104.886" y1="94.665" x2="104.886" y2="85.919" width="0.254" layer="1"/>
 </signal>
 <signal name="N$21">
@@
 <contactref element="X2" pad="3"/>
 <wire x1="102.489" y1="95.062" x2="102.886" y2="94.665" width="0.254" layer="1"/>
-<wire x1="102.886" y1="94.665" x2="102.886" y2="90.669" width="0.254" layer="1"/>
+<wire x1="102.886" y1="94.665" x2="102.886" y2="85.919" width="0.254" layer="1"/>
 </signal>
 <signal name="N$35">
@@
 <wire x1="103.886" y1="93.218" x2="103.886" y2="87.884" width="0.254" layer="1"/>
 <wire x1="103.886" y1="87.884" x2="104.886" y2="86.884" width="0.254" layer="1"/>
-<wire x1="104.886" y1="86.884" x2="104.886" y2="86.369" width="0.254" layer="1"/>
+<wire x1="104.886" y1="86.884" x2="104.886" y2="91.119" width="0.254" layer="1"/>
 <wire x1="103.544" y1="91.059" x2="103.886" y2="91.401" width="0.254" layer="16"/>
 <wire x1="103.886" y1="91.401" x2="103.886" y2="93.218" width="0.254" layer="16"/>
@@
 <wire x1="132.08" y1="91.186" x2="135.89" y2="91.186" width="1.016" layer="16"/>
 </signal>
-<signal name="BEFORE_MOSFET">
+<signal name="DRAIN_MOSFET">
 <contactref element="X1" pad="5"/>
 <contactref element="X1" pad="7"/>
@@
 <wire x1="121.412" y1="25.654" x2="121.412" y2="21.463" width="1.6764" layer="1"/>
 <wire x1="121.412" y1="21.463" x2="120.421" y2="21.463" width="0.4064" layer="1"/>
-<wire x1="120.421" y1="21.463" x2="120.412" y2="21.472" width="0.4064" layer="1"/>
+<wire x1="120.421" y1="21.463" x2="120.412" y2="26.222" width="0.4064" layer="1"/>
 <wire x1="121.412" y1="21.463" x2="122.403" y2="21.463" width="0.4064" layer="1"/>
-<wire x1="122.403" y1="21.463" x2="122.412" y2="21.472" width="0.4064" layer="1"/>
-<wire x1="120.412" y1="25.772" x2="122.412" y2="25.772" width="0.4064" layer="1"/>
-<wire x1="122.412" y1="25.772" x2="121.53" y2="25.772" width="0.4064" layer="1"/>
+<wire x1="122.403" y1="21.463" x2="122.412" y2="26.222" width="0.4064" layer="1"/>
+<wire x1="120.412" y1="21.022" x2="122.412" y2="21.022" width="0.4064" layer="1"/>
+<wire x1="122.412" y1="21.022" x2="121.53" y2="25.772" width="0.4064" layer="1"/>
 <wire x1="121.53" y1="25.772" x2="121.412" y2="25.654" width="0.4064" layer="1"/>
 </signal>

Commit message: rekick board  and  powerswitch board changes
Parts:
- R21, R25, R26, R29, R34, R36: device resistor-power:KH208R-8 -> resistor-power:KH214R-8
- moved R29 27.3 mm to (147.6, 93.0), turned to 270 degrees
- moved R21 27.0 mm to (142.7, 86.0), turned to 90 degrees
- moved R34 13.5 mm to (137.9, 93.0)
- moved R26 11.6 mm to (123.4, 86.0), turned to 90 degrees
- moved R36 8.76 mm to (128.3, 93.0), turned to 270 degrees
- moved C25 6.95 mm to (154.7, 86.6), turned to 0 degrees
- moved R25 5.51 mm to (133.1, 86.0)
- moved Q6 4.19 mm to (114.9, 77.4)
- moved C11 4.06 mm to (152.0, 69.3)
- moved P2 4.06 mm to (146.1, 69.3)
- moved D9 3.01 mm to (154.6, 54.9)
- moved U$7 2.95 mm to (133.7, 69.8)
- moved C52 0.63 mm to (152.0, 42.5)
- moved C55 0.63 mm to (147.6, 36.7)
- moved C56 0.63 mm to (147.6, 48.4)
Connections:
- new net N$8: R25.2, R26.1, R34.2, R36.1
- net CAP_330V: now also R29.1; no longer R26.1, R34.1
- net N$13: now also R25.1, R34.1; no longer R25.2, R26.2, R34.2, R36.2
- net N$51: now also R26.2, R36.2; no longer R25.1, R29.1, R36.1
Routing:
- net CAP_330V: track 113.5 -> 26.9 mm
- net N$51: track 27.1 -> 0.00 mm
- net N$13: track 19.0 -> 0.00 mm
- net COIL_IN: track 25.6 -> 13.9 mm
- net N$39: track 25.8 -> 22.7 mm
- net 24V_BOOSTER: track 192.8 -> 190.9 mm
