File: msl_electronic_boards/rekick2015/pcb/rekick2016-Flyback-v2.sch (EAGLE design)
At the start: 201 parts, among them IC1 74LVC1G02GW, IC2 4043D, IC3 LM1117, IC4 LM1458D, P1 39-30-06_S, P2 39-30-08_S, Q1 16MHz, Q2 IKW 25N120, Q3 PSMN7R8-120PS, Q5 IPD90P04P4L, Q6 IRF840, T1 BC859, T2 BC849, T3 BC849, T4 BC849, T5 IRLML6344TRPBF, T6 BC859, U1 TXB0108PWR, U3 LM2675, U4 LM2675, U5 ADUM4190BRIZ, U6 ADUM4190BRIZ, X1 87832-12, X2 87832-04

Commit message: rekick 2016 layout
Connections:
- removed net N$23: R26.2, R29.2
- removed net N$25: R34.2, R36.2
- net N$13: now also R26.2, R29.2, R34.2, R36.2
Changed lines of the file:
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@@
 <pinref part="R21" gate="G$1" pin="2"/>
 <wire x1="139.7" y1="96.52" x2="139.7" y2="93.98" width="0.1524" layer="91"/>
-</segment>
-</net>
-<net name="N$23" class="0">
-<segment>
 <pinref part="R29" gate="G$1" pin="2"/>
 <pinref part="R26" gate="G$1" pin="2"/>
 <wire x1="144.78" y1="96.52" x2="144.78" y2="93.98" width="0.1524" layer="91"/>
-</segment>
-</net>
-<net name="N$25" class="0">
-<segment>
+<wire x1="139.7" y1="93.98" x2="144.78" y2="93.98" width="0.1524" layer="91"/>
+<junction x="139.7" y="93.98"/>
+<junction x="144.78" y="93.98"/>
 <pinref part="R36" gate="G$1" pin="2"/>
 <pinref part="R34" gate="G$1" pin="2"/>
 <wire x1="149.86" y1="96.52" x2="149.86" y2="93.98" width="0.1524" layer="91"/>
+<wire x1="144.78" y1="93.98" x2="149.86" y2="93.98" width="0.1524" layer="91"/>
+<junction x="149.86" y="93.98"/>
 </segment>
 </net>

Commit message: rekick 2016 v2 done for robocup workshop
Connections:
- removed net N$49: Q2.D, U$7.A
- new net COIL_IN: P2-3.P, P2-7.P, Q2.D, U$7.A
- net CAP_0V: now also P2-4.P, P2-8.P
- net CAP_330V: now also P2-1.P, P2-2.P, P2-5.P, P2-6.P
Other:
- moved on the sheet: P2, P2-2, P2-3, P2-4, P2-5, P2-6, P2-7, P2-8
Changed lines of the file:
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@@
 <instance part="P1" gate="-5" x="71.12" y="147.32"/>
 <instance part="P1" gate="-6" x="71.12" y="144.78"/>
-<instance part="P2" gate="-1" x="71.12" y="127"/>
-<instance part="P2" gate="-2" x="71.12" y="124.46"/>
-<instance part="P2" gate="-3" x="71.12" y="121.92"/>
-<instance part="P2" gate="-4" x="71.12" y="119.38"/>
-<instance part="P2" gate="-5" x="71.12" y="116.84"/>
-<instance part="P2" gate="-6" x="71.12" y="114.3"/>
-<instance part="P2" gate="-7" x="71.12" y="111.76"/>
-<instance part="P2" gate="-8" x="71.12" y="109.22"/>
+<instance part="P2" gate="-1" x="68.58" y="114.3"/>
+<instance part="P2" gate="-2" x="68.58" y="111.76"/>
+<instance part="P2" gate="-3" x="68.58" y="109.22"/>
+<instance part="P2" gate="-4" x="68.58" y="106.68"/>
+<instance part="P2" gate="-5" x="68.58" y="104.14"/>
+<instance part="P2" gate="-6" x="68.58" y="101.6"/>
+<instance part="P2" gate="-7" x="68.58" y="99.06"/>
+<instance part="P2" gate="-8" x="68.58" y="96.52"/>
 <instance part="SUPPLY23" gate="G$1" x="55.88" y="142.24"/>
 <instance part="GND41" gate="1" x="63.5" y="139.7"/>
@@
 <wire x1="215.9" y1="55.88" x2="220.98" y2="55.88" width="0.1524" layer="91"/>
 </segment>
+<segment>
+<pinref part="P2" gate="-4" pin="P"/>
+<wire x1="66.04" y1="106.68" x2="58.42" y2="106.68" width="0.1524" layer="91"/>
+<wire x1="58.42" y1="106.68" x2="58.42" y2="96.52" width="0.1524" layer="91"/>
+<pinref part="P2" gate="-8" pin="P"/>
+<wire x1="66.04" y1="96.52" x2="58.42" y2="96.52" width="0.1524" layer="91"/>
+<wire x1="58.42" y1="106.68" x2="55.88" y2="106.68" width="0.1524" layer="91"/>
+<junction x="58.42" y="106.68"/>
+<label x="55.88" y="106.68" size="1.27" layer="95" rot="R180" xref="yes"/>
+</segment>
 </net>
 <net name="CAN_H" class="0">
@@
 <wire x1="55.88" y1="147.32" x2="55.88" y2="144.78" width="0.1524" layer="91"/>
 <junction x="63.5" y="147.32"/>
+</segment>
+</net>
+<net name="CAP_330V" class="0">
+<segment>
+<pinref part="P2" gate="-5" pin="P"/>
+<wire x1="66.04" y1="104.14" x2="63.5" y2="104.14" width="0.1524" layer="91"/>
+<wire x1="63.5" y1="104.14" x2="63.5" y2="101.6" width="0.1524" layer="91"/>
+<pinref part="P2" gate="-6" pin="P"/>
+<wire x1="63.5" y1="101.6" x2="66.04" y2="101.6" width="0.1524" layer="91"/>
+<pinref part="P2" gate="-2" pin="P"/>
+<wire x1="66.04" y1="111.76" x2="63.5" y2="111.76" width="0.1524" layer="91"/>
+<wire x1="63.5" y1="111.76" x2="63.5" y2="114.3" width="0.1524" layer="91"/>
+<pinref part="P2" gate="-1" pin="P"/>
+<wire x1="63.5" y1="114.3" x2="66.04" y2="114.3" width="0.1524" layer="91"/>
+<wire x1="63.5" y1="104.14" x2="63.5" y2="111.76" width="0.1524" layer="91"/>
+<junction x="63.5" y="104.14"/>
+<junction x="63.5" y="111.76"/>
+<wire x1="63.5" y1="111.76" x2="55.88" y2="111.76" width="0.1524" layer="91"/>
+<label x="55.88" y="111.76" size="1.27" layer="95" rot="R180" xref="yes"/>
+</segment>
+</net>
+<net name="COIL_IN" class="0">
+<segment>
+<pinref part="P2" gate="-7" pin="P"/>
+<wire x1="66.04" y1="99.06" x2="60.96" y2="99.06" width="0.1524" layer="91"/>
+<pinref part="P2" gate="-3" pin="P"/>
+<wire x1="66.04" y1="109.22" x2="60.96" y2="109.22" width="0.1524" layer="91"/>
+<wire x1="60.96" y1="99.06" x2="60.96" y2="109.22" width="0.1524" layer="91"/>
+<wire x1="60.96" y1="109.22" x2="55.88" y2="109.22" width="0.1524" layer="91"/>
+<junction x="60.96" y="109.22"/>
+<label x="55.88" y="109.22" size="1.27" layer="95" rot="R180" xref="yes"/>
 </segment>
 </net>
@@
 </segment>
 </net>
-<net name="N$49" class="0">
+<net name="COIL_IN" class="0">
 <segment>
 <pinref part="Q2" gate="1" pin="D"/>
-<wire x1="142.24" y1="147.32" x2="142.24" y2="152.4" width="0.1524" layer="91"/>
+<wire x1="142.24" y1="147.32" x2="142.24" y2="149.86" width="0.1524" layer="91"/>
 <pinref part="U$7" gate="G$1" pin="A"/>
-</segment>
-</net>
+<wire x1="142.24" y1="149.86" x2="142.24" y2="152.4" width="0.1524" layer="91"/>
+<wire x1="142.24" y1="149.86" x2="147.32" y2="149.86" width="0.1524" layer="91"/>
+<junction x="142.24" y="149.86"/>
+<label x="147.32" y="149.86" size="1.27" layer="95" xref="yes"/>
+</segment>
+</net>

Commit message: rekick2016 robocup workshop
Connections:
- removed net N$15: R4.2, R5.1
- removed net N$17: Q3.S, R63.1, U$9.CSP
- removed net N$18: Q3.G, R66.2
- removed net N$24: Q3.D, R3.2, R61.1, R62.1, R74.2, U$3.W12, U$3.W22, U$3.W32, U$3.W42
- removed net N$27: R6.2, R9.1, U6.+IN
- removed net N$8: C38.1, R5.2, R6.1, U5.+IN
- new net ADC_SPANNUNGSTEILER: C38.1, R5.2, R6.1, U5.+IN, X2.2
- new net AFTER_1MOHM_SPANNUNGSTEILER: R4.2, R5.1, X2.1
- new net BEFORE_MOSFET: Q3.D, R3.2, R61.1, R62.1, R74.2, U$3.W12, U$3.W22, U$3.W32, U$3.W42, X1.5, X1.6, X1.7, X1.8
- new net CSP: Q3.S, R63.1, U$9.CSP, X1.2
- new net FB_SPANNUNGSTEILER: R6.2, R9.1, U6.+IN, X2.3
- new net GATE: Q3.G, R66.2, X1.3, X1.4
- net CAP_0V: now also X2.4
- net GND1: now also X1.1, X1.10, X1.11, X1.12, X1.9
Other:
- moved on the sheet: R60, R66, X1, X2

Commit message: rekick 2016 + extra boards
Parts:
- X1: value 87832-12 -> 79109-12; device con-molex:87832-12 -> con-molex-milli-grid:79109-12
- X2: value 87832-04 -> 79109-04; device con-molex:87832-04 -> con-molex-milli-grid:79109-04
Connections:
- net BEFORE_MOSFET renamed DRAIN_MOSFET
Other:
- moved on the sheet: X1, X2
Changed lines of the file:
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@@
 <part name="R34" library="resistor-power" deviceset="R" device="KH208-8R"/>
 <part name="R36" library="resistor-power" deviceset="R" device="KH208-8R"/>
-<part name="X1" library="con-molex" deviceset="87832-12" device=""/>
+<part name="X1" library="con-molex-milli-grid" deviceset="79109-12" device=""/>
 <part name="C43" library="rcl" deviceset="C-EU" device="C1206" value="10µ/50V"/>
 <part name="C29" library="rcl" deviceset="C-EU" device="C1206" value="10µ/50V"/>
-<part name="X2" library="con-molex" deviceset="87832-04" device=""/>
+<part name="X2" library="con-molex-milli-grid" deviceset="79109-04" device=""/>
 <part name="P+17" library="supply1" deviceset="+12V" device=""/>
 <part name="SUPPLY24" library="supply2" deviceset="GND1" device=""/>
@@
 <pinref part="SUPPLY24" gate="G$1" pin="GND1"/>
 <wire x1="50.8" y1="60.96" x2="50.8" y2="63.5" width="0.1524" layer="91"/>
-<wire x1="50.8" y1="63.5" x2="60.96" y2="63.5" width="0.1524" layer="91"/>
+<wire x1="50.8" y1="63.5" x2="58.42" y2="63.5" width="0.1524" layer="91"/>
 <pinref part="X1" gate="G$1" pin="1"/>
 </segment>
@@
 <pinref part="X1" gate="G$1" pin="9"/>
 <pinref part="X1" gate="G$1" pin="11"/>
-<wire x1="60.96" y1="53.34" x2="60.96" y2="50.8" width="0.1524" layer="91"/>
+<wire x1="58.42" y1="53.34" x2="58.42" y2="50.8" width="0.1524" layer="91"/>
 <pinref part="X1" gate="G$1" pin="10"/>
-<wire x1="60.96" y1="53.34" x2="73.66" y2="53.34" width="0.1524" layer="91"/>
-<junction x="60.96" y="53.34"/>
+<wire x1="58.42" y1="53.34" x2="73.66" y2="53.34" width="0.1524" layer="91"/>
+<junction x="58.42" y="53.34"/>
 <pinref part="X1" gate="G$1" pin="12"/>
 <wire x1="73.66" y1="53.34" x2="73.66" y2="50.8" width="0.1524" layer="91"/>
 <junction x="73.66" y="53.34"/>
-<wire x1="73.66" y1="53.34" x2="78.74" y2="53.34" width="0.1524" layer="91"/>
-<label x="78.74" y="53.34" size="1.27" layer="95" xref="yes"/>
+<wire x1="73.66" y1="53.34" x2="76.2" y2="53.34" width="0.1524" layer="91"/>
+<label x="76.2" y="53.34" size="1.27" layer="95" xref="yes"/>
 </segment>
 </net>
@@
 <segment>
 <pinref part="X2" gate="G$1" pin="1"/>
-<wire x1="60.96" y1="38.1" x2="58.42" y2="38.1" width="0.1524" layer="91"/>
-<label x="58.42" y="38.1" size="1.27" layer="95" rot="R180" xref="yes"/>
+<wire x1="58.42" y1="38.1" x2="55.88" y2="38.1" width="0.1524" layer="91"/>
+<label x="55.88" y="38.1" size="1.27" layer="95" rot="R180" xref="yes"/>
 </segment>
 </net>
@@
 <segment>
 <pinref part="X2" gate="G$1" pin="3"/>
-<wire x1="58.42" y1="35.56" x2="60.96" y2="35.56" width="0.1524" layer="91"/>
-<label x="58.42" y="35.56" size="1.27" layer="95" rot="R180" xref="yes"/>
+<wire x1="55.88" y1="35.56" x2="58.42" y2="35.56" width="0.1524" layer="91"/>
+<label x="55.88" y="35.56" size="1.27" layer="95" rot="R180" xref="yes"/>
 </segment>
 </net>
@@
 <segment>
 <pinref part="X1" gate="G$1" pin="2"/>
-<wire x1="73.66" y1="63.5" x2="78.74" y2="63.5" width="0.1524" layer="91"/>
-<label x="78.74" y="63.5" size="1.27" layer="95" xref="yes"/>
+<wire x1="73.66" y1="63.5" x2="76.2" y2="63.5" width="0.1524" layer="91"/>
+<label x="76.2" y="63.5" size="1.27" layer="95" xref="yes"/>
 </segment>
 </net>
@@
 <segment>
 <pinref part="X1" gate="G$1" pin="4"/>
-<wire x1="73.66" y1="60.96" x2="78.74" y2="60.96" width="0.1524" layer="91"/>
+<wire x1="73.66" y1="60.96" x2="76.2" y2="60.96" width="0.1524" layer="91"/>
 <pinref part="X1" gate="G$1" pin="3"/>
-<wire x1="60.96" y1="60.96" x2="73.66" y2="60.96" width="0.1524" layer="91"/>
+<wire x1="58.42" y1="60.96" x2="73.66" y2="60.96" width="0.1524" layer="91"/>
 <junction x="73.66" y="60.96"/>
-<label x="78.74" y="60.96" size="1.27" layer="95" xref="yes"/>
-</segment>
-</net>
-<net name="BEFORE_MOSFET" class="0">
+<label x="76.2" y="60.96" size="1.27" layer="95" xref="yes"/>
+</segment>
+</net>
+<net name="DRAIN_MOSFET" class="0">
 <segment>
 <pinref part="X1" gate="G$1" pin="5"/>
 <pinref part="X1" gate="G$1" pin="7"/>
-<wire x1="60.96" y1="58.42" x2="60.96" y2="55.88" width="0.1524" layer="91"/>
+<wire x1="58.42" y1="58.42" x2="58.42" y2="55.88" width="0.1524" layer="91"/>
 <pinref part="X1" gate="G$1" pin="6"/>
-<wire x1="60.96" y1="58.42" x2="73.66" y2="58.42" width="0.1524" layer="91"/>
-<junction x="60.96" y="58.42"/>
+<wire x1="58.42" y1="58.42" x2="73.66" y2="58.42" width="0.1524" layer="91"/>
+<junction x="58.42" y="58.42"/>
 <pinref part="X1" gate="G$1" pin="8"/>
 <wire x1="73.66" y1="58.42" x2="73.66" y2="55.88" width="0.1524" layer="91"/>
 <junction x="73.66" y="58.42"/>
-<wire x1="73.66" y1="58.42" x2="78.74" y2="58.42" width="0.1524" layer="91"/>
-<label x="78.74" y="58.42" size="1.27" layer="95" xref="yes"/>
+<wire x1="73.66" y1="58.42" x2="76.2" y2="58.42" width="0.1524" layer="91"/>
+<label x="76.2" y="58.42" size="1.27" layer="95" xref="yes"/>
 </segment>
 </net>
@@
 </segment>
 </net>
-<net name="BEFORE_MOSFET" class="0">
+<net name="DRAIN_MOSFET" class="0">
 <segment>
 <pinref part="R61" gate="G$1" pin="1"/>

Commit message: rekick board  and  powerswitch board changes
Parts:
- R21, R25, R26, R29, R34, R36: device resistor-power:RKH208-8R -> resistor-power:RKH214-8R
Connections:
- new net N$8: R25.2, R26.1, R34.2, R36.1
- net CAP_330V: now also R29.1; no longer R26.1, R34.1
- net N$13: now also R25.1, R34.1; no longer R25.2, R26.2, R34.2, R36.2
- net N$51: now also R26.2, R36.2; no longer R25.1, R29.1, R36.1
Other:
- moved on the sheet: R21, R25, R26, R29, R34, R36
Changed lines of the file:
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@@
 <part name="SUPPLY20" library="supply2" deviceset="0V" device="" value="CAP_0V"/>
 <part name="GND29" library="supply1" deviceset="GND" device=""/>
-<part name="R21" library="resistor-power" deviceset="R" device="KH208-8R"/>
-<part name="R25" library="resistor-power" deviceset="R" device="KH208-8R"/>
-<part name="R26" library="resistor-power" deviceset="R" device="KH208-8R"/>
-<part name="R29" library="resistor-power" deviceset="R" device="KH208-8R"/>
+<part name="R21" library="resistor-power" deviceset="R" device="KH214-8R"/>
+<part name="R25" library="resistor-power" deviceset="R" device="KH214-8R"/>
+<part name="R26" library="resistor-power" deviceset="R" device="KH214-8R"/>
+<part name="R29" library="resistor-power" deviceset="R" device="KH214-8R"/>
 <part name="FRAME8" library="frames" deviceset="A4L-LOC" device=""/>
 <part name="GND30" library="supply1" deviceset="GND" device=""/>
@@
 <part name="SUPPLY23" library="supply2" deviceset="GND1" device=""/>
 <part name="GND41" library="supply1" deviceset="GND" device=""/>
-<part name="R34" library="resistor-power" deviceset="R" device="KH208-8R"/>
-<part name="R36" library="resistor-power" deviceset="R" device="KH208-8R"/>
+<part name="R34" library="resistor-power" deviceset="R" device="KH214-8R"/>
+<part name="R36" library="resistor-power" deviceset="R" device="KH214-8R"/>
 <part name="X1" library="con-molex-milli-grid" deviceset="79109-12" device=""/>
 <part name="C43" library="rcl" deviceset="C-EU" device="C1206" value="10µ/50V"/>
@@
 <instance part="R11" gate="G$1" x="119.38" y="66.04" rot="R90"/>
 <instance part="R2" gate="G$1" x="124.46" y="93.98" rot="R270"/>
-<instance part="R21" gate="G$1" x="139.7" y="101.6" rot="R270"/>
-<instance part="R25" gate="G$1" x="139.7" y="88.9" rot="R90"/>
-<instance part="R26" gate="G$1" x="144.78" y="101.6" rot="R270"/>
-<instance part="R29" gate="G$1" x="144.78" y="88.9" rot="R90"/>
-<instance part="R34" gate="G$1" x="149.86" y="101.6" rot="R270"/>
-<instance part="R36" gate="G$1" x="149.86" y="88.9" rot="R90"/>
+<instance part="R21" gate="G$1" x="139.7" y="109.22" rot="R270"/>
+<instance part="R25" gate="G$1" x="139.7" y="99.06" rot="R270"/>
+<instance part="R26" gate="G$1" x="139.7" y="88.9" rot="R270"/>
+<instance part="R29" gate="G$1" x="147.32" y="109.22" rot="R270"/>
+<instance part="R34" gate="G$1" x="147.32" y="99.06" rot="R270"/>
+<instance part="R36" gate="G$1" x="147.32" y="88.9" rot="R270"/>
 </instances>
 <busses>
@@
 </segment>
 <segment>
-<label x="127" y="109.22" size="1.778" layer="95" rot="R180" xref="yes"/>
-<wire x1="127" y1="109.22" x2="132.08" y2="109.22" width="0.1524" layer="91"/>
+<label x="129.54" y="114.3" size="1.778" layer="95" rot="R180" xref="yes"/>
+<wire x1="129.54" y1="114.3" x2="132.08" y2="114.3" width="0.1524" layer="91"/>
 <pinref part="R10" gate="G$1" pin="1"/>
-<wire x1="132.08" y1="109.22" x2="139.7" y2="109.22" width="0.1524" layer="91"/>
-<wire x1="139.7" y1="109.22" x2="144.78" y2="109.22" width="0.1524" layer="91"/>
-<wire x1="144.78" y1="109.22" x2="149.86" y2="109.22" width="0.1524" layer="91"/>
-<wire x1="132.08" y1="99.06" x2="132.08" y2="109.22" width="0.1524" layer="91"/>
-<junction x="132.08" y="109.22"/>
+<wire x1="132.08" y1="114.3" x2="139.7" y2="114.3" width="0.1524" layer="91"/>
+<wire x1="139.7" y1="114.3" x2="147.32" y2="114.3" width="0.1524" layer="91"/>
+<wire x1="147.32" y1="114.3" x2="149.86" y2="114.3" width="0.1524" layer="91"/>
+<wire x1="132.08" y1="99.06" x2="132.08" y2="114.3" width="0.1524" layer="91"/>
+<junction x="132.08" y="114.3"/>
 <pinref part="R2" gate="G$1" pin="1"/>
 <wire x1="124.46" y1="99.06" x2="132.08" y2="99.06" width="0.1524" layer="91"/>
 <junction x="132.08" y="99.06"/>
 <pinref part="R21" gate="G$1" pin="1"/>
-<wire x1="139.7" y1="106.68" x2="139.7" y2="109.22" width="0.1524" layer="91"/>
-<junction x="139.7" y="109.22"/>
-<pinref part="R26" gate="G$1" pin="1"/>
-<wire x1="144.78" y1="106.68" x2="144.78" y2="109.22" width="0.1524" layer="91"/>
-<junction x="144.78" y="109.22"/>
-<pinref part="R34" gate="G$1" pin="1"/>
-<wire x1="149.86" y1="106.68" x2="149.86" y2="109.22" width="0.1524" layer="91"/>
+<junction x="139.7" y="114.3"/>
+<pinref part="R29" gate="G$1" pin="1"/>
+<junction x="147.32" y="114.3"/>
 </segment>
 </net>
@@
 <segment>
 <pinref part="Q6" gate="G$1" pin="D"/>
+<wire x1="139.7" y1="83.82" x2="139.7" y2="81.28" width="0.1524" layer="91"/>
+<pinref part="R26" gate="G$1" pin="2"/>
+<pinref part="R36" gate="G$1" pin="2"/>
+<wire x1="139.7" y1="81.28" x2="139.7" y2="78.74" width="0.1524" layer="91"/>
+<wire x1="139.7" y1="81.28" x2="147.32" y2="81.28" width="0.1524" layer="91"/>
+<wire x1="147.32" y1="81.28" x2="147.32" y2="83.82" width="0.1524" layer="91"/>
+<junction x="139.7" y="81.28"/>
+</segment>
+</net>
+<net name="N$8" class="0">
+<segment>
+<pinref part="R26" gate="G$1" pin="1"/>
+<pinref part="R25" gate="G$1" pin="2"/>
+<pinref part="R34" gate="G$1" pin="2"/>
+<pinref part="R36" gate="G$1" pin="1"/>
+<wire x1="139.7" y1="93.98" x2="147.32" y2="93.98" width="0.1524" layer="91"/>
+<junction x="139.7" y="93.98"/>
+<junction x="147.32" y="93.98"/>
+</segment>
+</net>
+<net name="N$13" class="0">
+<segment>
 <pinref part="R25" gate="G$1" pin="1"/>
-<wire x1="139.7" y1="83.82" x2="139.7" y2="81.28" width="0.1524" layer="91"/>
-<pinref part="R29" gate="G$1" pin="1"/>
-<wire x1="139.7" y1="81.28" x2="139.7" y2="78.74" width="0.1524" layer="91"/>
-<wire x1="144.78" y1="83.82" x2="144.78" y2="81.28" width="0.1524" layer="91"/>
-<wire x1="144.78" y1="81.28" x2="139.7" y2="81.28" width="0.1524" layer="91"/>
-<junction x="139.7" y="81.28"/>
-<pinref part="R36" gate="G$1" pin="1"/>
-<wire x1="149.86" y1="83.82" x2="149.86" y2="81.28" width="0.1524" layer="91"/>
-<wire x1="149.86" y1="81.28" x2="144.78" y2="81.28" width="0.1524" layer="91"/>
-<junction x="144.78" y="81.28"/>
-</segment>
-</net>
-<net name="N$13" class="0">
-<segment>
-<pinref part="R25" gate="G$1" pin="2"/>
 <pinref part="R21" gate="G$1" pin="2"/>
-<wire x1="139.7" y1="96.52" x2="139.7" y2="93.98" width="0.1524" layer="91"/>
 <pinref part="R29" gate="G$1" pin="2"/>
-<pinref part="R26" gate="G$1" pin="2"/>
-<wire x1="144.78" y1="96.52" x2="144.78" y2="93.98" width="0.1524" layer="91"/>
-<wire x1="139.7" y1="93.98" x2="144.78" y2="93.98" width="0.1524" layer="91"/>
-<junction x="139.7" y="93.98"/>
-<junction x="144.78" y="93.98"/>
-<pinref part="R36" gate="G$1" pin="2"/>
-<pinref part="R34" gate="G$1" pin="2"/>
-<wire x1="149.86" y1="96.52" x2="149.86" y2="93.98" width="0.1524" layer="91"/>
-<wire x1="144.78" y1="93.98" x2="149.86" y2="93.98" width="0.1524" layer="91"/>
-<junction x="149.86" y="93.98"/>
-</segment>
-</net>
+<pinref part="R34" gate="G$1" pin="1"/>
+<wire x1="139.7" y1="104.14" x2="147.32" y2="104.14" width="0.1524" layer="91"/>
+<junction x="139.7" y="104.14"/>
+<junction x="147.32" y="104.14"/>
+</segment>
+</net>
